Commit message: added v2 platform files

File: rb1_base_description/robots/rb1_base_platform_standalone_v1.urdf.xacro (robot description, xacro)
@@ -33,5 +33,5 @@
 	<xacro:property name="omni_back_z" value="0.0265" />
 	<xacro:property name="omni_front_x" value="0.133" />
-	<xacro:property name="omni_front_y" value="0.148" />
+	<xacro:property name="omni_front_y" value="0.144" />
 	<xacro:property name="omni_front_z" value="0.0265" />
 	<!-- Flag to select the high or low quality model -->
@@ -80,9 +80,8 @@
 		<origin xyz="-0.18 0.0 0.170" rpy="0 0 0"/>
 	</xacro:sensor_imu>
-    <xacro:sensor_orbbec_astra name="orbbec_astra" parent="base_link">
-        <origin xyz="0.234 0.0 0.092" rpy="-1.5708 -1.5708 0"/>
-    </xacro:sensor_orbbec_astra>
-    <!-- xacro:sensor_kinect name="kinect" parent="base_link">
-        <origin xyz="0.6 0.0 0.102" rpy="0 0 0"/>
-    </xacro:sensor_kinect -->
+<!--
+    <xacro:sensor_kinect name="kinect" parent="base_link">
+        <origin xyz="0.3 0.0 0.16" rpy="0 0 0"/>
+    </xacro:sensor_kinect>
+-->
 </robot>

File: rb1_base_description/robots/rb1_base_platform_v1.urdf.xacro (robot description, xacro)
@@ -7,17 +7,9 @@
 	<!-- Import RB1 base elements -->
     <xacro:include filename="$(find rb1_base_description)/urdf/bases/rb1_base.urdf.xacro" />
-    <gazebo>
-      <plugin name="ros_control" filename="libgazebo_ros_control.so">
-        <robotNamespace>/rb1</robotNamespace>
-        <robotParam>robot_description</robotParam>
-        <controlPeriod>0.001</controlPeriod>
-	    <robotSimType>gazebo_ros_control/DefaultRobotHWSim</robotSimType>
-      </plugin>
-    </gazebo>
 	<!-- Import RB1 wheels -->
 	<xacro:include filename="$(find rb1_base_description)/urdf/wheels/rubber_wheel.urdf.xacro" />
 	<xacro:include filename="$(find rb1_base_description)/urdf/wheels/omni_wheel.urdf.xacro" />
 	<!-- Import all available sensors -->
-    <xacro:include filename="$(find robotnik_sensors)/urdf/all_sensors.urdf.xacro"/>
+	<xacro:include filename="$(find robotnik_sensors)/urdf/all_sensors.urdf.xacro" />
 	<!-- ***************** -->
 	<!-- Global parameters -->
@@ -33,5 +25,5 @@
 	<xacro:property name="omni_back_z" value="0.0265" />
 	<xacro:property name="omni_front_x" value="0.133" />
-	<xacro:property name="omni_front_y" value="0.148" />
+	<xacro:property name="omni_front_y" value="0.144" />
 	<xacro:property name="omni_front_z" value="0.0265" />
 	<!-- Flag to select the high or low quality model -->
@@ -68,10 +60,7 @@
 		<origin xyz="0.210 0.0 0.305" rpy="0 0 0"/>
 	</xacro:sensor_hokuyo_utm30lx -->
-    <!-- xacro:sensor_hokuyo_urg04lx name="hokuyo1" parent="base_link">
-        <origin xyz="0.220 0.0 0.170" rpy="0 3.1416 3.1416"/>
+    <!-- xacro:sensor_hokuyo_urg04lx name="hokuyo" parent="base_link">
+        <origin xyz="0.223 0.0 0.209" rpy="0 3.1416 3.1416"/>
     </xacro:sensor_hokuyo_urg04lx -->
-	<!-- xacro:sensor_hokuyo_ust10lx name="hokuyo" parent="base_link">
-		<origin xyz="0.223 0.0 0.159" rpy="0 0 0"/>
-	</xacro:sensor_hokuyo_ust10lx -->
 	<xacro:sensor_hokuyo_ust10lx name="hokuyo" parent="base_link">
 		<origin xyz="0.223 0.0 0.159" rpy="0 3.1416 3.1416"/>
@@ -80,9 +69,8 @@
 		<origin xyz="-0.18 0.0 0.170" rpy="0 0 0"/>
 	</xacro:sensor_imu>
-    <xacro:sensor_orbbec_astra name="orbbec_astra" parent="base_link">
-        <origin xyz="0.234 0.0 0.092" rpy="-1.5708 -1.5708 0"/>
-    </xacro:sensor_orbbec_astra>
-    <!-- xacro:sensor_kinect name="kinect" parent="base_link">
-        <origin xyz="0.6 0.0 0.102" rpy="0 0 0"/>
-    </xacro:sensor_kinect -->
+<!--
+    <xacro:sensor_kinect name="kinect" parent="base_link">
+        <origin xyz="0.3 0.0 0.16" rpy="0 0 0"/>
+    </xacro:sensor_kinect>
+-->
 </robot>

File: rb1_base_description/urdf/bases/rb1_base_v1.urdf.xacro (robot description, xacro)
@@ -33,10 +33,10 @@
        <xacro:if value="${hq}">
        <geometry>
-	     <mesh filename="package://rb1_base_description/meshes/bases/rb1v2_base.dae"/>
+	     <mesh filename="package://rb1_base_description/meshes/bases/rb1_base.dae"/>
        </geometry>
        </xacro:if>
        <xacro:unless value="${hq}">
        <geometry>
-       <mesh filename="package://rb1_base_description/meshes/bases/rb1v2_base.stl"/>
+       <mesh filename="package://rb1_base_description/meshes/bases/rb1_base.stl"/>
        </geometry>
        </xacro:unless>
@@ -48,40 +48,5 @@
        <origin xyz="0 0 0" rpy="0 0 0 " />
        <geometry>
-         <mesh filename="package://rb1_base_description/meshes/bases/rb1v2_base.dae"/>
-       </geometry>
-    </collision>
-  </link>
-  <joint name="front_cover_joint" type="fixed">
-     <origin xyz="0.220 0.0 0.004" rpy="0 0 0 " />
-     <parent link="base_link"/>
-     <child link="front_cover_link" />
-  </joint>
-  <!-- FRONT COVER -->
-  <link name="front_cover_link">
-    <inertial>
-      <mass value="0.25" />
-      <origin xyz="0 0 0" />
-      <inertia  ixx="0.00007" ixy="0.0"  ixz="0.0"  iyy="0.00007"  iyz="0.0"  izz="0.0078" />
-    </inertial>
-    <visual>
-       <origin xyz="0 0 0" rpy="0 0 0" />
-       <xacro:if value="${hq}">
-       <geometry>
-	     <mesh filename="package://rb1_base_description/meshes/bases/rb1v2_front_cover.dae"/>
-       </geometry>
-       </xacro:if>
-       <xacro:unless value="${hq}">
-       <geometry>
-       <mesh filename="package://rb1_base_description/meshes/bases/rb1v2_front_cover.stl"/>
-       </geometry>
-       </xacro:unless>
-       <material name="black">
-         <color rgba="0.0 0.0 0.0 1"/>
-       </material>
-    </visual>
-    <collision>
-       <origin xyz="0 0 0" rpy="0 0 0 " />
-       <geometry>
-         <mesh filename="package://rb1_base_description/meshes/bases/rb1v2_front_cover.dae"/>
+         <mesh filename="package://rb1_base_description/meshes/bases/rb1_base.dae"/>
        </geometry>
     </collision>

File: rb1_base_description/urdf/wheels/omni_wheel_v1.urdf.xacro (robot description, xacro)
@@ -28,5 +28,5 @@
           <origin xyz="0 0 0" rpy="0 0 0" />
           <geometry>
-				<mesh filename="package://rb1_base_description/meshes/wheels/rb1v2_omniwheel.dae" />
+				<mesh filename="package://rb1_base_description/meshes/wheels/wheel_omni_4inch.dae" />
           </geometry>
         </xacro:if>
