Commit message: Minor changes

File: rb1_base_description/robots/rb1_base_v2.urdf.xacro (robot description, xacro)
@@ -65,16 +65,16 @@
 		<origin xyz="0.220 0.0 0.170" rpy="0 3.1416 3.1416"/>
 	</xacro:sensor_hokuyo_urg04lx -->
-	<!-- xacro:sensor_hokuyo_ust10lx name="base_front_laser" parent="base_link">
-		<origin xyz="0.223 0.0 0.159" rpy="0 0 0"/>
-	</xacro:sensor_hokuyo_ust10lx -->
+	<xacro:sensor_hokuyo_ust10lx name="base_front_laser" parent="base_link">
+		<origin xyz="0.223 0.0 0.159" rpy="3.1416 0 0"/>
+	</xacro:sensor_hokuyo_ust10lx>
 	<!-- Name the components as base_front_laser or base_laser or front_laser or
 	a name which identify uniquely the component within the robot -->
-	<xacro:sensor_rplidar_a2 name="base_front_laser" parent="base_link">
+	<!--xacro:sensor_rplidar_a2 name="base_front_laser" parent="base_link">
 		<origin xyz="0.210 0.0 0.199" rpy="3.1415 0 0"/>
-	</xacro:sensor_rplidar_a2>
+	</xacro:sensor_rplidar_a2-->
 	<!-- CAMERA -->
-	<!--xacro:sensor_orbbec_astra name="base_front_camera" parent="base_link">
+	<xacro:sensor_orbbec_astra name="base_front_camera" parent="base_link">
 		<origin xyz="0.234 0.0125 0.107" rpy="0 0 0"/>
-	</xacro:sensor_orbbec_astra-->
+	</xacro:sensor_orbbec_astra>
 	<!-- xacro:sensor_kinect name="base_front_camera" parent="base_link">
 		<origin xyz="0.6 0.0 0.102" rpy="0 0 0"/>

Commit message: Adjusted the position of the wheels

File: rb1_base_description/robots/rb1_base_v2.urdf.xacro (robot description, xacro)
@@ -23,13 +23,13 @@
 	<!-- FOR RUBBER WHEEL -->
 	<xacro:property name="wheel_offset_x" value="0.0" />    <!-- x,y,z in translation from base_link to the center of the wheel -->
-	<xacro:property name="wheel_offset_y" value="0.2165" />
-	<xacro:property name="wheel_offset_z" value="0.0512" />
+	<xacro:property name="wheel_offset_y" value="0.217" />
+	<xacro:property name="wheel_offset_z" value="0.051" />
 	<!-- FOR OMNI WHEEL -->
 	<xacro:property name="omni_back_x" value="0.195" />
 	<xacro:property name="omni_back_y" value="0.0" />
-	<xacro:property name="omni_back_z" value="0.0258" />
+	<xacro:property name="omni_back_z" value="0.0265" />
 	<xacro:property name="omni_front_x" value="0.133" />
 	<xacro:property name="omni_front_y" value="0.148" />
-	<xacro:property name="omni_front_z" value="0.0258" />
+	<xacro:property name="omni_front_z" value="0.0265" />
 	<!-- Flag to select the high or low quality model -->
 	<xacro:property name="hq" value="true" />
@@ -48,4 +48,5 @@
 	</xacro:rubber_wheel>
 	<!-- OMNI WHEELS -->
+	<!-- -->
 	<xacro:omni_wheel name="omni_back" parent="base_link" hq="${hq}">
 		<origin xyz="-${omni_back_x} ${omni_back_y} ${omni_back_z}" rpy="0 0 0"/>
@@ -57,4 +58,5 @@
 		<origin xyz="${omni_front_x} -${omni_front_y} ${omni_front_z}" rpy="0 0 0"/>
 	</xacro:omni_wheel>
+	<!-- -->
 	<!-- SENSORS -->
 	<!-- LASER -->

File: rb1_base_description/robots/rb1_base_v3.urdf.xacro (robot description, xacro)
@@ -24,12 +24,12 @@
 	<xacro:property name="wheel_offset_x" value="0.0" />    <!-- x,y,z in translation from base_link to the center of the wheel -->
 	<xacro:property name="wheel_offset_y" value="0.218" />
-	<xacro:property name="wheel_offset_z" value="0.0512" />
+	<xacro:property name="wheel_offset_z" value="0.051" />
 	<!-- FOR OMNI WHEEL -->
 	<xacro:property name="omni_back_x" value="0.195" />
 	<xacro:property name="omni_back_y" value="0.0" />
-	<xacro:property name="omni_back_z" value="0.0258" />
+	<xacro:property name="omni_back_z" value="0.0265" />
 	<xacro:property name="omni_front_x" value="0.132" />
 	<xacro:property name="omni_front_y" value="0.1535" />
-	<xacro:property name="omni_front_z" value="0.0258" />
+	<xacro:property name="omni_front_z" value="0.0265" />
 	<!-- Flag to select the high or low quality model -->
 	<xacro:property name="hq" value="true" />

File: rb1_base_description/urdf/wheels/omni_wheel.urdf.xacro (robot description, xacro)
@@ -29,5 +29,5 @@
           <origin xyz="0 0 0" rpy="0 0 0" />
           <geometry>
-				<mesh filename="package://rb1_base_description/meshes/wheels/rb1v3_omniwheel.dae" />
+				<mesh filename="package://rb1_base_description/meshes/wheels/rb1v2_omniwheel.dae" />
           </geometry>
         </xacro:if>

File: rb1_base_description/urdf/wheels/rubber_wheel.urdf.xacro (robot description, xacro)
@@ -30,8 +30,8 @@
 			<geometry>
 				<xacro:if value="${reflect}">
-					<mesh filename="package://rb1_base_description/meshes/wheels/rb1v3_rubberwheel_6inch.dae" />
+					<mesh filename="package://rb1_base_description/meshes/wheels/wheel_rubber_6inch.dae" />
 				</xacro:if>
 				<xacro:unless value="${reflect}">
-					<mesh filename="package://rb1_base_description/meshes/wheels/rb1v3_rubberwheel_6inch.dae" />
+					<mesh filename="package://rb1_base_description/meshes/wheels/wheel_rubber_6inch.dae" />
 				</xacro:unless>
 			</geometry>
