Commit message: rb1_base_description: updated xacro to remove warning

File: rb1_base_description/robots/rb1_base_platform_v3.urdf.xacro (robot description, xacro)
@@ -37,6 +37,4 @@
 	<!-- Gazebo ros control plugins -->
 	<xacro:ros_control/>
-	<!-- Gazebo skid steering plugins -->
-	<xacro:diff_drive/>
 	<!-- WHEELS -->
 	<xacro:rubber_wheel name="right" parent="base_link" reflect="false" hq="${hq}">

File: rb1_base_description/urdf/elevator/elevator.urdf.xacro (robot description, xacro)
@@ -10,5 +10,5 @@
 		<parent link="${parent}"/>
 		<child link="elevator_base_link"/>
-		<insert_block name="origin" />
+		<xacro:insert_block name="origin" />
 	</joint>
 	<link name="elevator_base_link">

File: rb1_base_description/urdf/others/kinova_base.urdf.xacro (robot description, xacro)
@@ -8,5 +8,5 @@
       <parent link="${parent}"/>
       <child link="${prefix}kinova_base_link"/>
-      <insert_block name="origin" />
+      <xacro:insert_block name="origin" />
       <axis xyz="0 0 1" rpy="0 0 0" />
     </joint>

File: rb1_base_description/urdf/wheels/omni_wheel.urdf.xacro (robot description, xacro)
@@ -3,7 +3,7 @@
   <xacro:property name="M_PI" value="3.1415926535897931" />
   <!-- Wheels -->
-  <property name="omni_wheel_radius" value="0.051" />
-  <property name="omni_wheel_height" value="0.040" />
-  <property name="omni_wheel_mass" value="0.3" /> <!-- in kg-->
+  <xacro:property name="omni_wheel_radius" value="0.051" />
+  <xacro:property name="omni_wheel_height" value="0.040" />
+  <xacro:property name="omni_wheel_mass" value="0.3" /> <!-- in kg-->
   <xacro:macro name="cylinder_inertia" params="m r h">
     <inertia  ixx="${m*(3*r*r+h*h)/12}" ixy = "0" ixz = "0"
@@ -18,5 +18,5 @@
       <parent link="${parent}"/>
       <child link="${name}_wheel"/>
-      <insert_block name="origin" />
+      <xacro:insert_block name="origin" />
       <axis xyz="0 1 0" rpy="0 0 0" />
       <limit effort="100" velocity="100"/>

File: rb1_base_description/urdf/wheels/rubber_wheel.urdf.xacro (robot description, xacro)
@@ -5,7 +5,7 @@
 	<xacro:property name="M_PI" value="3.1415926535897931" />
 	<!-- Wheels -->
-	<property name="wheel_radius" value="0.076" />
-	<property name="wheel_height" value="0.025" />
-	<property name="wheel_mass" value="1.0" /> <!-- in kg-->
+	<xacro:property name="wheel_radius" value="0.076" />
+	<xacro:property name="wheel_height" value="0.025" />
+	<xacro:property name="wheel_mass" value="1.0" /> <!-- in kg-->
 	<xacro:macro name="cylinder_inertia" params="m r h">
 		<inertia	ixx="${m*(3*r*r+h*h)/12}" ixy = "0" ixz = "0"
@@ -18,5 +18,5 @@
 		<parent link="${parent}"/>
 		<child link="${name}_wheel_link"/>
-		<insert_block name="origin" />
+		<xacro:insert_block name="origin" />
 		<axis xyz="0 1 0" rpy="0 0 0" />
 		<limit effort="100" velocity="100"/>
