Commit message: [rb1_base_description]: xacro files modififed to multirobot

File: rb1_base_description/robots/rb1_base_platform_standalone_multi.urdf.xacro (robot description, xacro)
@@ -6,14 +6,8 @@
    <!-- ***************** -->
    <!-- First we import all posible elements defined in the urdf.xacro files. All these elements are defined as macro:xacros -->
+   <!-- gazebo elements -->
+   <xacro:include filename="$(find rb1_base_description)/urdf/common.gazebo.xacro" />
    <!-- Import RB1 base elements -->
    <xacro:include filename="$(find rb1_base_description)/urdf/bases/rb1_base.urdf.xacro" />
-   <gazebo>
-      <plugin name="ros_control" filename="libgazebo_ros_control.so">
-        <!-- robotNamespace>/rb1</robotNamespace -->
-        <robotParam>robot_description</robotParam>
-        <controlPeriod>0.001</controlPeriod>
-	    <robotSimType>gazebo_ros_control/DefaultRobotHWSim</robotSimType>
-      </plugin>
-   </gazebo>
    <!-- Import RB1 wheels -->
    <xacro:include filename="$(find rb1_base_description)/urdf/wheels/rubber_wheel.urdf.xacro" />
@@ -38,4 +32,6 @@
 	<!-- Flag to select the high or low quality model -->
 	<xacro:property name="hq" value="true" />
+	<xacro:arg name="prefix_topic" default=""/>
+	<xacro:arg name="prefix_frame" default="rb1_"/>
 	<!-- *************** -->
 	<!-- Robots Elements -->
@@ -43,24 +39,25 @@
 	<!-- Here we create the robot elements using the xacro:macros imported at the beggining of this file -->
 	<!-- RB-1 base -->
-	<xacro:rb1_base name="rb1_base" publish_bf="true" hq="${hq}" />
-	<!-- Gazebo ros control plugins -->
-	<xacro:ros_control/>
+	<xacro:rb1_base prefix_frame="$(arg prefix_frame)" publish_bf="true" hq="${hq}" />
+	<!-- Gazebo ros control pluggins -->
+	<xacro:ros_control prefix_topic="$(arg prefix_topic)" prefix_frame="$(arg prefix_frame)"/>
+	<xacro:gazebo_colors prefix_topic="$(arg prefix_topic)" prefix_frame="$(arg prefix_frame)"/>
 	<!-- Gazebo skid steering plugins -->
 	<!-- xacro:diff_drive/ -->
 	<!-- WHEELS -->
-	<xacro:rubber_wheel name="right" parent="base_link" reflect="false" hq="${hq}">
+	<xacro:rubber_wheel name="$(arg prefix_frame)right" parent="$(arg prefix_frame)base_link" reflect="false" hq="${hq}">
 		<origin xyz="${wheel_offset_x} -${wheel_offset_y} ${wheel_offset_z}" rpy="0 0 0"/>
 	</xacro:rubber_wheel>
-	<xacro:rubber_wheel name="left" parent="base_link" reflect="true" hq="${hq}">
+	<xacro:rubber_wheel name="$(arg prefix_frame)left" parent="$(arg prefix_frame)base_link" reflect="true" hq="${hq}">
 		<origin xyz="${wheel_offset_x} ${wheel_offset_y} ${wheel_offset_z}" rpy="0 0 0"/>
 	</xacro:rubber_wheel>
     <!-- OMNI DIRECTIONAL WHEELS -->
-	<xacro:omni_wheel name="omni_back" parent="base_link" hq="${hq}">
+	<xacro:omni_wheel name="$(arg prefix_frame)omni_back" parent="$(arg prefix_frame)base_link" hq="${hq}">
 		<origin xyz="-${omni_back_x} ${omni_back_y} ${omni_back_z}" rpy="0 0 0"/>
 	</xacro:omni_wheel>
-	<xacro:omni_wheel name="omni_front_left" parent="base_link" hq="${hq}">
+	<xacro:omni_wheel name="$(arg prefix_frame)omni_front_left" parent="$(arg prefix_frame)base_link" hq="${hq}">
 		<origin xyz="${omni_front_x} ${omni_front_y} ${omni_front_z}" rpy="0 0 0"/>
 	</xacro:omni_wheel>
-	<xacro:omni_wheel name="omni_front_right" parent="base_link" hq="${hq}">
+	<xacro:omni_wheel name="$(arg prefix_frame)omni_front_right" parent="$(arg prefix_frame)base_link" hq="${hq}">
 		<origin xyz="${omni_front_x} -${omni_front_y} ${omni_front_z}" rpy="0 0 0"/>
 	</xacro:omni_wheel>
@@ -75,8 +72,8 @@
 		<origin xyz="0.223 0.0 0.159" rpy="0 0 0"/>
 	</xacro:sensor_hokuyo_ust10lx -->
-	<xacro:sensor_hokuyo_ust10lx name="hokuyo" parent="base_link">
+	<xacro:sensor_hokuyo_ust10lx name="hokuyo" prefix_frame="$(arg prefix_frame)" prefix_topic="$(arg prefix_topic)" parent="$(arg prefix_frame)base_link">
 		<origin xyz="0.223 0.0 0.159" rpy="0 3.1416 3.1416"/>
 	</xacro:sensor_hokuyo_ust10lx>
-	<xacro:sensor_imu name="imu" parent="base_link">
+	<xacro:sensor_imu name="imu" prefix_frame="$(arg prefix_frame)" prefix_topic="$(arg prefix_topic)" parent="$(arg prefix_frame)base_link">
 		<origin xyz="-0.18 0.0 0.170" rpy="0 0 0"/>
 	</xacro:sensor_imu>
@@ -84,5 +81,5 @@
         <origin xyz="0.234 0.0125 0.107" rpy="0 0 0"/>
     </xacro:sensor_orbbec_astra -->
-    <xacro:sensor_orbbec_astra name="orbbec_astra" parent="base_link">
+    <xacro:sensor_orbbec_astra name="orbbec_astra" prefix_frame="$(arg prefix_frame)" prefix_topic="$(arg prefix_topic)" parent="$(arg prefix_frame)base_link">
         <origin xyz="0.234 0.0125 0.107" rpy="0 0 0"/>
     </xacro:sensor_orbbec_astra>

File: rb1_base_description/urdf/bases/rb1_base.gazebo.xacro (robot description, xacro)
@@ -1,4 +1,4 @@
 <?xml version="1.0"?>
-<robot xmlns:xacro="http://ros.org/wiki/xacro">
+<robot xmlns:xacro="http://www.ros.org/wiki/xacro">
 	<!-- DIFFERENCIAL DRIVE GAZEBO PLUGIN -->
 	<xacro:macro name="gazebo_differencial_drive">
@@ -7,6 +7,6 @@
 				<!--alwaysOn>true</alwaysOn-->
 				<updateRate>50.0</updateRate>
-				<leftJoint>left_wheel_joint</leftJoint>
-				<rightJoint>right_wheel_joint</rightJoint>
+				<leftJoint>$(prefix_frame)rb1_a_left_wheel_joint</leftJoint>
+				<rightJoint>$(prefix_frame)rb1_a_right_wheel_joint</rightJoint>
 				<!--leftJoint>joint_right_wheel</leftJoint>
 				<rightJoint>joint_left_wheel</rightJoint-->
@@ -17,6 +17,6 @@
 				<commandTopic>rb1/cmd_vel</commandTopic>
 				<odometryTopic>odom</odometryTopic>
-				<odometryFrame>odom</odometryFrame>
-				<robotBaseFrame>base_link</robotBaseFrame>
+				<odometryFrame>$(prefix_frame)odom</odometryFrame>
+				<robotBaseFrame>$(prefix_frame)base_link</robotBaseFrame>
 				<!-- robotNamespace></robotNamespace -->
 				<rosDebugLevel>na</rosDebugLevel>
@@ -32,4 +32,14 @@
 		</gazebo>
 	</xacro:macro>
+	<xacro:macro name="ros_control" params="prefix_frame prefix_topic">
+	   <gazebo>
+      <plugin name="ros_control" filename="libgazebo_ros_control.so">
+        <!--robotNamespace>/rb1</robotNamespace-->
+        <robotParam>robot_description</robotParam>
+        <controlPeriod>0.001</controlPeriod>
+	    <robotSimType>gazebo_ros_control/DefaultRobotHWSim</robotSimType>
+      </plugin>
+   </gazebo>
+   </xacro:macro>
 	<gazebo reference="base_footprint">
 		<material>Gazebo/Green</material>

File: rb1_base_description/urdf/bases/rb1_base.urdf.xacro (robot description, xacro)
@@ -1,5 +1,5 @@
 <?xml version="1.0"?>
 <robot name="rb1_base" xmlns:xacro="http://www.ros.org/wiki/xacro">
-  <xacro:macro name="rb1_base" params="name publish_bf hq">
+  <xacro:macro name="rb1_base" params="prefix_frame publish_bf hq">
   <!-- Robot mechanical and motor parameters -->
   <xacro:property name="PI" value="3.1415926535897931"/>
@@ -7,5 +7,5 @@
   <!-- BASE FOOTPRINT -->
   <xacro:if value="${publish_bf}">
-    <link name="base_footprint">
+    <link name="${prefix_frame}base_footprint">
       <visual>
           <origin xyz="0 0 0" rpy="0 0 0" />
@@ -17,10 +17,10 @@
     <joint name="base_footprint_joint" type="fixed">
        <origin xyz="0 0 ${wheel_radius - wheel_offset_z}" rpy="0 0 0" />
-      <parent link="base_footprint"/>
-      <child link="base_link" />
+      <parent link="${prefix_frame}base_footprint"/>
+      <child link="${prefix_frame}base_link" />
     </joint>
   </xacro:if>
   <!-- BASE_LINK -->
-  <link name="base_link">
+  <link name="${prefix_frame}base_link">
     <inertial>
       <mass value="25.0" />
@@ -53,9 +53,9 @@
   <joint name="front_cover_joint" type="fixed">
      <origin xyz="0.220 0.0 0.004" rpy="0 0 0 " />
-     <parent link="base_link"/>
-     <child link="front_cover_link" />
+     <parent link="${prefix_frame}base_link"/>
+     <child link="${prefix_frame}front_cover_link" />
   </joint>
   <!-- FRONT COVER -->
-  <link name="front_cover_link">
+  <link name="${prefix_frame}front_cover_link">
     <inertial>
       <mass value="0.25" />
@@ -89,9 +89,9 @@
   <joint name="base_docking_joint" type="fixed">
      <origin xyz="0.030 0.000 0.068" rpy="0 0 0 " />
-     <parent link="front_cover_link"/>
-     <child link="base_docking_contact" />
+     <parent link="${prefix_frame}front_cover_link"/>
+     <child link="${prefix_frame}base_docking_contact" />
   </joint>
   <!-- FRONT COVER -->
-  <link name="base_docking_contact" />
+  <link name="${prefix_frame}base_docking_contact" />
   </xacro:macro>
 </robot>

File: rb1_base_description/urdf/bases/rb1_base_v2.urdf.xacro (robot description, xacro)
@@ -1,5 +1,5 @@
 <?xml version="1.0"?>
 <robot name="rb1_base" xmlns:xacro="http://www.ros.org/wiki/xacro">
-  <xacro:macro name="rb1_base" params="name publish_bf hq">
+  <xacro:macro name="rb1_base_v2" params="prefix_frame publish_bf hq">
   <!-- Robot mechanical and motor parameters -->
   <xacro:property name="PI" value="3.1415926535897931"/>
@@ -7,5 +7,5 @@
   <!-- BASE FOOTPRINT -->
   <xacro:if value="${publish_bf}">
-    <link name="base_footprint">
+    <link name="${prefix_frame}base_footprint">
       <visual>
           <origin xyz="0 0 0" rpy="0 0 0" />
@@ -17,10 +17,10 @@
     <joint name="base_footprint_joint" type="fixed">
        <origin xyz="0 0 ${wheel_radius - wheel_offset_z}" rpy="0 0 0" />
-      <parent link="base_footprint"/>
-      <child link="base_link" />
+      <parent link="${prefix_frame}base_footprint"/>
+      <child link="${prefix_frame}base_link" />
     </joint>
   </xacro:if>
   <!-- BASE_LINK -->
-  <link name="base_link">
+  <link name="${prefix_frame}base_link">
     <inertial>
       <mass value="25.0" />
@@ -53,9 +53,9 @@
   <joint name="front_cover_joint" type="fixed">
      <origin xyz="0.220 0.0 0.004" rpy="0 0 0 " />
-     <parent link="base_link"/>
-     <child link="front_cover_link" />
+     <parent link="${prefix_frame}base_link"/>
+     <child link="${prefix_frame}front_cover_link" />
   </joint>
   <!-- FRONT COVER -->
-  <link name="front_cover_link">
+  <link name="${prefix_frame}front_cover_link">
     <inertial>
       <mass value="0.25" />
@@ -89,9 +89,9 @@
   <joint name="base_docking_joint" type="fixed">
      <origin xyz="0.030 0.000 0.068" rpy="0 0 0 " />
-     <parent link="front_cover_link"/>
-     <child link="base_docking_contact" />
+     <parent link="${prefix_frame}front_cover_link"/>
+     <child link="${prefix_frame}base_docking_contact_link" />
   </joint>
   <!-- DOCKING LINK -->
-  <link name="base_docking_contact" />
+  <link name="${prefix_frame}base_docking_contact_link" />
   </xacro:macro>
 </robot>

File: rb1_base_description/urdf/bases/rb1_base_v3.urdf.xacro (robot description, xacro)
@@ -1,5 +1,5 @@
 <?xml version="1.0"?>
 <robot name="rb1_base" xmlns:xacro="http://www.ros.org/wiki/xacro">
-  <xacro:macro name="rb1_base" params="name publish_bf hq">
+  <xacro:macro name="rb1_base_v3" params="prefix_frame publish_bf hq">
   <!-- Robot mechanical and motor parameters -->
   <xacro:property name="PI" value="3.1415926535897931"/>
@@ -7,5 +7,5 @@
   <!-- BASE FOOTPRINT -->
   <xacro:if value="${publish_bf}">
-    <link name="base_footprint">
+    <link name="${prefix_frame}base_footprint">
       <visual>
           <origin xyz="0 0 0" rpy="0 0 0" />
@@ -17,10 +17,10 @@
     <joint name="base_footprint_joint" type="fixed">
        <origin xyz="0 0 ${wheel_radius - wheel_offset_z}" rpy="0 0 0" />
-      <parent link="base_footprint"/>
-      <child link="base_link" />
+      <parent link="${prefix_frame}base_footprint"/>
+      <child link="${prefix_frame}base_link" />
     </joint>
   </xacro:if>
   <!-- BASE_LINK -->
-  <link name="base_link">
+  <link name="${prefix_frame}base_link">
     <inertial>
       <mass value="25.0" />
@@ -53,9 +53,9 @@
   <joint name="front_cover_joint" type="fixed">
      <origin xyz="0.220 0.0 0.004" rpy="0 0 0 " />
-     <parent link="base_link"/>
-     <child link="front_cover_link" />
+     <parent link="${prefix_frame}base_link"/>
+     <child link="${prefix_frame}front_cover_link" />
   </joint>
   <!-- FRONT COVER -->
-  <link name="front_cover_link">
+  <link name="${prefix_frame}front_cover_link">
     <inertial>
       <mass value="0.25" />
@@ -88,9 +88,9 @@
   <joint name="top_covert_joint" type="fixed">
      <origin xyz="0.0 0.0 0.243" rpy="0 0 0 " />
-     <parent link="base_footprint"/>
-     <child link="top_cover_link" />
+     <parent link="${prefix_frame}base_footprint"/>
+     <child link="${prefix_frame}top_cover_link" />
   </joint>
   <!-- FRONT COVER -->
-  <link name="top_cover_link">
+  <link name="${prefix_frame}top_cover_link">
     <inertial>
       <mass value="0.25" />
@@ -124,9 +124,9 @@
   <joint name="base_docking_joint" type="fixed">
      <origin xyz="0.030 0.000 0.068" rpy="0 0 0 " />
-     <parent link="front_cover_link"/>
-     <child link="base_docking_contact" />
+     <parent link="${prefix_frame}front_cover_link"/>
+     <child link="${prefix_frame}base_docking_contact_link" />
   </joint>
   <!-- DOCKING LINK -->
-  <link name="base_docking_contact" />
+  <link name="${prefix_frame}base_docking_contact_link" />
   </xacro:macro>
 </robot>

File: rb1_base_description/urdf/common.gazebo.xacro (robot description, xacro)
@@ -2,12 +2,23 @@
 <robot xmlns:xacro="http://www.ros.org/wiki/xacro">
 <!-- ROS CONTROL GAZEBO PLUGIN -->
-	<xacro:macro name="ros_control">
-		<gazebo>
-			<plugin name="ros_control" filename="libgazebo_ros_control.so">
-				<robotNamespace>/</robotNamespace	>
-				<!--robotParam>robot_description</robotParam-->
-				<!--controlPeriod>0.001</controlPeriod-->
-				<robotSimType>gazebo_ros_control/DefaultRobotHWSim</robotSimType>
-			</plugin>
+	<xacro:macro name="ros_control" params="prefix_frame prefix_topic">
+	   <gazebo>
+      <plugin name="ros_control" filename="libgazebo_ros_control.so">
+        <!--robotNamespace>/rb1</robotNamespace-->
+        <robotParam>robot_description</robotParam>
+        <controlPeriod>0.001</controlPeriod>
+	    <robotSimType>gazebo_ros_control/DefaultRobotHWSim</robotSimType>
+      </plugin>
+   </gazebo>
+   </xacro:macro>
+   <xacro:macro name="gazebo_colors" params="prefix_frame prefix_topic">
+		<gazebo reference="$(arg prefix_frame)base_footprint">
+			<material>Gazebo/Green</material>
+		</gazebo>
+		<gazebo reference="$(arg prefix_frame)base_link">
+			<material>Gazebo/Grey</material>
+		</gazebo>
+		<gazebo reference="$(arg prefix_frame)front_cover_link">
+			<material>Gazebo/Black</material>
 		</gazebo>
 	</xacro:macro>

File: rb1_base_description/urdf/elevator/elevator.urdf.xacro (robot description, xacro)
@@ -2,15 +2,15 @@
 <robot xmlns:xacro="http://www.ros.org/wiki/xacro">
 	<!--xacro:include filename="$(find rb1_base_description)/urdf/bases/rb1_elevator.gazebo.xacro" /-->
-	<xacro:macro name="elevator_platform" params="parent hq *origin">
+	<xacro:macro name="elevator_platform" params="name parent hq *origin">
 	<!-- PARAMS: -->
 	<!-- name : name of the link: -->
 	<!-- hq: selects model in high quality (.dae) -->
 	<!-- ELEVATOR_BASE_LINK -->
-	<joint name="elevator_base_joint" type="fixed">
+	<joint name="${name}_base_joint" type="fixed">
 		<parent link="${parent}"/>
-		<child link="elevator_base_link"/>
+		<child link="${name}_base_link"/>
 		<xacro:insert_block name="origin" />
 	</joint>
-	<link name="elevator_base_link">
+	<link name="${name}_base_link">
 		<!--inertial>
 			<mass value="25.0" />
@@ -44,12 +44,12 @@
 	</link>
 	<!-- ELEVATOR PLATFORM -->
-	<joint name="elevator_platform_joint" type="prismatic">
+	<joint name="${name}_platform_joint" type="prismatic">
 			<origin xyz="0.0 0.0 0.041" rpy="0 0 0 " />
-			<parent link="elevator_base_link"/>
-			<child link="elevator_platform_link" />
+			<parent link="${name}_base_link"/>
+			<child link="${name}_platform_link" />
 			<axis xyz="0 0 1"/>
 			<limit effort="1.0" lower="0.0" upper="0.034" velocity="0.5"/>
 	</joint>
-	<link name="elevator_platform_link">
+	<link name="${name}_platform_link">
 		<!--inertial>
 			<mass value="0.25" />

File: rb1_base_description/urdf/wheels/rubber_wheel.gazebo.xacro (robot description, xacro)
@@ -1,4 +1,4 @@
 <?xml version="1.0"?>
-<robot xmlns:xacro="http://ros.org/wiki/xacro">
+<robot xmlns:xacro="http://www.ros.org/wiki/xacro">
 	<xacro:macro name="rubber_wheel_gazebo" params="name">
 		<gazebo reference="${name}_wheel_link">

File: rb1_base_description/urdf/wheels/rubber_wheel.transmission.xacro (robot description, xacro)
@@ -1,4 +1,4 @@
 <?xml version="1.0"?>
-<robot xmlns:xacro="http://ros.org/wiki/xacro">
+<robot xmlns:xacro="http://www.ros.org/wiki/xacro">
 	<!-- Rubber wheel transmission -->
 	<xacro:macro name="rubber_wheel_transmission" params="name">
@@ -10,5 +10,5 @@
 				<!--hardwareInterface>EffortJointInterface</hardwareInterface-->
 				<!-- for ros control controller -->
-				<hardwareInterface>VelocityJointInterface</hardwareInterface>
+				<hardwareInterface>hardware_interface/VelocityJointInterface</hardwareInterface>
 			</joint>
 			<actuator name="${name}_wheel_joint_motor">
