Commit message: [rb1_base_description]:xacros updated to multirobot

File: rb1_base_description/robots/rb1_base_platform_standalone_multi.urdf.xacro (robot description, xacro)
@@ -32,6 +32,5 @@
 	<!-- Flag to select the high or low quality model -->
 	<xacro:property name="hq" value="true" />
-	<xacro:arg name="prefix_topic" default=""/>
-	<xacro:arg name="prefix_frame" default="rb1_"/>
+	<xacro:arg name="prefix" default="rb1_"/>
 	<!-- *************** -->
 	<!-- Robots Elements -->
@@ -39,25 +38,25 @@
 	<!-- Here we create the robot elements using the xacro:macros imported at the beggining of this file -->
 	<!-- RB-1 base -->
-	<xacro:rb1_base prefix_frame="$(arg prefix_frame)" publish_bf="true" hq="${hq}" />
+	<xacro:rb1_base prefix="$(arg prefix)" publish_bf="true" hq="${hq}" />
 	<!-- Gazebo ros control pluggins -->
-	<xacro:ros_control prefix_topic="$(arg prefix_topic)" prefix_frame="$(arg prefix_frame)"/>
-	<xacro:gazebo_colors prefix_topic="$(arg prefix_topic)" prefix_frame="$(arg prefix_frame)"/>
+	<xacro:ros_control/>
+	<xacro:gazebo_colors prefix="$(arg prefix)"/>
 	<!-- Gazebo skid steering plugins -->
 	<!-- xacro:diff_drive/ -->
-	<!-- WHEELS -->
-	<xacro:rubber_wheel name="$(arg prefix_frame)right" parent="$(arg prefix_frame)base_link" reflect="false" hq="${hq}">
+    <!-- WHEELS -->
+	<xacro:rubber_wheel prefix="$(arg prefix)right" parent="$(arg prefix)base_link" reflect="false" hq="${hq}">
 		<origin xyz="${wheel_offset_x} -${wheel_offset_y} ${wheel_offset_z}" rpy="0 0 0"/>
 	</xacro:rubber_wheel>
-	<xacro:rubber_wheel name="$(arg prefix_frame)left" parent="$(arg prefix_frame)base_link" reflect="true" hq="${hq}">
+	<xacro:rubber_wheel prefix="$(arg prefix)left" parent="$(arg prefix)base_link" reflect="true" hq="${hq}">
 		<origin xyz="${wheel_offset_x} ${wheel_offset_y} ${wheel_offset_z}" rpy="0 0 0"/>
 	</xacro:rubber_wheel>
     <!-- OMNI DIRECTIONAL WHEELS -->
-	<xacro:omni_wheel name="$(arg prefix_frame)omni_back" parent="$(arg prefix_frame)base_link" hq="${hq}">
+	<xacro:omni_wheel prefix="$(arg prefix)omni_back" parent="$(arg prefix)base_link" hq="${hq}">
 		<origin xyz="-${omni_back_x} ${omni_back_y} ${omni_back_z}" rpy="0 0 0"/>
 	</xacro:omni_wheel>
-	<xacro:omni_wheel name="$(arg prefix_frame)omni_front_left" parent="$(arg prefix_frame)base_link" hq="${hq}">
+	<xacro:omni_wheel prefix="$(arg prefix)omni_front_left" parent="$(arg prefix)base_link" hq="${hq}">
 		<origin xyz="${omni_front_x} ${omni_front_y} ${omni_front_z}" rpy="0 0 0"/>
 	</xacro:omni_wheel>
-	<xacro:omni_wheel name="$(arg prefix_frame)omni_front_right" parent="$(arg prefix_frame)base_link" hq="${hq}">
+	<xacro:omni_wheel prefix="$(arg prefix)omni_front_right" parent="$(arg prefix)base_link" hq="${hq}">
 		<origin xyz="${omni_front_x} -${omni_front_y} ${omni_front_z}" rpy="0 0 0"/>
 	</xacro:omni_wheel>
@@ -72,8 +71,8 @@
 		<origin xyz="0.223 0.0 0.159" rpy="0 0 0"/>
 	</xacro:sensor_hokuyo_ust10lx -->
-	<xacro:sensor_hokuyo_ust10lx name="hokuyo" prefix_frame="$(arg prefix_frame)" prefix_topic="$(arg prefix_topic)" parent="$(arg prefix_frame)base_link">
+	<xacro:sensor_hokuyo_ust10lx prefix="$(arg prefix)hokuyo" parent="$(arg prefix)base_link">
 		<origin xyz="0.223 0.0 0.159" rpy="0 3.1416 3.1416"/>
 	</xacro:sensor_hokuyo_ust10lx>
-	<xacro:sensor_imu name="imu" prefix_frame="$(arg prefix_frame)" prefix_topic="$(arg prefix_topic)" parent="$(arg prefix_frame)base_link">
+	<xacro:sensor_imu prefix="$(arg prefix)imu" parent="$(arg prefix)base_link">
 		<origin xyz="-0.18 0.0 0.170" rpy="0 0 0"/>
 	</xacro:sensor_imu>
@@ -81,5 +80,5 @@
         <origin xyz="0.234 0.0125 0.107" rpy="0 0 0"/>
     </xacro:sensor_orbbec_astra -->
-    <xacro:sensor_orbbec_astra name="orbbec_astra" prefix_frame="$(arg prefix_frame)" prefix_topic="$(arg prefix_topic)" parent="$(arg prefix_frame)base_link">
+    <xacro:sensor_orbbec_astra prefix="$(arg prefix)orbbec_astra" parent="$(arg prefix)base_link">
         <origin xyz="0.234 0.0125 0.107" rpy="0 0 0"/>
     </xacro:sensor_orbbec_astra>

File: rb1_base_description/robots/rb1_base_platform_v3_multi.urdf.xacro (robot description, xacro)
@@ -36,35 +36,34 @@
 	<!-- Here we create the robot elements using the xacro:macros imported at the beggining of this file -->
 	<!-- RB-1 base -->
-	<xacro:rb1_base prefix_frame="$(arg prefix_frame)" publish_bf="true" hq="${hq}" />
-	<xacro:arg name="prefix_topic" default=""/>
-	<xacro:arg name="prefix_frame" default="rb1_"/>
+	<xacro:rb1_base prefix="$(arg prefix)" publish_bf="true" hq="${hq}" />
+	<xacro:arg name="prefix" default="rb1_"/>
 	<!-- Gazebo ros control pluggins -->
-	<xacro:ros_control prefix_topic="$(arg prefix_topic)" prefix_frame="$(arg prefix_frame)"/>
-	<xacro:gazebo_colors prefix_topic="$(arg prefix_topic)" prefix_frame="$(arg prefix_frame)"/>
+	<xacro:ros_control/>
+	<xacro:gazebo_colors prefix="$(arg prefix)"/>
 	<!-- WHEELS -->
-	<xacro:rubber_wheel name="$(arg prefix_frame)right" parent="$(arg prefix_frame)base_link" reflect="false" hq="${hq}">
+	<xacro:rubber_wheel prefix="$(arg prefix)right" parent="$(arg prefix)base_link" reflect="false" hq="${hq}">
 		<origin xyz="${wheel_offset_x} -${wheel_offset_y} ${wheel_offset_z}" rpy="0 0 0"/>
 	</xacro:rubber_wheel>
-	<xacro:rubber_wheel name="$(arg prefix_frame)left" parent="$(arg prefix_frame)base_link" reflect="true" hq="${hq}">
+	<xacro:rubber_wheel prefix="$(arg prefix)left" parent="$(arg prefix)base_link" reflect="true" hq="${hq}">
 		<origin xyz="${wheel_offset_x} ${wheel_offset_y} ${wheel_offset_z}" rpy="0 0 0"/>
 	</xacro:rubber_wheel>
     <!-- OMNI DIRECTIONAL WHEELS -->
-	<xacro:omni_wheel name="$(arg prefix_frame)omni_back" parent="$(arg prefix_frame)base_link" hq="${hq}">
+	<xacro:omni_wheel prefix="$(arg prefix)omni_back" parent="$(arg prefix)base_link" hq="${hq}">
 		<origin xyz="-${omni_back_x} ${omni_back_y} ${omni_back_z}" rpy="0 0 0"/>
 	</xacro:omni_wheel>
-	<xacro:omni_wheel name="$(arg prefix_frame)omni_front_left" parent="$(arg prefix_frame)base_link" hq="${hq}">
+	<xacro:omni_wheel prefix="$(arg prefix)omni_front_left" parent="$(arg prefix)base_link" hq="${hq}">
 		<origin xyz="${omni_front_x} ${omni_front_y} ${omni_front_z}" rpy="0 0 0"/>
 	</xacro:omni_wheel>
-	<xacro:omni_wheel name="$(arg prefix_frame)omni_front_right" parent="$(arg prefix_frame)base_link" hq="${hq}">
+	<xacro:omni_wheel prefix="$(arg prefix)omni_front_right" parent="$(arg prefix)base_link" hq="${hq}">
 		<origin xyz="${omni_front_x} -${omni_front_y} ${omni_front_z}" rpy="0 0 0"/>
 	</xacro:omni_wheel>
 	<!-- SENSORS -->
-	<xacro:sensor_sick_tim551 name="laser_sick" prefix_frame="$(arg prefix_frame)" prefix_topic="$(arg prefix_topic)" parent="$(arg prefix_frame)base_link">
+	<xacro:sensor_sick_tim551 prefix="$(arg prefix)laser_sick" parent="$(arg prefix)base_link">
 		<origin xyz="0.220 0.0 0.1686" rpy="0 3.1416 3.1416"/>
 	</xacro:sensor_sick_tim551>
-	<xacro:sensor_imu name="imu" prefix_frame="$(arg prefix_frame)" prefix_topic="$(arg prefix_topic)" parent="$(arg prefix_frame)base_link">
+	<xacro:sensor_imu prefix="$(arg prefix)imu" parent="$(arg prefix)base_link">
 		<origin xyz="0.002 0.053 0.1485" rpy="0 0 0"/>
 	</xacro:sensor_imu>
-    <xacro:sensor_orbbec_astra name="orbbec_astra" prefix_frame="$(arg prefix_frame)" prefix_topic="$(arg prefix_topic)" parent="$(arg prefix_frame)base_link">
+    <xacro:sensor_orbbec_astra prefix="$(arg prefix)orbbec_astra" parent="$(arg prefix)base_link">
         <origin xyz="0.234 0.0125 0.107" rpy="0 0 0"/>
     </xacro:sensor_orbbec_astra>

File: rb1_base_description/robots/rb1_base_v2_elevator_multi.urdf.xacro (robot description, xacro)
@@ -45,55 +45,54 @@
 	<!-- ROBOT COMPONENTS -->
 	<!-- *************** -->
-	<xacro:arg name="prefix_topic" default=""/>
-	<xacro:arg name="prefix_frame" default="rb1_"/>
+	<xacro:arg name="prefix" default="rb1_"/>
 	<!-- Here we create the robot elements using the xacro:macros imported at the beggining of this file -->
 	<!-- BASE -->
-	<xacro:rb1_base_v2 prefix_frame="$(arg prefix_frame)" publish_bf="true" hq="${hq}" />
+	<xacro:rb1_base_v2 prefix="$(arg prefix)" publish_bf="true" hq="${hq}" />
 	<!-- WHEELS -->
-	<xacro:rubber_wheel name="$(arg prefix_frame)right" parent="$(arg prefix_frame)base_link" reflect="false" hq="${hq}">
+	<xacro:rubber_wheel prefix="$(arg prefix)right" parent="$(arg prefix)base_link" reflect="false" hq="${hq}">
 		<origin xyz="${wheel_offset_x} -${wheel_offset_y} ${wheel_offset_z}" rpy="0 0 0"/>
 	</xacro:rubber_wheel>
-	<xacro:rubber_wheel name="$(arg prefix_frame)left" parent="$(arg prefix_frame)base_link" reflect="true" hq="${hq}">
+	<xacro:rubber_wheel prefix="$(arg prefix)left" parent="$(arg prefix)base_link" reflect="true" hq="${hq}">
 		<origin xyz="${wheel_offset_x} ${wheel_offset_y} ${wheel_offset_z}" rpy="0 0 0"/>
 	</xacro:rubber_wheel>
     <!-- OMNI DIRECTIONAL WHEELS -->
-	<xacro:omni_wheel name="$(arg prefix_frame)omni_back" parent="$(arg prefix_frame)base_link" hq="${hq}">
+	<xacro:omni_wheel prefix="$(arg prefix)omni_back" parent="$(arg prefix)base_link" hq="${hq}">
 		<origin xyz="-${omni_back_x} ${omni_back_y} ${omni_back_z}" rpy="0 0 0"/>
 	</xacro:omni_wheel>
-	<xacro:omni_wheel name="$(arg prefix_frame)omni_front_left" parent="$(arg prefix_frame)base_link" hq="${hq}">
+	<xacro:omni_wheel prefix="$(arg prefix)omni_front_left" parent="$(arg prefix)base_link" hq="${hq}">
 		<origin xyz="${omni_front_x} ${omni_front_y} ${omni_front_z}" rpy="0 0 0"/>
 	</xacro:omni_wheel>
-	<xacro:omni_wheel name="$(arg prefix_frame)omni_front_right" parent="$(arg prefix_frame)base_link" hq="${hq}">
+	<xacro:omni_wheel prefix="$(arg prefix)omni_front_right" parent="$(arg prefix)base_link" hq="${hq}">
 		<origin xyz="${omni_front_x} -${omni_front_y} ${omni_front_z}" rpy="0 0 0"/>
 	</xacro:omni_wheel>
 	<!-- ELEVATOR_PLATFORM -->
-	<xacro:elevator_platform name="$(arg prefix_frame)elevator" parent="$(arg prefix_frame)base_link" hq="${hq}">
+	<xacro:elevator_platform prefix="$(arg prefix)elevator" parent="$(arg prefix)base_link" hq="${hq}">
 		<origin xyz="${elevator_x} -${elevator_y} ${elevator_z}" rpy="0 0 0"/>
 	</xacro:elevator_platform>
 	<!-- SENSORS -->
 	<!-- LASER -->
-	<!-- xacro:sensor_hokuyo_utm30lx name="front_laser" parent="base_link">
+	<!-- xacro:sensor_hokuyo_utm30lx prefix="$(arg prefix)front_laser" parent="$(arg prefix)base_link">
 		<origin xyz="0.210 0.0 0.305" rpy="0 0 0"/>
 	</xacro:sensor_hokuyo_utm30lx -->
-	<!-- xacro:sensor_hokuyo_urg04lx name="front_laser" parent="base_link">
+	<!-- xacro:sensor_hokuyo_urg04lx prefix="$(arg prefix)front_laser" parent="$(arg prefix)base_link">
 		<origin xyz="0.220 0.0 0.170" rpy="0 3.1416 3.1416"/>
 	</xacro:sensor_hokuyo_urg04lx -->
-	<!-- xacro:sensor_hokuyo_ust10lx name="front_laser" parent="base_link">
+	<!-- xacro:sensor_hokuyo_ust10lx prefix="$(arg prefix)front_laser" parent="$(arg prefix)base_link">
 		<origin xyz="0.223 0.0 0.159" rpy="0 0 0"/>
 	</xacro:sensor_hokuyo_ust10lx -->
 	<!-- Name the components as base_front_laser or base_laser or front_laser or
 	a name which identify uniquely the component within the robot -->
-	<xacro:sensor_rplidar_a2 name="base_front_laser" prefix_frame="$(arg prefix_frame)" prefix_topic="$(arg prefix_topic)" parent="$(arg prefix_frame)base_link">
+	<xacro:sensor_rplidar_a2 prefix="$(arg prefix)base_front_laser" parent="$(arg prefix)base_link">
 		<origin xyz="0.210 0.0 0.199" rpy="3.1415 0 0"/>
 	</xacro:sensor_rplidar_a2>
 	<!-- CAMERA -->
-	<!--xacro:sensor_orbbec_astra name="base_front_camera" parent="base_link">
+	<!--xacro:sensor_orbbec_astra prefix="$(arg prefix)base_front_camera" parent="$(arg prefix)base_link">
 		<origin xyz="0.234 0.0125 0.107" rpy="0 0 0"/>
 	</xacro:sensor_orbbec_astra-->
-	<!-- xacro:sensor_kinect name="front_camera" parent="base_link">
+	<!-- xacro:sensor_kinect prefix="$(arg prefix)front_camera" parent="$(arg prefix)base_link">
 		<origin xyz="0.6 0.0 0.102" rpy="0 0 0"/>
 	</xacro:sensor_kinect -->
 	<!-- IMU -->
-	<xacro:sensor_imu name="imu" prefix_frame="$(arg prefix_frame)" prefix_topic="$(arg prefix_topic)" parent="$(arg prefix_frame)base_link">
+	<xacro:sensor_imu prefix="$(arg prefix)imu" parent="$(arg prefix)base_link">
 		<origin xyz="-0.18 0.0 0.170" rpy="0 0 0"/>
 	</xacro:sensor_imu>
@@ -102,5 +101,5 @@
 	<!-- ************** -->
 	<!-- Gazebo ros control pluggins -->
-	<xacro:ros_control prefix_topic="$(arg prefix_topic)" prefix_frame="$(arg prefix_frame)"/>
-	<xacro:gazebo_colors prefix_topic="$(arg prefix_topic)" prefix_frame="$(arg prefix_frame)"/>
+	<xacro:ros_control/>
+	<xacro:gazebo_colors prefix="$(arg prefix)"/>
 </robot>

File: rb1_base_description/robots/rb1_base_v2_multi.urdf.xacro (robot description, xacro)
@@ -36,24 +36,23 @@
 	<!-- ROBOT COMPONENTS -->
 	<!-- *************** -->
-	<xacro:arg name="prefix_topic" default=""/>
-	<xacro:arg name="prefix_frame" default="rb1_"/>
+	<xacro:arg name="prefix" default="rb1_"/>
 	<!-- Here we create the robot elements using the xacro:macros imported at the beggining of this file -->
 	<!-- BASE -->
-	<xacro:rb1_base_v2 prefix_frame="$(arg prefix_frame)" publish_bf="true" hq="${hq}" />
+	<xacro:rb1_base_v2 prefix="$(arg prefix)" publish_bf="true" hq="${hq}" />
 	<!-- WHEELS -->
-	<xacro:rubber_wheel name="$(arg prefix_frame)right" parent="$(arg prefix_frame)base_link" reflect="false" hq="${hq}">
+	<xacro:rubber_wheel prefix="$(arg prefix)right" parent="$(arg prefix)base_link" reflect="false" hq="${hq}">
 		<origin xyz="${wheel_offset_x} -${wheel_offset_y} ${wheel_offset_z}" rpy="0 0 0"/>
 	</xacro:rubber_wheel>
-	<xacro:rubber_wheel name="$(arg prefix_frame)left" parent="$(arg prefix_frame)base_link" reflect="true" hq="${hq}">
+	<xacro:rubber_wheel prefix="$(arg prefix)left" parent="$(arg prefix)base_link" reflect="true" hq="${hq}">
 		<origin xyz="${wheel_offset_x} ${wheel_offset_y} ${wheel_offset_z}" rpy="0 0 0"/>
 	</xacro:rubber_wheel>
     <!-- OMNI DIRECTIONAL WHEELS -->
-	<xacro:omni_wheel name="$(arg prefix_frame)omni_back" parent="$(arg prefix_frame)base_link" hq="${hq}">
+	<xacro:omni_wheel prefix="$(arg prefix)omni_back" parent="$(arg prefix)base_link" hq="${hq}">
 		<origin xyz="-${omni_back_x} ${omni_back_y} ${omni_back_z}" rpy="0 0 0"/>
 	</xacro:omni_wheel>
-	<xacro:omni_wheel name="$(arg prefix_frame)omni_front_left" parent="$(arg prefix_frame)base_link" hq="${hq}">
+	<xacro:omni_wheel prefix="$(arg prefix)omni_front_left" parent="$(arg prefix)base_link" hq="${hq}">
 		<origin xyz="${omni_front_x} ${omni_front_y} ${omni_front_z}" rpy="0 0 0"/>
 	</xacro:omni_wheel>
-	<xacro:omni_wheel name="$(arg prefix_frame)omni_front_right" parent="$(arg prefix_frame)base_link" hq="${hq}">
+	<xacro:omni_wheel prefix="$(arg prefix)omni_front_right" parent="$(arg prefix)base_link" hq="${hq}">
 		<origin xyz="${omni_front_x} -${omni_front_y} ${omni_front_z}" rpy="0 0 0"/>
 	</xacro:omni_wheel>
@@ -61,27 +60,27 @@
 	<!-- SENSORS -->
 	<!-- LASER -->
-	<!-- xacro:sensor_hokuyo_utm30lx name="base_front_laser" parent="base_link">
+	<!-- xacro:sensor_hokuyo_utm30lx prefix="$(arg prefix)base_front_laser" parent="$(arg prefix)base_link">
 		<origin xyz="0.210 0.0 0.305" rpy="0 0 0"/>
 	</xacro:sensor_hokuyo_utm30lx -->
-	<!-- xacro:sensor_hokuyo_urg04lx name="base_front_laser" parent="base_link">
+	<!-- xacro:sensor_hokuyo_urg04lx prefix="$(arg prefix)base_front_laser" parent="$(arg prefix)base_link">
 		<origin xyz="0.220 0.0 0.170" rpy="0 3.1416 3.1416"/>
 	</xacro:sensor_hokuyo_urg04lx -->
-	<xacro:sensor_hokuyo_ust10lx name="hokuyo" prefix_frame="$(arg prefix_frame)" prefix_topic="$(arg prefix_topic)" parent="$(arg prefix_frame)base_link">
+	<xacro:sensor_hokuyo_ust10lx prefix="$(arg prefix)hokuyo" parent="$(arg prefix)base_link">
 		<origin xyz="0.223 0.0 0.159" rpy="3.1416 0 0"/>
 	</xacro:sensor_hokuyo_ust10lx>
 	<!-- Name the components as base_front_laser or base_laser or front_laser or
 	a name which identify uniquely the component within the robot -->
-	<!--xacro:sensor_rplidar_a2 name="base_front_laser" parent="base_link">
+	<!--xacro:sensor_rplidar_a2 prefix="$(arg prefix)base_front_laser" parent="$(arg prefix)base_link">
 		<origin xyz="0.210 0.0 0.199" rpy="3.1415 0 0"/>
 	</xacro:sensor_rplidar_a2-->
 	<!-- CAMERA -->
-	<xacro:sensor_orbbec_astra name="orbbec_astra" prefix_frame="$(arg prefix_frame)" prefix_topic="$(arg prefix_topic)" parent="$(arg prefix_frame)base_link">
+	<xacro:sensor_orbbec_astra prefix="$(arg prefix)orbbec_astra" parent="$(arg prefix)base_link">
 		<origin xyz="0.234 0.0125 0.107" rpy="0 0 0"/>
 	</xacro:sensor_orbbec_astra>
-	<!-- xacro:sensor_kinect name="base_front_camera" parent="base_link">
+	<!-- xacro:sensor_kinect prefix="$(arg prefix)base_front_camera" parent="$(arg prefix)base_link">
 		<origin xyz="0.6 0.0 0.102" rpy="0 0 0"/>
 	</xacro:sensor_kinect -->
 	<!-- IMU -->
-	<xacro:sensor_imu name="imu" prefix_frame="$(arg prefix_frame)" prefix_topic="$(arg prefix_topic)" parent="$(arg prefix_frame)base_link">
+	<xacro:sensor_imu prefix="$(arg prefix)imu" parent="$(arg prefix)base_link">
 		<origin xyz="-0.18 0.0 0.170" rpy="0 0 0"/>
 	</xacro:sensor_imu>
@@ -90,5 +89,5 @@
 	<!-- ************** -->
 	<!-- Gazebo ros control pluggins -->
-	<xacro:ros_control prefix_topic="$(arg prefix_topic)" prefix_frame="$(arg prefix_frame)"/>
-	<xacro:gazebo_colors prefix_topic="$(arg prefix_topic)" prefix_frame="$(arg prefix_frame)"/>
+	<xacro:ros_control/>
+	<xacro:gazebo_colors prefix="$(arg prefix)"/>
 </robot>

File: rb1_base_description/robots/rb1_base_v3_multi.urdf.xacro (robot description, xacro)
@@ -37,51 +37,50 @@
 	<!-- ROBOT COMPONENTS -->
 	<!-- *************** -->
-	<xacro:arg name="prefix_topic" default=""/>
-	<xacro:arg name="prefix_frame" default="rb1_"/>
+	<xacro:arg name="prefix" default="rb1_"/>
 	<!-- Here we create the robot elements using the xacro:macros imported at the beggining of this file -->
 	<!-- BASE -->
-	<xacro:rb1_base_v3 prefix_frame="$(arg prefix_frame)" publish_bf="true" hq="${hq}" />
+	<xacro:rb1_base_v3 prefix="$(arg prefix)" publish_bf="true" hq="${hq}" />
 	<!-- WHEELS -->
-	<xacro:rubber_wheel name="$(arg prefix_frame)right" parent="$(arg prefix_frame)base_link" reflect="false" hq="${hq}">
+	<xacro:rubber_wheel prefix="$(arg prefix)right" parent="$(arg prefix)base_link" reflect="false" hq="${hq}">
 		<origin xyz="${wheel_offset_x} -${wheel_offset_y} ${wheel_offset_z}" rpy="0 0 0"/>
 	</xacro:rubber_wheel>
-	<xacro:rubber_wheel name="$(arg prefix_frame)left" parent="$(arg prefix_frame)base_link" reflect="true" hq="${hq}">
+	<xacro:rubber_wheel prefix="$(arg prefix)left" parent="$(arg prefix)base_link" reflect="true" hq="${hq}">
 		<origin xyz="${wheel_offset_x} ${wheel_offset_y} ${wheel_offset_z}" rpy="0 0 0"/>
 	</xacro:rubber_wheel>
     <!-- OMNI DIRECTIONAL WHEELS -->
-	<xacro:omni_wheel name="$(arg prefix_frame)omni_back" parent="$(arg prefix_frame)base_link" hq="${hq}">
+	<xacro:omni_wheel prefix="$(arg prefix)omni_back" parent="$(arg prefix)base_link" hq="${hq}">
 		<origin xyz="-${omni_back_x} ${omni_back_y} ${omni_back_z}" rpy="0 0 0"/>
 	</xacro:omni_wheel>
-	<xacro:omni_wheel name="$(arg prefix_frame)omni_front_left" parent="$(arg prefix_frame)base_link" hq="${hq}">
+	<xacro:omni_wheel prefix="$(arg prefix)omni_front_left" parent="$(arg prefix)base_link" hq="${hq}">
 		<origin xyz="${omni_front_x} ${omni_front_y} ${omni_front_z}" rpy="0 0 0"/>
 	</xacro:omni_wheel>
-	<xacro:omni_wheel name="$(arg prefix_frame)omni_front_right" parent="$(arg prefix_frame)base_link" hq="${hq}">
+	<xacro:omni_wheel prefix="$(arg prefix)omni_front_right" parent="$(arg prefix)base_link" hq="${hq}">
 		<origin xyz="${omni_front_x} -${omni_front_y} ${omni_front_z}" rpy="0 0 0"/>
 	</xacro:omni_wheel>
 	<!-- SENSORS -->
 	<!-- LASER -->
-	<!-- xacro:sensor_hokuyo_utm30lx name="front_laser" parent="base_link">
+	<!-- xacro:sensor_hokuyo_utm30lx prefix="$(arg prefix)front_laser" parent="$(arg prefix)base_link">
 		<origin xyz="0.210 0.0 0.305" rpy="0 0 0"/>
 	</xacro:sensor_hokuyo_utm30lx -->
-	<!-- xacro:sensor_hokuyo_urg04lx name="front_laser" parent="base_link">
+	<!-- xacro:sensor_hokuyo_urg04lx prefix="$(arg prefix)front_laser" parent="$(arg prefix)base_link">
 		<origin xyz="0.220 0.0 0.170" rpy="0 3.1416 3.1416"/>
 	</xacro:sensor_hokuyo_urg04lx -->
-	<!-- xacro:sensor_hokuyo_ust10lx name="front_laser" parent="base_link">
+	<!-- xacro:sensor_hokuyo_ust10lx prefix="$(arg prefix)front_laser" parent="$(arg prefix)base_link">
 		<origin xyz="0.223 0.0 0.159" rpy="0 0 0"/>
 	</xacro:sensor_hokuyo_ust10lx -->
 	<!-- Name the components as base_front_laser or base_laser or front_laser or
 	a name which identify uniquely the component within the robot -->
-	<xacro:sensor_rplidar_a2 name="base_front_laser" prefix_frame="$(arg prefix_frame)" prefix_topic="$(arg prefix_topic)" parent="$(arg prefix_frame)base_link">
+	<xacro:sensor_rplidar_a2 prefix="$(arg prefix)base_front_laser" parent="$(arg prefix)base_link">
 		<origin xyz="0.210 0.0 0.199" rpy="3.1415 0 0"/>
 	</xacro:sensor_rplidar_a2>
 	<!-- CAMERA -->
-	<!--xacro:sensor_orbbec_astra name="base_front_camera" parent="base_link">
+	<!--xacro:sensor_orbbec_astra prefix="$(arg prefix)base_front_camera" parent="$(arg prefix)base_link">
 		<origin xyz="0.234 0.0125 0.107" rpy="0 0 0"/>
 	</xacro:sensor_orbbec_astra-->
-	<!-- xacro:sensor_kinect name="front_camera" parent="base_link">
+	<!-- xacro:sensor_kinect prefix="$(arg prefix)front_camera" parent="$(arg prefix)base_link">
 		<origin xyz="0.6 0.0 0.102" rpy="0 0 0"/>
 	</xacro:sensor_kinect -->
 	<!-- IMU -->
-	<xacro:sensor_imu name="imu" prefix_frame="$(arg prefix_frame)" prefix_topic="$(arg prefix_topic)" parent="$(arg prefix_frame)base_link">
+	<xacro:sensor_imu prefix="$(arg prefix)imu" parent="$(arg prefix)base_link">
 		<origin xyz="-0.18 0.0 0.170" rpy="0 0 0"/>
 	</xacro:sensor_imu>
@@ -90,5 +89,5 @@
 	<!-- ************** -->
 	<!-- Gazebo ros control pluggins -->
-	<xacro:ros_control prefix_topic="$(arg prefix_topic)" prefix_frame="$(arg prefix_frame)"/>
-	<xacro:gazebo_colors prefix_topic="$(arg prefix_topic)" prefix_frame="$(arg prefix_frame)"/>
+	<xacro:ros_control/>
+	<xacro:gazebo_colors prefix="$(arg prefix)"/>
 </robot>
