Commit message: [rb1_base_description]:xacros updated to multirobot

File: rb1_base_description/urdf/bases/rb1_base.urdf.xacro (robot description, xacro)
@@ -1,5 +1,5 @@
 <?xml version="1.0"?>
 <robot name="rb1_base" xmlns:xacro="http://www.ros.org/wiki/xacro">
-  <xacro:macro name="rb1_base" params="prefix_frame publish_bf hq">
+  <xacro:macro name="rb1_base" params="prefix publish_bf hq">
   <!-- Robot mechanical and motor parameters -->
   <xacro:property name="PI" value="3.1415926535897931"/>
@@ -7,5 +7,5 @@
   <!-- BASE FOOTPRINT -->
   <xacro:if value="${publish_bf}">
-    <link name="${prefix_frame}base_footprint">
+    <link name="${prefix}base_footprint">
       <visual>
           <origin xyz="0 0 0" rpy="0 0 0" />
@@ -15,12 +15,12 @@
       </visual>
     </link>
-    <joint name="base_footprint_joint" type="fixed">
+    <joint name="${prefix}base_footprint_joint" type="fixed">
        <origin xyz="0 0 ${wheel_radius - wheel_offset_z}" rpy="0 0 0" />
-      <parent link="${prefix_frame}base_footprint"/>
-      <child link="${prefix_frame}base_link" />
+      <parent link="${prefix}base_footprint"/>
+      <child link="${prefix}base_link" />
     </joint>
   </xacro:if>
   <!-- BASE_LINK -->
-  <link name="${prefix_frame}base_link">
+  <link name="${prefix}base_link">
     <inertial>
       <mass value="25.0" />
@@ -51,11 +51,11 @@
     </collision>
   </link>
-  <joint name="front_cover_joint" type="fixed">
+  <joint name="${prefix}front_cover_joint" type="fixed">
      <origin xyz="0.220 0.0 0.004" rpy="0 0 0 " />
-     <parent link="${prefix_frame}base_link"/>
-     <child link="${prefix_frame}front_cover_link" />
+     <parent link="${prefix}base_link"/>
+     <child link="${prefix}front_cover_link" />
   </joint>
   <!-- FRONT COVER -->
-  <link name="${prefix_frame}front_cover_link">
+  <link name="${prefix}front_cover_link">
     <inertial>
       <mass value="0.25" />
@@ -87,11 +87,11 @@
   </link>
   <!-- DOCKING CONTACTS -->
-  <joint name="base_docking_joint" type="fixed">
+  <joint name="${prefix}base_docking_joint" type="fixed">
      <origin xyz="0.030 0.000 0.068" rpy="0 0 0 " />
-     <parent link="${prefix_frame}front_cover_link"/>
-     <child link="${prefix_frame}base_docking_contact" />
+     <parent link="${prefix}front_cover_link"/>
+     <child link="${prefix}base_docking_contact" />
   </joint>
   <!-- FRONT COVER -->
-  <link name="${prefix_frame}base_docking_contact" />
+  <link name="${prefix}base_docking_contact" />
   </xacro:macro>
 </robot>

File: rb1_base_description/urdf/bases/rb1_base_v0.urdf.xacro (robot description, xacro)
@@ -1,5 +1,5 @@
 <?xml version="1.0"?>
 <robot name="rb1_base" xmlns:xacro="http://www.ros.org/wiki/xacro">
-  <xacro:macro name="rb1_base_v0" params="name publish_bf hq">
+  <xacro:macro name="rb1_base_v0" params="prefix publish_bf hq">
   <!-- Robot mechanical and motor parameters -->
   <xacro:property name="PI" value="3.1415926535897931"/>
@@ -7,5 +7,5 @@
   <!-- BASE FOOTPRINT -->
   <xacro:if value="${publish_bf}">
-    <link name="base_footprint">
+    <link name="${prefix}base_footprint">
       <visual>
           <origin xyz="0 0 0" rpy="0 0 0" />
@@ -15,12 +15,12 @@
       </visual>
     </link>
-    <joint name="base_footprint_joint" type="fixed">
+    <joint name="${prefix}base_footprint_joint" type="fixed">
        <origin xyz="0 0 ${wheel_radius - wheel_offset_z}" rpy="0 0 0" />
-      <parent link="base_footprint"/>
-      <child link="base_link" />
+      <parent link="${prefix}base_footprint"/>
+      <child link="${prefix}base_link" />
     </joint>
   </xacro:if>
   <!-- BASE_LINK -->
-  <link name="base_link">
+  <link name="${prefix}base_link">
     <inertial>
       <mass value="25.0" />

File: rb1_base_description/urdf/bases/rb1_base_v1.urdf.xacro (robot description, xacro)
@@ -1,5 +1,5 @@
 <?xml version="1.0"?>
 <robot name="rb1_base" xmlns:xacro="http://www.ros.org/wiki/xacro">
-  <xacro:macro name="rb1_base_v1" params="name publish_bf hq">
+  <xacro:macro name="rb1_base_v1" params="prefix publish_bf hq">
   <!-- Robot mechanical and motor parameters -->
   <xacro:property name="PI" value="3.1415926535897931"/>
@@ -7,5 +7,5 @@
   <!-- BASE FOOTPRINT -->
   <xacro:if value="${publish_bf}">
-    <link name="base_footprint">
+    <link name="${prefix}base_footprint">
       <visual>
           <origin xyz="0 0 0" rpy="0 0 0" />
@@ -15,12 +15,12 @@
       </visual>
     </link>
-    <joint name="base_footprint_joint" type="fixed">
+    <joint name="${prefix}base_footprint_joint" type="fixed">
        <origin xyz="0 0 ${wheel_radius - wheel_offset_z}" rpy="0 0 0" />
-      <parent link="base_footprint"/>
-      <child link="base_link" />
+      <parent link="${prefix}base_footprint"/>
+      <child link="${prefix}base_link" />
     </joint>
   </xacro:if>
   <!-- BASE_LINK -->
-  <link name="base_link">
+  <link name="${prefix}base_link">
     <inertial>
       <mass value="25.0" />

File: rb1_base_description/urdf/bases/rb1_base_v2.urdf.xacro (robot description, xacro)
@@ -1,5 +1,5 @@
 <?xml version="1.0"?>
 <robot name="rb1_base" xmlns:xacro="http://www.ros.org/wiki/xacro">
-  <xacro:macro name="rb1_base_v2" params="prefix_frame publish_bf hq">
+  <xacro:macro name="rb1_base_v2" params="prefix publish_bf hq">
   <!-- Robot mechanical and motor parameters -->
   <xacro:property name="PI" value="3.1415926535897931"/>
@@ -7,5 +7,5 @@
   <!-- BASE FOOTPRINT -->
   <xacro:if value="${publish_bf}">
-    <link name="${prefix_frame}base_footprint">
+    <link name="${prefix}base_footprint">
       <visual>
           <origin xyz="0 0 0" rpy="0 0 0" />
@@ -15,12 +15,12 @@
       </visual>
     </link>
-    <joint name="base_footprint_joint" type="fixed">
+    <joint name="${prefix}base_footprint_joint" type="fixed">
        <origin xyz="0 0 ${wheel_radius - wheel_offset_z}" rpy="0 0 0" />
-      <parent link="${prefix_frame}base_footprint"/>
-      <child link="${prefix_frame}base_link" />
+      <parent link="${prefix}base_footprint"/>
+      <child link="${prefix}base_link" />
     </joint>
   </xacro:if>
   <!-- BASE_LINK -->
-  <link name="${prefix_frame}base_link">
+  <link name="${prefix}base_link">
     <inertial>
       <mass value="25.0" />
@@ -51,11 +51,11 @@
     </collision>
   </link>
-  <joint name="front_cover_joint" type="fixed">
+  <joint name="${prefix}front_cover_joint" type="fixed">
      <origin xyz="0.220 0.0 0.004" rpy="0 0 0 " />
-     <parent link="${prefix_frame}base_link"/>
-     <child link="${prefix_frame}front_cover_link" />
+     <parent link="${prefix}base_link"/>
+     <child link="${prefix}front_cover_link" />
   </joint>
   <!-- FRONT COVER -->
-  <link name="${prefix_frame}front_cover_link">
+  <link name="${prefix}front_cover_link">
     <inertial>
       <mass value="0.25" />
@@ -87,11 +87,11 @@
   </link>
   <!-- DOCKING CONTACTS -->
-  <joint name="base_docking_joint" type="fixed">
+  <joint name="${prefix}base_docking_joint" type="fixed">
      <origin xyz="0.030 0.000 0.068" rpy="0 0 0 " />
-     <parent link="${prefix_frame}front_cover_link"/>
-     <child link="${prefix_frame}base_docking_contact_link" />
+     <parent link="${prefix}front_cover_link"/>
+     <child link="${prefix}base_docking_contact_link" />
   </joint>
   <!-- DOCKING LINK -->
-  <link name="${prefix_frame}base_docking_contact_link" />
+  <link name="${prefix}base_docking_contact_link" />
   </xacro:macro>
 </robot>

File: rb1_base_description/urdf/bases/rb1_base_v3.urdf.xacro (robot description, xacro)
@@ -1,5 +1,5 @@
 <?xml version="1.0"?>
 <robot name="rb1_base" xmlns:xacro="http://www.ros.org/wiki/xacro">
-  <xacro:macro name="rb1_base_v3" params="prefix_frame publish_bf hq">
+  <xacro:macro name="rb1_base_v3" params="prefix publish_bf hq">
   <!-- Robot mechanical and motor parameters -->
   <xacro:property name="PI" value="3.1415926535897931"/>
@@ -7,5 +7,5 @@
   <!-- BASE FOOTPRINT -->
   <xacro:if value="${publish_bf}">
-    <link name="${prefix_frame}base_footprint">
+    <link name="${prefix}base_footprint">
       <visual>
           <origin xyz="0 0 0" rpy="0 0 0" />
@@ -15,12 +15,12 @@
       </visual>
     </link>
-    <joint name="base_footprint_joint" type="fixed">
+    <joint name="${prefix}base_footprint_joint" type="fixed">
        <origin xyz="0 0 ${wheel_radius - wheel_offset_z}" rpy="0 0 0" />
-      <parent link="${prefix_frame}base_footprint"/>
-      <child link="${prefix_frame}base_link" />
+      <parent link="${prefix}base_footprint"/>
+      <child link="${prefix}base_link" />
     </joint>
   </xacro:if>
   <!-- BASE_LINK -->
-  <link name="${prefix_frame}base_link">
+  <link name="${prefix}base_link">
     <inertial>
       <mass value="25.0" />
@@ -51,11 +51,11 @@
     </collision>
   </link>
-  <joint name="front_cover_joint" type="fixed">
+  <joint name="${prefix}front_cover_joint" type="fixed">
      <origin xyz="0.220 0.0 0.004" rpy="0 0 0 " />
-     <parent link="${prefix_frame}base_link"/>
-     <child link="${prefix_frame}front_cover_link" />
+     <parent link="${prefix}base_link"/>
+     <child link="${prefix}front_cover_link" />
   </joint>
   <!-- FRONT COVER -->
-  <link name="${prefix_frame}front_cover_link">
+  <link name="${prefix}front_cover_link">
     <inertial>
       <mass value="0.25" />
@@ -86,11 +86,11 @@
     </collision>
   </link>
-  <joint name="top_covert_joint" type="fixed">
+  <joint name="${prefix}top_covert_joint" type="fixed">
      <origin xyz="0.0 0.0 0.243" rpy="0 0 0 " />
-     <parent link="${prefix_frame}base_footprint"/>
-     <child link="${prefix_frame}top_cover_link" />
+     <parent link="${prefix}base_footprint"/>
+     <child link="${prefix}top_cover_link" />
   </joint>
   <!-- FRONT COVER -->
-  <link name="${prefix_frame}top_cover_link">
+  <link name="${prefix}top_cover_link">
     <inertial>
       <mass value="0.25" />
@@ -122,11 +122,11 @@
   </link>
   <!-- DOCKING CONTACTS -->
-  <joint name="base_docking_joint" type="fixed">
+  <joint name="${prefix}base_docking_joint" type="fixed">
      <origin xyz="0.030 0.000 0.068" rpy="0 0 0 " />
-     <parent link="${prefix_frame}front_cover_link"/>
-     <child link="${prefix_frame}base_docking_contact_link" />
+     <parent link="${prefix}front_cover_link"/>
+     <child link="${prefix}base_docking_contact_link" />
   </joint>
   <!-- DOCKING LINK -->
-  <link name="${prefix_frame}base_docking_contact_link" />
+  <link name="${prefix}base_docking_contact_link" />
   </xacro:macro>
 </robot>

File: rb1_base_description/urdf/common.gazebo.xacro (robot description, xacro)
@@ -2,5 +2,5 @@
 <robot xmlns:xacro="http://www.ros.org/wiki/xacro">
 <!-- ROS CONTROL GAZEBO PLUGIN -->
-	<xacro:macro name="ros_control" params="prefix_frame prefix_topic">
+	<xacro:macro name="ros_control">
 	   <gazebo>
       <plugin name="ros_control" filename="libgazebo_ros_control.so">
@@ -12,12 +12,12 @@
    </gazebo>
    </xacro:macro>
-   <xacro:macro name="gazebo_colors" params="prefix_frame prefix_topic">
-		<gazebo reference="$(arg prefix_frame)base_footprint">
+   <xacro:macro name="gazebo_colors" params="prefix">
+		<gazebo reference="$(arg prefix)base_footprint">
 			<material>Gazebo/Green</material>
 		</gazebo>
-		<gazebo reference="$(arg prefix_frame)base_link">
+		<gazebo reference="$(arg prefix)base_link">
 			<material>Gazebo/Grey</material>
 		</gazebo>
-		<gazebo reference="$(arg prefix_frame)front_cover_link">
+		<gazebo reference="$(arg prefix)front_cover_link">
 			<material>Gazebo/Black</material>
 		</gazebo>

File: rb1_base_description/urdf/elevator/elevator.urdf.xacro (robot description, xacro)
@@ -2,15 +2,15 @@
 <robot xmlns:xacro="http://www.ros.org/wiki/xacro">
 	<!--xacro:include filename="$(find rb1_base_description)/urdf/bases/rb1_elevator.gazebo.xacro" /-->
-	<xacro:macro name="elevator_platform" params="name parent hq *origin">
+	<xacro:macro name="elevator_platform" params="prefix parent hq *origin">
 	<!-- PARAMS: -->
 	<!-- name : name of the link: -->
 	<!-- hq: selects model in high quality (.dae) -->
 	<!-- ELEVATOR_BASE_LINK -->
-	<joint name="${name}_base_joint" type="fixed">
+	<joint name="${prefix}_base_joint" type="fixed">
 		<parent link="${parent}"/>
-		<child link="${name}_base_link"/>
+		<child link="${prefix}_base_link"/>
 		<xacro:insert_block name="origin" />
 	</joint>
-	<link name="${name}_base_link">
+	<link name="${prefix}_base_link">
 		<!--inertial>
 			<mass value="25.0" />
@@ -44,12 +44,12 @@
 	</link>
 	<!-- ELEVATOR PLATFORM -->
-	<joint name="${name}_platform_joint" type="prismatic">
+	<joint name="${prefix}_platform_joint" type="prismatic">
 			<origin xyz="0.0 0.0 0.041" rpy="0 0 0 " />
-			<parent link="${name}_base_link"/>
-			<child link="${name}_platform_link" />
+			<parent link="${prefix}_base_link"/>
+			<child link="${prefix}_platform_link" />
 			<axis xyz="0 0 1"/>
 			<limit effort="1.0" lower="0.0" upper="0.034" velocity="0.5"/>
 	</joint>
-	<link name="${name}_platform_link">
+	<link name="${prefix}_platform_link">
 		<!--inertial>
 			<mass value="0.25" />

File: rb1_base_description/urdf/wheels/omni_wheel.urdf.xacro (robot description, xacro)
@@ -12,10 +12,10 @@
      />
   </xacro:macro>
-  <xacro:macro name="omni_wheel" params="name parent *origin hq">
+  <xacro:macro name="omni_wheel" params="prefix parent *origin hq">
 <!--WHEEL TIRE -->
     <!-- joint name="joint_${name}_wheel" type="continuous" -->
-    <joint name="joint_${name}_wheel" type="fixed">
+    <joint name="${prefix}wheel_joint" type="fixed">
       <parent link="${parent}"/>
-      <child link="${name}_wheel"/>
+      <child link="${prefix}wheel_link"/>
       <xacro:insert_block name="origin" />
       <axis xyz="0 1 0" rpy="0 0 0" />
@@ -23,5 +23,5 @@
       <joint_properties damping="0.0" friction="0.0"/>
     </joint>
-    <link name="${name}_wheel">
+    <link name="${prefix}wheel_link">
       <visual>
         <!-- HIGH RESOLUTION WHEELS -->
@@ -67,5 +67,5 @@
       </actuator>
     </transmission -->
-    <gazebo reference="${name}_wheel">
+    <gazebo reference="${prefix}wheel">
 		<mu1 value="0"/>
 		<mu2 value="0"/>

File: rb1_base_description/urdf/wheels/rubber_wheel.gazebo.xacro (robot description, xacro)
@@ -1,6 +1,6 @@
 <?xml version="1.0"?>
 <robot xmlns:xacro="http://www.ros.org/wiki/xacro">
-	<xacro:macro name="rubber_wheel_gazebo" params="name">
-		<gazebo reference="${name}_wheel_link">
+	<xacro:macro name="rubber_wheel_gazebo" params="prefix">
+		<gazebo reference="${prefix}_wheel_link">
 			<mu1 value="5.0"/>
 			<mu2 value="0.5"/>

File: rb1_base_description/urdf/wheels/rubber_wheel.transmission.xacro (robot description, xacro)
@@ -2,9 +2,9 @@
 <robot xmlns:xacro="http://www.ros.org/wiki/xacro">
 	<!-- Rubber wheel transmission -->
-	<xacro:macro name="rubber_wheel_transmission" params="name">
+	<xacro:macro name="rubber_wheel_transmission" params="prefix">
 	<!-- Transmission is important to link the joints and the controller (see rb1_control/config/rb1_control.yaml)-->
-		<transmission name="${name}_wheel_joint_trans">
+		<transmission name="${prefix}_wheel_joint_trans">
 			<type>transmission_interface/SimpleTransmission</type>
-			<joint name="${name}_wheel_joint">
+			<joint name="${prefix}_wheel_joint">
 				<!-- for the gazebo plugin -->
 				<!--hardwareInterface>EffortJointInterface</hardwareInterface-->
@@ -12,5 +12,5 @@
 				<hardwareInterface>hardware_interface/VelocityJointInterface</hardwareInterface>
 			</joint>
-			<actuator name="${name}_wheel_joint_motor">
+			<actuator name="${prefix}_wheel_joint_motor">
 				<mechanicalReduction>1</mechanicalReduction>
 				<motorTorqueConstant>20</motorTorqueConstant>

File: rb1_base_description/urdf/wheels/rubber_wheel.urdf.xacro (robot description, xacro)
@@ -13,9 +13,9 @@
 					izz="${m*r*r/2}" />
 	</xacro:macro>
-	<xacro:macro name="rubber_wheel" params="name parent *origin reflect hq">
+	<xacro:macro name="rubber_wheel" params="prefix parent *origin reflect hq">
 	<!--WHEEL TIRE -->
-	<joint name="${name}_wheel_joint" type="continuous">
+	<joint name="${prefix}_wheel_joint" type="continuous">
 		<parent link="${parent}"/>
-		<child link="${name}_wheel_link"/>
+		<child link="${prefix}_wheel_link"/>
 		<xacro:insert_block name="origin" />
 		<axis xyz="0 1 0" rpy="0 0 0" />
@@ -23,5 +23,5 @@
 		<joint_properties damping="0.0" friction="0.0"/>
 	</joint>
-	<link name="${name}_wheel_link">
+	<link name="${prefix}_wheel_link">
 		<visual>
 		<!-- HIGH RESOLUTION WHEELS -->
@@ -57,6 +57,6 @@
       </inertial>
     </link>
-	<xacro:rubber_wheel_transmission name="${name}" />
-	<xacro:rubber_wheel_gazebo name="${name}" />
+	<xacro:rubber_wheel_transmission prefix="${prefix}" />
+	<xacro:rubber_wheel_gazebo prefix="${prefix}" />
   </xacro:macro>
 </robot>
