Commit message: added sensor to non standalone platform

File: rb1_base_description/robots/rb1_base_platform.urdf.xacro (robot description, xacro)
@@ -25,5 +25,5 @@
 	<xacro:property name="omni_back_z" value="0.0265" />
 	<xacro:property name="omni_front_x" value="0.133" />
-	<xacro:property name="omni_front_y" value="0.144" />
+	<xacro:property name="omni_front_y" value="0.148" />
 	<xacro:property name="omni_front_z" value="0.0265" />
 	<!-- Flag to select the high or low quality model -->
@@ -69,4 +69,7 @@
 		<origin xyz="-0.18 0.0 0.170" rpy="0 0 0"/>
 	</xacro:sensor_imu>
+    <xacro:sensor_orbbec_astra name="orbbec_astra" parent="base_link">
+        <origin xyz="0.234 0.0125 0.107" rpy="0 0 0"/>
+    </xacro:sensor_orbbec_astra>
 <!--
     <xacro:sensor_kinect name="kinect" parent="base_link">

Commit message: MOD: Normalize directories

File: rb1_base_description/robots/rb1_base_platform.urdf.xacro (robot description, xacro)
@@ -1,24 +1,25 @@
 <?xml version="1.0"?>
-<robot name="rb1_base_platform" xmlns:xacro="http://www.ros.org/wiki/xacro">
-	<!-- ***************** -->
-	<!-- Imported elements -->
-	<!-- ***************** -->
+<robot name="rb1_base" xmlns:xacro="http://www.ros.org/wiki/xacro">
+	<!-- ************* -->
+	<!-- IMPORT MACROS -->
+	<!-- ************* -->
 	<!-- First we import all posible elements defined in the urdf.xacro files. All these elements are defined as macro:xacros -->
-	<!-- Import RB1 base elements -->
+	<!-- BASES -->
     <xacro:include filename="$(find rb1_base_description)/urdf/bases/rb1_base.urdf.xacro" />
-	<!-- Import RB1 wheels -->
+	<!-- WHEELS -->
 	<xacro:include filename="$(find rb1_base_description)/urdf/wheels/rubber_wheel.urdf.xacro" />
 	<xacro:include filename="$(find rb1_base_description)/urdf/wheels/omni_wheel.urdf.xacro" />
-	<!-- Import all available sensors -->
+    <!-- SENSORS -->
 	<xacro:include filename="$(find robotnik_sensors)/urdf/all_sensors.urdf.xacro" />
-	<!-- ***************** -->
-	<!-- Global parameters -->
-	<!-- ***************** -->
+	<!-- ********** -->
+	<!-- PROPERTIES -->
+	<!-- ********** -->
+	<!-- MATH -->
 	<xacro:property name="PI" value="3.1415926535897931"/>
-	<!-- Wheel parameters -->
+    <!-- MOTOR WHEELS -->
 	<xacro:property name="wheel_offset_x" value="0.0" />    <!-- x,y,z in translation from base_link to the center of the wheel -->
 	<xacro:property name="wheel_offset_y" value="0.217" />
 	<xacro:property name="wheel_offset_z" value="0.051" />
-	<!-- Castor paramters -->
+	<!-- CASTOR WHEELS -->
 	<xacro:property name="omni_back_x" value="0.195" />
 	<xacro:property name="omni_back_y" value="0.0" />
@@ -35,8 +36,8 @@
 	<!-- RB-1 base -->
 	<xacro:rb1_base name="rb1_base" publish_bf="true" hq="${hq}" />
-	<!-- Gazebo ros control plugins -->
-	<xacro:ros_control/>
-	<!-- Gazebo skid steering plugins -->
-	<xacro:diff_drive/>
+	<!-- ROS CONTROL GAZEBO PLUGIN -->
+	<!--xacro:ros_control/-->
+	<!-- DIFFERENCIAL DRIVE GAZEBO PLUGIN -->
+	<!--xacro:diff_drive/-->
 	<!-- WHEELS -->
 	<xacro:rubber_wheel name="right" parent="base_link" reflect="false" hq="${hq}">
@@ -57,23 +58,27 @@
 	</xacro:omni_wheel>
 	<!-- SENSORS -->
-	<!-- xacro:sensor_hokuyo_utm30lx name="hokuyo" parent="base_link">
+	<!-- LASER -->
+	<!-- xacro:sensor_hokuyo_utm30lx name="front_laser" parent="base_link">
 		<origin xyz="0.210 0.0 0.305" rpy="0 0 0"/>
 	</xacro:sensor_hokuyo_utm30lx -->
-    <!-- xacro:sensor_hokuyo_urg04lx name="hokuyo" parent="base_link">
-        <origin xyz="0.223 0.0 0.209" rpy="0 3.1416 3.1416"/>
+    <!-- xacro:sensor_hokuyo_urg04lx name="front_laser" parent="base_link">
+        <origin xyz="0.220 0.0 0.170" rpy="0 3.1416 3.1416"/>
     </xacro:sensor_hokuyo_urg04lx -->
-	<xacro:sensor_hokuyo_ust10lx name="hokuyo" parent="base_link">
+	<!-- xacro:sensor_hokuyo_ust10lx name="front_laser" parent="base_link">
+		<origin xyz="0.223 0.0 0.159" rpy="0 0 0"/>
+	</xacro:sensor_hokuyo_ust10lx -->
+	<xacro:sensor_hokuyo_ust10lx name="front_laser" parent="base_link">
 		<origin xyz="0.223 0.0 0.159" rpy="0 3.1416 3.1416"/>
 	</xacro:sensor_hokuyo_ust10lx>
-	<xacro:sensor_imu name="imu" parent="base_link">
-		<origin xyz="-0.18 0.0 0.170" rpy="0 0 0"/>
-	</xacro:sensor_imu>
-    <xacro:sensor_orbbec_astra name="orbbec_astra" parent="base_link">
+	<!-- CAMERA -->
+    <xacro:sensor_orbbec_astra name="front_camera" parent="base_link">
         <origin xyz="0.234 0.0125 0.107" rpy="0 0 0"/>
     </xacro:sensor_orbbec_astra>
-<!--
-    <xacro:sensor_kinect name="kinect" parent="base_link">
-        <origin xyz="0.3 0.0 0.16" rpy="0 0 0"/>
-    </xacro:sensor_kinect>
--->
+    <!-- xacro:sensor_kinect name="front_camera" parent="base_link">
+        <origin xyz="0.6 0.0 0.102" rpy="0 0 0"/>
+    </xacro:sensor_kinect -->
+    <!-- IMU -->
+    <xacro:sensor_imu name="imu" parent="base_link">
+        <origin xyz="-0.18 0.0 0.170" rpy="0 0 0"/>
+    </xacro:sensor_imu>
 </robot>

File: rb1_base_description/urdf/wheels/omni_wheel.urdf.xacro (robot description, xacro)
@@ -9,5 +9,6 @@
     <inertia  ixx="${m*(3*r*r+h*h)/12}" ixy = "0" ixz = "0"
               iyy="${m*(3*r*r+h*h)/12}" iyz = "0"
-              izz="${m*r*r/2}" />
+              izz="${m*r*r/2}"
+     />
   </xacro:macro>
   <xacro:macro name="omni_wheel" params="name parent *origin hq">
@@ -67,11 +68,24 @@
     </transmission -->
     <gazebo reference="${name}_wheel">
-			<mu1 value="0.0"/>
-			<mu2 value="0.0"/>
-			<kp value="10000000.0" />
-			<kd value="1.0" />
-			<fdir1 value="1 0 0"/>
-            <turnGravityOff>false</turnGravityOff>
+		<mu1 value="0"/>
+		<mu2 value="0"/>
+		<kp value="10000000.0" />
+		<kd value="1.0" />
+		<fdir1 value="1 0 0"/>
+		<material>Gazebo/Black</material>
+		<turnGravityOff>false</turnGravityOff>
     </gazebo>
+    <!--gazebo reference="${name}_wheel">
+		<kp>500000.0</kp>
+		<kd>10.0</kd>
+		<mu1>10</mu1>
+		<mu2>10</mu2>
+		<fdir1>1 0 0</fdir1>
+		<maxVel>1.0</maxVel>
+		<minDepth>0.003</minDepth>
+		<material>Gazebo/Black</material>
+		<turnGravityOff>false</turnGravityOff>
+		<implicitSpringDamper>1</implicitSpringDamper>
+    </gazebo-->
   </xacro:macro>
 </robot>

File: rb1_base_description/urdf/wheels/rubber_wheel.urdf.xacro (robot description, xacro)
@@ -1,46 +1,48 @@
 <?xml version="1.0"?>
 <robot name="wheel" xmlns:xacro="http://www.ros.org/wiki/xacro">
-  <xacro:property name="M_PI" value="3.1415926535897931" />
-  <!-- Wheels -->
-  <property name="wheel_radius" value="0.076" />
-  <property name="wheel_height" value="0.025" />
-  <property name="wheel_mass" value="1.0" /> <!-- in kg-->
-  <xacro:macro name="cylinder_inertia" params="m r h">
-    <inertia  ixx="${m*(3*r*r+h*h)/12}" ixy = "0" ixz = "0"
-              iyy="${m*(3*r*r+h*h)/12}" iyz = "0"
-              izz="${m*r*r/2}" />
-  </xacro:macro>
-  <xacro:macro name="rubber_wheel" params="name parent *origin reflect hq">
-  <!--WHEEL TIRE -->
-    <joint name="joint_${name}_wheel" type="continuous">
-      <parent link="${parent}"/>
-      <child link="${name}_wheel"/>
-      <insert_block name="origin" />
-      <axis xyz="0 1 0" rpy="0 0 0" />
-      <limit effort="100" velocity="100"/>
-      <joint_properties damping="0.0" friction="0.0"/>
-    </joint>
-    <link name="${name}_wheel">
-      <visual>
-        <!-- HIGH RESOLUTION WHEELS -->
-        <xacro:if value="${hq}">
-          <origin xyz="0 0 0" rpy="0 0 0" />
-          <geometry>
-			<xacro:if value="${reflect}">
-				<mesh filename="package://rb1_base_description/meshes/wheels/wheel_rubber_6inch.dae" />
-			</xacro:if>
-			<xacro:unless value="${reflect}">
-				<mesh filename="package://rb1_base_description/meshes/wheels/wheel_rubber_6inch.dae" />
-			</xacro:unless>
-          </geometry>
-        </xacro:if>
-       <!-- LOW RESOLUTION WHEELS -->
-        <xacro:unless value="${hq}">
-          <origin xyz="0 0 0" rpy="${M_PI/2} 0 0" />
-          <geometry>
-            <cylinder length="${wheel_height}" radius="${wheel_radius}" />
-          </geometry>
-        </xacro:unless>
-      </visual>
+	<xacro:include filename="$(find rb1_base_description)/urdf/wheels/rubber_wheel.transmission.xacro"/>
+	<xacro:include filename="$(find rb1_base_description)/urdf/wheels/rubber_wheel.gazebo.xacro"/>
+	<xacro:property name="M_PI" value="3.1415926535897931" />
+	<!-- Wheels -->
+	<property name="wheel_radius" value="0.076" />
+	<property name="wheel_height" value="0.025" />
+	<property name="wheel_mass" value="1.0" /> <!-- in kg-->
+	<xacro:macro name="cylinder_inertia" params="m r h">
+		<inertia	ixx="${m*(3*r*r+h*h)/12}" ixy = "0" ixz = "0"
+					iyy="${m*(3*r*r+h*h)/12}" iyz = "0"
+					izz="${m*r*r/2}" />
+	</xacro:macro>
+	<xacro:macro name="rubber_wheel" params="name parent *origin reflect hq">
+	<!--WHEEL TIRE -->
+	<joint name="${name}_wheel_joint" type="continuous">
+		<parent link="${parent}"/>
+		<child link="${name}_wheel_link"/>
+		<insert_block name="origin" />
+		<axis xyz="0 1 0" rpy="0 0 0" />
+		<limit effort="100" velocity="100"/>
+		<joint_properties damping="0.0" friction="0.0"/>
+	</joint>
+	<link name="${name}_wheel_link">
+		<visual>
+		<!-- HIGH RESOLUTION WHEELS -->
+		<xacro:if value="${hq}">
+			<origin xyz="0 0 0" rpy="0 0 0" />
+			<geometry>
+				<xacro:if value="${reflect}">
+					<mesh filename="package://rb1_base_description/meshes/wheels/wheel_rubber_6inch.dae" />
+				</xacro:if>
+				<xacro:unless value="${reflect}">
+					<mesh filename="package://rb1_base_description/meshes/wheels/wheel_rubber_6inch.dae" />
+				</xacro:unless>
+			</geometry>
+		</xacro:if>
+		<!-- LOW RESOLUTION WHEELS -->
+		<xacro:unless value="${hq}">
+			<origin xyz="0 0 0" rpy="${M_PI/2} 0 0" />
+			<geometry>
+				<cylinder length="${wheel_height}" radius="${wheel_radius}" />
+			</geometry>
+		</xacro:unless>
+		</visual>
       <collision>
 		<origin xyz="0 0 0" rpy="${M_PI/2} 0 0" />
@@ -55,26 +57,6 @@
       </inertial>
     </link>
-    <!-- Transmission is important to link the joints and the controller (see rb1_control/config/rb1_control.yaml)-->
-    <transmission name="${name}_wheel_joint_trans">
-      <type>transmission_interface/SimpleTransmission</type>
-      <joint name="joint_${name}_wheel">
-          <!-- for the gazebo plugin -->
-          <!-- hardwareInterface>EffortJointInterface</hardwareInterface -->
-          <!-- for ros control controller -->
-          <hardwareInterface>VelocityJointInterface</hardwareInterface>
-      </joint>
-      <actuator name="${name}_wheel_joint_motor">
-        <mechanicalReduction>1</mechanicalReduction>
-        <motorTorqueConstant>20</motorTorqueConstant>
-      </actuator>
-    </transmission>
-    <gazebo reference="${name}_wheel">
-			<mu1 value="5.0"/>
-			<mu2 value="0.5"/>
-			<kp value="10000000.0" />
-			<kd value="1.0" />
-			<fdir1 value="1 0 0"/>
-      <turnGravityOff>false</turnGravityOff>
-    </gazebo>
+	<xacro:rubber_wheel_transmission name="${name}" />
+	<xacro:rubber_wheel_gazebo name="${name}" />
   </xacro:macro>
 </robot>
