Commit message: rb1_base_description: updated sensor parameters in urdf

File: rb1_base_description/robots/rb1_base_platform.urdf.xacro (robot description, xacro)
@@ -59,25 +59,25 @@
 	<!-- SENSORS -->
 	<!-- LASER -->
-	<!-- xacro:sensor_hokuyo_utm30lx name="front_laser" parent="base_link">
+	<!-- xacro:sensor_hokuyo_utm30lx prefix="front_laser" parent="base_link">
 		<origin xyz="0.210 0.0 0.305" rpy="0 0 0"/>
 	</xacro:sensor_hokuyo_utm30lx -->
-    <!-- xacro:sensor_hokuyo_urg04lx name="front_laser" parent="base_link">
+    <!-- xacro:sensor_hokuyo_urg04lx prefix="front_laser" parent="base_link">
         <origin xyz="0.220 0.0 0.170" rpy="0 3.1416 3.1416"/>
     </xacro:sensor_hokuyo_urg04lx -->
-	<!-- xacro:sensor_hokuyo_ust10lx name="front_laser" parent="base_link">
+	<!-- xacro:sensor_hokuyo_ust10lx prefix="front_laser" parent="base_link">
 		<origin xyz="0.223 0.0 0.159" rpy="0 0 0"/>
 	</xacro:sensor_hokuyo_ust10lx -->
-	<xacro:sensor_hokuyo_ust10lx name="front_laser" parent="base_link">
+	<xacro:sensor_hokuyo_ust10lx prefix="front_laser" parent="base_link">
 		<origin xyz="0.223 0.0 0.159" rpy="0 3.1416 3.1416"/>
 	</xacro:sensor_hokuyo_ust10lx>
 	<!-- CAMERA -->
-    <xacro:sensor_orbbec_astra name="front_camera" parent="base_link">
+    <xacro:sensor_orbbec_astra prefix="front_camera" parent="base_link">
         <origin xyz="0.234 0.0125 0.107" rpy="0 0 0"/>
     </xacro:sensor_orbbec_astra>
-    <!-- xacro:sensor_kinect name="front_camera" parent="base_link">
+    <!-- xacro:sensor_kinect prefix="front_camera" parent="base_link">
         <origin xyz="0.6 0.0 0.102" rpy="0 0 0"/>
     </xacro:sensor_kinect -->
     <!-- IMU -->
-    <xacro:sensor_imu name="imu" parent="base_link">
+    <xacro:sensor_imu prefix="imu" parent="base_link">
         <origin xyz="-0.18 0.0 0.170" rpy="0 0 0"/>
     </xacro:sensor_imu>

File: rb1_base_description/robots/rb1_base_platform_kinova.urdf.xacro (robot description, xacro)
@@ -66,23 +66,23 @@
 	</xacro:omni_wheel>
 	<!-- SENSORS -->
-	<!-- xacro:sensor_hokuyo_utm30lx name="hokuyo" parent="base_link">
+	<!-- xacro:sensor_hokuyo_utm30lx prefix="hokuyo" parent="base_link">
 		<origin xyz="0.210 0.0 0.305" rpy="0 0 0"/>
 	</xacro:sensor_hokuyo_utm30lx -->
-    <!-- xacro:sensor_hokuyo_urg04lx name="hokuyo1" parent="base_link">
+    <!-- xacro:sensor_hokuyo_urg04lx prefix="hokuyo1" parent="base_link">
         <origin xyz="0.220 0.0 0.170" rpy="0 3.1416 3.1416"/>
     </xacro:sensor_hokuyo_urg04lx -->
-	<!-- xacro:sensor_hokuyo_ust10lx name="hokuyo" parent="base_link">
+	<!-- xacro:sensor_hokuyo_ust10lx prefix="hokuyo" parent="base_link">
 		<origin xyz="0.223 0.0 0.159" rpy="0 0 0"/>
 	</xacro:sensor_hokuyo_ust10lx -->
-	<xacro:sensor_hokuyo_ust10lx name="hokuyo" parent="base_link">
+	<xacro:sensor_hokuyo_ust10lx prefix="hokuyo" parent="base_link">
 		<origin xyz="0.223 0.0 0.159" rpy="0 3.1416 3.1416"/>
 	</xacro:sensor_hokuyo_ust10lx>
-	<xacro:sensor_imu name="imu" parent="base_link">
+	<xacro:sensor_imu prefix="imu" parent="base_link">
 		<origin xyz="-0.18 0.0 0.170" rpy="0 0 0"/>
 	</xacro:sensor_imu>
-    <!-- xacro:sensor_orbbec_astra name="orbbec_astra" parent="base_link">
+    <!-- xacro:sensor_orbbec_astra prefix="orbbec_astra" parent="base_link">
         <origin xyz="0.234 0.0125 0.107" rpy="0 0 0"/>
     </xacro:sensor_orbbec_astra -->
-    <xacro:sensor_orbbec_astra name="orbbec_astra" parent="base_link">
+    <xacro:sensor_orbbec_astra prefix="orbbec_astra" parent="base_link">
         <origin xyz="0.234 0.0125 0.107" rpy="0 0 0"/>
     </xacro:sensor_orbbec_astra>
@@ -90,5 +90,5 @@
         <origin xyz="0.0 0.0 0.213" rpy="0 0 0"/>
     </xacro:kinova_base>
-    <!-- xacro:sensor_kinect name="kinect" parent="base_link">
+    <!-- xacro:sensor_kinect prefix="kinect" parent="base_link">
         <origin xyz="0.6 0.0 0.102" rpy="0 0 0"/>
     </xacro:sensor_kinect -->

File: rb1_base_description/robots/rb1_base_platform_kinova_j2n6a300.urdf.xacro (robot description, xacro)
@@ -68,23 +68,23 @@
 	</xacro:omni_wheel>
 	<!-- SENSORS -->
-	<!-- xacro:sensor_hokuyo_utm30lx name="hokuyo" parent="base_link">
+	<!-- xacro:sensor_hokuyo_utm30lx prefix="hokuyo" parent="base_link">
 		<origin xyz="0.210 0.0 0.305" rpy="0 0 0"/>
 	</xacro:sensor_hokuyo_utm30lx -->
-    <!-- xacro:sensor_hokuyo_urg04lx name="hokuyo1" parent="base_link">
+    <!-- xacro:sensor_hokuyo_urg04lx prefix="hokuyo1" parent="base_link">
         <origin xyz="0.220 0.0 0.170" rpy="0 3.1416 3.1416"/>
     </xacro:sensor_hokuyo_urg04lx -->
-	<!-- xacro:sensor_hokuyo_ust10lx name="hokuyo" parent="base_link">
+	<!-- xacro:sensor_hokuyo_ust10lx prefix="hokuyo" parent="base_link">
 		<origin xyz="0.223 0.0 0.159" rpy="0 0 0"/>
 	</xacro:sensor_hokuyo_ust10lx -->
-	<xacro:sensor_hokuyo_ust10lx name="hokuyo" parent="base_link">
+	<xacro:sensor_hokuyo_ust10lx prefix="hokuyo" parent="base_link">
 		<origin xyz="0.223 0.0 0.159" rpy="0 3.1416 3.1416"/>
 	</xacro:sensor_hokuyo_ust10lx>
-	<xacro:sensor_imu name="imu" parent="base_link">
+	<xacro:sensor_imu prefix="imu" parent="base_link">
 		<origin xyz="-0.18 0.0 0.170" rpy="0 0 0"/>
 	</xacro:sensor_imu>
-    <!-- xacro:sensor_orbbec_astra name="orbbec_astra" parent="base_link">
+    <!-- xacro:sensor_orbbec_astra prefix="orbbec_astra" parent="base_link">
         <origin xyz="0.234 0.0125 0.107" rpy="0 0 0"/>
     </xacro:sensor_orbbec_astra -->
-    <xacro:sensor_orbbec_astra name="orbbec_astra" parent="base_link">
+    <xacro:sensor_orbbec_astra prefix="orbbec_astra" parent="base_link">
         <origin xyz="0.234 0.0125 0.107" rpy="0 0 0"/>
     </xacro:sensor_orbbec_astra>

File: rb1_base_description/robots/rb1_base_platform_standalone_multi.urdf.xacro (robot description, xacro)
@@ -66,26 +66,26 @@
 	</xacro:omni_wheel>
 	<!-- SENSORS -->
-	<!-- xacro:sensor_hokuyo_utm30lx name="hokuyo" parent="base_link">
+	<!-- xacro:sensor_hokuyo_utm30lx prefix="hokuyo" parent="base_link">
 		<origin xyz="0.210 0.0 0.305" rpy="0 0 0"/>
 	</xacro:sensor_hokuyo_utm30lx -->
-    <!-- xacro:sensor_hokuyo_urg04lx name="hokuyo1" parent="base_link">
+    <!-- xacro:sensor_hokuyo_urg04lx prefix="hokuyo1" parent="base_link">
         <origin xyz="0.220 0.0 0.170" rpy="0 3.1416 3.1416"/>
     </xacro:sensor_hokuyo_urg04lx -->
-	<!-- xacro:sensor_hokuyo_ust10lx name="hokuyo" parent="base_link">
+	<!-- xacro:sensor_hokuyo_ust10lx prefix="hokuyo" parent="base_link">
 		<origin xyz="0.223 0.0 0.159" rpy="0 0 0"/>
 	</xacro:sensor_hokuyo_ust10lx -->
-	<xacro:sensor_hokuyo_ust10lx name="hokuyo" parent="base_link">
+	<xacro:sensor_hokuyo_ust10lx prefix="hokuyo" parent="base_link">
 		<origin xyz="0.223 0.0 0.159" rpy="0 3.1416 3.1416"/>
 	</xacro:sensor_hokuyo_ust10lx>
-	<xacro:sensor_imu name="imu" parent="base_link">
+	<xacro:sensor_imu prefix="imu" parent="base_link">
 		<origin xyz="-0.18 0.0 0.170" rpy="0 0 0"/>
 	</xacro:sensor_imu>
-    <!-- xacro:sensor_orbbec_astra name="orbbec_astra" parent="base_link">
+    <!-- xacro:sensor_orbbec_astra prefix="orbbec_astra" parent="base_link">
         <origin xyz="0.234 0.0125 0.107" rpy="0 0 0"/>
     </xacro:sensor_orbbec_astra -->
-    <xacro:sensor_orbbec_astra name="orbbec_astra" parent="base_link">
+    <xacro:sensor_orbbec_astra prefix="orbbec_astra" parent="base_link">
         <origin xyz="0.234 0.0125 0.107" rpy="0 0 0"/>
     </xacro:sensor_orbbec_astra>
-    <!-- xacro:sensor_kinect name="kinect" parent="base_link">
+    <!-- xacro:sensor_kinect prefix="kinect" parent="base_link">
         <origin xyz="0.6 0.0 0.102" rpy="0 0 0"/>
     </xacro:sensor_kinect -->

File: rb1_base_description/robots/rb1_base_platform_v2.urdf.xacro (robot description, xacro)
@@ -57,18 +57,18 @@
 	</xacro:omni_wheel>
 	<!-- SENSORS -->
-	<!-- xacro:sensor_hokuyo_utm30lx name="hokuyo" parent="base_link">
+	<!-- xacro:sensor_hokuyo_utm30lx prefix="hokuyo" parent="base_link">
 		<origin xyz="0.210 0.0 0.305" rpy="0 0 0"/>
 	</xacro:sensor_hokuyo_utm30lx -->
-    <!-- xacro:sensor_hokuyo_urg04lx name="hokuyo" parent="base_link">
+    <!-- xacro:sensor_hokuyo_urg04lx prefix="hokuyo" parent="base_link">
         <origin xyz="0.223 0.0 0.209" rpy="0 3.1416 3.1416"/>
     </xacro:sensor_hokuyo_urg04lx -->
-	<xacro:sensor_hokuyo_ust10lx name="hokuyo" parent="base_link">
+	<xacro:sensor_hokuyo_ust10lx prefix="hokuyo" parent="base_link">
 		<origin xyz="0.220 0.0 0.216" rpy="0 3.1416 3.1416"/>
 	</xacro:sensor_hokuyo_ust10lx>
-	<xacro:sensor_imu name="imu" parent="base_link">
+	<xacro:sensor_imu prefix="imu" parent="base_link">
 		<origin xyz="0.002 0.053 0.1485" rpy="0 0 0"/>
 	</xacro:sensor_imu>
 <!--
-    <xacro:sensor_kinect name="kinect" parent="base_link">
+    <xacro:sensor_kinect prefix="kinect" parent="base_link">
         <origin xyz="0.3 0.0 0.16" rpy="0 0 0"/>
     </xacro:sensor_kinect>

File: rb1_base_description/robots/rb1_base_platform_v3.urdf.xacro (robot description, xacro)
@@ -60,8 +60,8 @@
 		<origin xyz="0.220 0.0 0.1686" rpy="0 3.1416 3.1416"/>
 	</xacro:sensor_sick_tim551>
-	<xacro:sensor_imu name="imu" parent="base_link">
+	<xacro:sensor_imu prefix="imu" parent="base_link">
 		<origin xyz="0.002 0.053 0.1485" rpy="0 0 0"/>
 	</xacro:sensor_imu>
-    	<xacro:sensor_orbbec_astra name="front_camera" parent="base_link">
+    	<xacro:sensor_orbbec_astra prefix="front_camera" parent="base_link">
         	<origin xyz="0.234 0.0125 0.1055" rpy="0 0 0"/>
     	</xacro:sensor_orbbec_astra>

File: rb1_base_description/robots/rb1_base_v0.urdf.xacro (robot description, xacro)
@@ -59,27 +59,27 @@
 	<!-- SENSORS -->
 	<!-- LASER -->
-	<!-- xacro:sensor_hokuyo_utm30lx name="front_laser" parent="base_link">
+	<!-- xacro:sensor_hokuyo_utm30lx prefix="front_laser" parent="base_link">
 		<origin xyz="0.210 0.0 0.305" rpy="0 0 0"/>
 	</xacro:sensor_hokuyo_utm30lx -->
-	<!-- xacro:sensor_hokuyo_urg04lx name="front_laser" parent="base_link">
+	<!-- xacro:sensor_hokuyo_urg04lx prefix="front_laser" parent="base_link">
 		<origin xyz="0.220 0.0 0.170" rpy="0 3.1416 3.1416"/>
 	</xacro:sensor_hokuyo_urg04lx -->
-	<!-- xacro:sensor_hokuyo_ust10lx name="front_laser" parent="base_link">
+	<!-- xacro:sensor_hokuyo_ust10lx prefix="front_laser" parent="base_link">
 		<origin xyz="0.223 0.0 0.159" rpy="0 0 0"/>
 	</xacro:sensor_hokuyo_ust10lx -->
 	<!-- Name the components as base_front_laser or base_laser or front_laser or
 	a name which identify uniquely the component within the robot -->
-	<!--xacro:sensor_rplidar_a2 name="base_front_laser" parent="base_link">
+	<!--xacro:sensor_rplidar_a2 prefix="base_front_laser" parent="base_link">
 		<origin xyz="0.210 0.0 0.199" rpy="3.1415 0 0"/>
 	</xacro:sensor_rplidar_a2-->
 	<!-- CAMERA -->
-	<!--xacro:sensor_orbbec_astra name="base_front_camera" parent="base_link">
+	<!--xacro:sensor_orbbec_astra prefix="base_front_camera" parent="base_link">
 		<origin xyz="0.234 0.0125 0.107" rpy="0 0 0"/>
 	</xacro:sensor_orbbec_astra-->
-	<!-- xacro:sensor_kinect name="front_camera" parent="base_link">
+	<!-- xacro:sensor_kinect prefix="front_camera" parent="base_link">
 		<origin xyz="0.6 0.0 0.102" rpy="0 0 0"/>
 	</xacro:sensor_kinect -->
 	<!-- IMU -->
-	<xacro:sensor_imu name="imu" parent="base_link">
+	<xacro:sensor_imu prefix="imu" parent="base_link">
 		<origin xyz="-0.18 0.0 0.170" rpy="0 0 0"/>
 	</xacro:sensor_imu>

File: rb1_base_description/robots/rb1_base_v1.urdf.xacro (robot description, xacro)
@@ -59,27 +59,27 @@
 	<!-- SENSORS -->
 	<!-- LASER -->
-	<!-- xacro:sensor_hokuyo_utm30lx name="front_laser" parent="base_link">
+	<!-- xacro:sensor_hokuyo_utm30lx prefix="front_laser" parent="base_link">
 		<origin xyz="0.210 0.0 0.305" rpy="0 0 0"/>
 	</xacro:sensor_hokuyo_utm30lx -->
-	<!-- xacro:sensor_hokuyo_urg04lx name="front_laser" parent="base_link">
+	<!-- xacro:sensor_hokuyo_urg04lx prefix="front_laser" parent="base_link">
 		<origin xyz="0.220 0.0 0.170" rpy="0 3.1416 3.1416"/>
 	</xacro:sensor_hokuyo_urg04lx -->
-	<!-- xacro:sensor_hokuyo_ust10lx name="front_laser" parent="base_link">
+	<!-- xacro:sensor_hokuyo_ust10lx prefix="front_laser" parent="base_link">
 		<origin xyz="0.223 0.0 0.159" rpy="0 0 0"/>
 	</xacro:sensor_hokuyo_ust10lx -->
 	<!-- Name the components as base_front_laser or base_laser or front_laser or
 	a name which identify uniquely the component within the robot -->
-	<xacro:sensor_rplidar_a2 name="base_front_laser" parent="base_link">
+	<xacro:sensor_rplidar_a2 prefix="base_front_laser" parent="base_link">
 		<origin xyz="0.210 0.0 0.199" rpy="3.1415 0 0"/>
 	</xacro:sensor_rplidar_a2>
 	<!-- CAMERA -->
-	<!--xacro:sensor_orbbec_astra name="base_front_camera" parent="base_link">
+	<!--xacro:sensor_orbbec_astra prefix="base_front_camera" parent="base_link">
 		<origin xyz="0.234 0.0125 0.107" rpy="0 0 0"/>
 	</xacro:sensor_orbbec_astra-->
-	<!-- xacro:sensor_kinect name="front_camera" parent="base_link">
+	<!-- xacro:sensor_kinect prefix="front_camera" parent="base_link">
 		<origin xyz="0.6 0.0 0.102" rpy="0 0 0"/>
 	</xacro:sensor_kinect -->
 	<!-- IMU -->
-	<xacro:sensor_imu name="imu" parent="base_link">
+	<xacro:sensor_imu prefix="imu" parent="base_link">
 		<origin xyz="-0.18 0.0 0.170" rpy="0 0 0"/>
 	</xacro:sensor_imu>

File: rb1_base_description/robots/rb1_base_v2.urdf.xacro (robot description, xacro)
@@ -61,27 +61,27 @@
 	<!-- SENSORS -->
 	<!-- LASER -->
-	<!-- xacro:sensor_hokuyo_utm30lx name="base_front_laser" parent="base_link">
+	<!-- xacro:sensor_hokuyo_utm30lx prefix="base_front_laser" parent="base_link">
 		<origin xyz="0.210 0.0 0.305" rpy="0 0 0"/>
 	</xacro:sensor_hokuyo_utm30lx -->
-	<!-- xacro:sensor_hokuyo_urg04lx name="base_front_laser" parent="base_link">
+	<!-- xacro:sensor_hokuyo_urg04lx prefix="base_front_laser" parent="base_link">
 		<origin xyz="0.220 0.0 0.170" rpy="0 3.1416 3.1416"/>
 	</xacro:sensor_hokuyo_urg04lx -->
-	<xacro:sensor_hokuyo_ust10lx name="base_front_laser" parent="base_link">
+	<xacro:sensor_hokuyo_ust10lx prefix="base_front_laser" parent="base_link">
 		<origin xyz="0.223 0.0 0.159" rpy="3.1416 0 0"/>
 	</xacro:sensor_hokuyo_ust10lx>
 	<!-- Name the components as base_front_laser or base_laser or front_laser or
 	a name which identify uniquely the component within the robot -->
-	<!--xacro:sensor_rplidar_a2 name="base_front_laser" parent="base_link">
+	<!--xacro:sensor_rplidar_a2 prefix="base_front_laser" parent="base_link">
 		<origin xyz="0.210 0.0 0.199" rpy="3.1415 0 0"/>
 	</xacro:sensor_rplidar_a2-->
 	<!-- CAMERA -->
-	<xacro:sensor_orbbec_astra name="base_front_camera" parent="base_link">
+	<xacro:sensor_orbbec_astra prefix="base_front_camera" parent="base_link">
 		<origin xyz="0.234 0.0125 0.107" rpy="0 0 0"/>
 	</xacro:sensor_orbbec_astra>
-	<!-- xacro:sensor_kinect name="base_front_camera" parent="base_link">
+	<!-- xacro:sensor_kinect prefix="base_front_camera" parent="base_link">
 		<origin xyz="0.6 0.0 0.102" rpy="0 0 0"/>
 	</xacro:sensor_kinect -->
 	<!-- IMU -->
-	<xacro:sensor_imu name="imu" parent="base_link">
+	<xacro:sensor_imu prefix="imu" parent="base_link">
 		<origin xyz="-0.18 0.0 0.170" rpy="0 0 0"/>
 	</xacro:sensor_imu>

File: rb1_base_description/robots/rb1_base_v2_elevator.urdf.xacro (robot description, xacro)
@@ -71,27 +71,27 @@
 	<!-- SENSORS -->
 	<!-- LASER -->
-	<!-- xacro:sensor_hokuyo_utm30lx name="front_laser" parent="base_link">
+	<!-- xacro:sensor_hokuyo_utm30lx prefix="front_laser" parent="base_link">
 		<origin xyz="0.210 0.0 0.305" rpy="0 0 0"/>
 	</xacro:sensor_hokuyo_utm30lx -->
-	<!-- xacro:sensor_hokuyo_urg04lx name="front_laser" parent="base_link">
+	<!-- xacro:sensor_hokuyo_urg04lx prefix="front_laser" parent="base_link">
 		<origin xyz="0.220 0.0 0.170" rpy="0 3.1416 3.1416"/>
 	</xacro:sensor_hokuyo_urg04lx -->
-	<!-- xacro:sensor_hokuyo_ust10lx name="front_laser" parent="base_link">
+	<!-- xacro:sensor_hokuyo_ust10lx prefix="front_laser" parent="base_link">
 		<origin xyz="0.223 0.0 0.159" rpy="0 0 0"/>
 	</xacro:sensor_hokuyo_ust10lx -->
 	<!-- Name the components as base_front_laser or base_laser or front_laser or
 	a name which identify uniquely the component within the robot -->
-	<xacro:sensor_rplidar_a2 name="base_front_laser" parent="base_link">
+	<xacro:sensor_rplidar_a2 prefix="base_front_laser" parent="base_link">
 		<origin xyz="0.210 0.0 0.199" rpy="3.1415 0 0"/>
 	</xacro:sensor_rplidar_a2>
 	<!-- CAMERA -->
-	<!--xacro:sensor_orbbec_astra name="base_front_camera" parent="base_link">
+	<!--xacro:sensor_orbbec_astra prefix="base_front_camera" parent="base_link">
 		<origin xyz="0.234 0.0125 0.107" rpy="0 0 0"/>
 	</xacro:sensor_orbbec_astra-->
-	<!-- xacro:sensor_kinect name="front_camera" parent="base_link">
+	<!-- xacro:sensor_kinect prefix="front_camera" parent="base_link">
 		<origin xyz="0.6 0.0 0.102" rpy="0 0 0"/>
 	</xacro:sensor_kinect -->
 	<!-- IMU -->
-	<xacro:sensor_imu name="imu" parent="base_link">
+	<xacro:sensor_imu prefix="imu" parent="base_link">
 		<origin xyz="-0.18 0.0 0.170" rpy="0 0 0"/>
 	</xacro:sensor_imu>

File: rb1_base_description/robots/rb1_base_v3.urdf.xacro (robot description, xacro)
@@ -59,27 +59,27 @@
 	<!-- SENSORS -->
 	<!-- LASER -->
-	<!-- xacro:sensor_hokuyo_utm30lx name="front_laser" parent="base_link">
+	<!-- xacro:sensor_hokuyo_utm30lx prefix="front_laser" parent="base_link">
 		<origin xyz="0.210 0.0 0.305" rpy="0 0 0"/>
 	</xacro:sensor_hokuyo_utm30lx -->
-	<!-- xacro:sensor_hokuyo_urg04lx name="front_laser" parent="base_link">
+	<!-- xacro:sensor_hokuyo_urg04lx prefix="front_laser" parent="base_link">
 		<origin xyz="0.220 0.0 0.170" rpy="0 3.1416 3.1416"/>
 	</xacro:sensor_hokuyo_urg04lx -->
-	<!-- xacro:sensor_hokuyo_ust10lx name="front_laser" parent="base_link">
+	<!-- xacro:sensor_hokuyo_ust10lx prefix="front_laser" parent="base_link">
 		<origin xyz="0.223 0.0 0.159" rpy="0 0 0"/>
 	</xacro:sensor_hokuyo_ust10lx -->
 	<!-- Name the components as base_front_laser or base_laser or front_laser or
 	a name which identify uniquely the component within the robot -->
-	<xacro:sensor_rplidar_a2 name="base_front_laser" parent="base_link">
+	<xacro:sensor_rplidar_a2 prefix="base_front_laser" parent="base_link">
 		<origin xyz="0.210 0.0 0.199" rpy="3.1415 0 0"/>
 	</xacro:sensor_rplidar_a2>
 	<!-- CAMERA -->
-	<!--xacro:sensor_orbbec_astra name="base_front_camera" parent="base_link">
+	<!--xacro:sensor_orbbec_astra prefix="base_front_camera" parent="base_link">
 		<origin xyz="0.234 0.0125 0.107" rpy="0 0 0"/>
 	</xacro:sensor_orbbec_astra-->
-	<!-- xacro:sensor_kinect name="front_camera" parent="base_link">
+	<!-- xacro:sensor_kinect prefix="front_camera" parent="base_link">
 		<origin xyz="0.6 0.0 0.102" rpy="0 0 0"/>
 	</xacro:sensor_kinect -->
 	<!-- IMU -->
-	<xacro:sensor_imu name="imu" parent="base_link">
+	<xacro:sensor_imu prefix="imu" parent="base_link">
 		<origin xyz="-0.18 0.0 0.170" rpy="0 0 0"/>
 	</xacro:sensor_imu>

File: rb1_base_description/urdf/bases/rb1_base.urdf.xacro (robot description, xacro)
@@ -45,5 +45,5 @@
     </visual>
     <collision>
-       <origin xyz="0 0 0" rpy="0 0 0 " />
+       <origin xyz="0 0 0" rpy="0 0 0" />
        <geometry>
          <mesh filename="package://rb1_base_description/meshes/bases/rb1v2_base.dae"/>
@@ -52,5 +52,5 @@
   </link>
   <joint name="front_cover_joint" type="fixed">
-     <origin xyz="0.220 0.0 0.004" rpy="0 0 0 " />
+     <origin xyz="0.220 0.0 0.004" rpy="0 0 0" />
      <parent link="base_link"/>
      <child link="front_cover_link" />
@@ -80,5 +80,5 @@
     </visual>
     <collision>
-       <origin xyz="0 0 0" rpy="0 0 0 " />
+       <origin xyz="0 0 0" rpy="0 0 0" />
        <geometry>
          <mesh filename="package://rb1_base_description/meshes/bases/rb1v2_front_cover.dae"/>
@@ -88,5 +88,5 @@
   <!-- DOCKING CONTACTS -->
   <joint name="base_docking_joint" type="fixed">
-     <origin xyz="0.030 0.000 0.068" rpy="0 0 0 " />
+     <origin xyz="0.030 0.000 0.068" rpy="0 0 0" />
      <parent link="front_cover_link"/>
      <child link="base_docking_contact" />

File: rb1_base_description/urdf/bases/rb1_base_v0.urdf.xacro (robot description, xacro)
@@ -45,5 +45,5 @@
     </visual>
     <collision>
-       <origin xyz="0 0 0" rpy="0 0 0 " />
+       <origin xyz="0 0 0" rpy="0 0 0" />
        <geometry>
          <mesh filename="package://rb1_base_description/meshes/bases/rb1v0_base.dae"/>

File: rb1_base_description/urdf/bases/rb1_base_v1.urdf.xacro (robot description, xacro)
@@ -45,5 +45,5 @@
     </visual>
     <collision>
-       <origin xyz="0 0 0" rpy="0 0 0 " />
+       <origin xyz="0 0 0" rpy="0 0 0" />
        <geometry>
          <mesh filename="package://rb1_base_description/meshes/bases/rb1v1_base.dae"/>

File: rb1_base_description/urdf/bases/rb1_base_v2.urdf.xacro (robot description, xacro)
@@ -45,5 +45,5 @@
     </visual>
     <collision>
-       <origin xyz="0 0 0" rpy="0 0 0 " />
+       <origin xyz="0 0 0" rpy="0 0 0" />
        <geometry>
          <mesh filename="package://rb1_base_description/meshes/bases/rb1v2_base.dae"/>
@@ -52,5 +52,5 @@
   </link>
   <joint name="front_cover_joint" type="fixed">
-     <origin xyz="0.220 0.0 0.004" rpy="0 0 0 " />
+     <origin xyz="0.220 0.0 0.004" rpy="0 0 0" />
      <parent link="base_link"/>
      <child link="front_cover_link" />
@@ -80,5 +80,5 @@
     </visual>
     <collision>
-       <origin xyz="0 0 0" rpy="0 0 0 " />
+       <origin xyz="0 0 0" rpy="0 0 0" />
        <geometry>
          <mesh filename="package://rb1_base_description/meshes/bases/rb1v2_front_cover.dae"/>
@@ -88,5 +88,5 @@
   <!-- DOCKING CONTACTS -->
   <joint name="base_docking_joint" type="fixed">
-     <origin xyz="0.030 0.000 0.068" rpy="0 0 0 " />
+     <origin xyz="0.030 0.000 0.068" rpy="0 0 0" />
      <parent link="front_cover_link"/>
      <child link="base_docking_contact" />
