Commit message: rb1_base_description: updated sensor parameters in urdf

File: rb1_base_description/urdf/bases/rb1_base_v3.urdf.xacro (robot description, xacro)
@@ -45,5 +45,5 @@
     </visual>
     <collision>
-       <origin xyz="0 0 0" rpy="0 0 0 " />
+       <origin xyz="0 0 0" rpy="0 0 0" />
        <geometry>
          <mesh filename="package://rb1_base_description/meshes/bases/rb1_base_v3.stl"/>
@@ -52,5 +52,5 @@
   </link>
   <joint name="front_cover_joint" type="fixed">
-     <origin xyz="0.220 0.0 0.004" rpy="0 0 0 " />
+     <origin xyz="0.220 0.0 0.004" rpy="0 0 0" />
      <parent link="base_link"/>
      <child link="front_cover_link" />
@@ -80,5 +80,5 @@
     </visual>
     <collision>
-       <origin xyz="0 0 0" rpy="0 0 0 " />
+       <origin xyz="0 0 0" rpy="0 0 0" />
        <geometry>
          <mesh filename="package://rb1_base_description/meshes/bases/rb1_front_cover_v3.stl"/>
@@ -87,5 +87,5 @@
   </link>
   <joint name="top_covert_joint" type="fixed">
-     <origin xyz="0.0 0.0 0.243" rpy="0 0 0 " />
+     <origin xyz="0.0 0.0 0.243" rpy="0 0 0" />
      <parent link="base_footprint"/>
      <child link="top_cover_link" />
@@ -115,5 +115,5 @@
     </visual>
     <collision>
-       <origin xyz="0 0 0" rpy="0 0 0 " />
+       <origin xyz="0 0 0" rpy="0 0 0" />
        <geometry>
          <mesh filename="package://rb1_base_description/meshes/bases/rb1_top_cover_v3.stl"/>
@@ -123,5 +123,5 @@
   <!-- DOCKING CONTACTS -->
   <joint name="base_docking_joint" type="fixed">
-     <origin xyz="0.030 0.000 0.068" rpy="0 0 0 " />
+     <origin xyz="0.030 0.000 0.068" rpy="0 0 0" />
      <parent link="front_cover_link"/>
      <child link="base_docking_contact" />

File: rb1_base_description/urdf/elevator/elevator.urdf.xacro (robot description, xacro)
@@ -37,5 +37,5 @@
 		</visual>
 		<collision>
-			<origin xyz="0 0 0" rpy="0 0 0 " />
+			<origin xyz="0 0 0" rpy="0 0 0" />
 			<geometry>
 				<mesh filename="package://rb1_base_description/meshes/elevator/rb1_elevator_base.dae"/>
@@ -45,5 +45,5 @@
 	<!-- ELEVATOR PLATFORM -->
 	<joint name="elevator_platform_joint" type="prismatic">
-			<origin xyz="0.0 0.0 0.041" rpy="0 0 0 " />
+			<origin xyz="0.0 0.0 0.041" rpy="0 0 0" />
 			<parent link="elevator_base_link"/>
 			<child link="elevator_platform_link" />
@@ -74,5 +74,5 @@
 		</visual>
 		<collision>
-			<origin xyz="0 0 0" rpy="0 0 0 " />
+			<origin xyz="0 0 0" rpy="0 0 0" />
 			<geometry>
 				<mesh filename="package://rb1_base_description/meshes/elevator/rb1_elevator_platform.dae"/>

File: rb1_base_description/urdf/inertia.urdf.xacro (robot description, xacro)
@@ -4,6 +4,6 @@
   <!-- TODO Solid sphere of radius r and mass m-->
   <xacro:macro name="solid_sphere_inertia" params="m r">
-    <inertia  ixx="${(2*r*r*m)/5}" ixy = "0" ixz = "0"
-              iyy="${(2*r*r*m)/5}" iyz = "0"
+    <inertia  ixx="${(2*r*r*m)/5}" ixy="0" ixz="0"
+              iyy="${(2*r*r*m)/5}" iyz="0"
               izz="${(2*r*r*m)/5}"
      />
@@ -11,6 +11,6 @@
   <!-- TODO Hollow sphere of radius r and mass m-->
   <xacro:macro name="solid_sphere_inertia" params="m r">
-    <inertia  ixx="${(2*r*r*m)/3}" ixy = "0" ixz = "0"
-              iyy="${(2*r*r*m)/3}" iyz = "0"
+    <inertia  ixx="${(2*r*r*m)/3}" ixy="0" ixz="0"
+              iyy="${(2*r*r*m)/3}" iyz="0"
               izz="${(2*r*r*m)/3}"
      />
@@ -18,6 +18,6 @@
   <!-- TODO Solid ellipsoid of semi-axes a, b, c and mass m-->
   <xacro:macro name="ellipsoid_semi_axes_inertia" params="a b c m r">
-    <inertia  ixx="${(m*(b*b+c*c))/5}" ixy = "0" ixz = "0"
-              iyy="${(m*(a*a+c*c))/5}" iyz = "0"
+    <inertia  ixx="${(m*(b*b+c*c))/5}" ixy="0" ixz="0"
+              iyy="${(m*(a*a+c*c))/5}" iyz="0"
               izz="${(m*(a*a+b*b))/5}"
      />
@@ -25,6 +25,6 @@
   <!-- TODO Right circular cone with radius r, height h and mass m, about the apex -->
   <xacro:macro name="right_circular_cone_inertia" params="m r h">
-    <inertia  ixx="${((3*m*(h*h))/5)+((3*m*(r*r))/20)}" ixy = "0" ixz = "0"
-              iyy="${((3*m*(h*h))/5)+((3*m*(r*r))/20)}" iyz = "0"
+    <inertia  ixx="${((3*m*(h*h))/5)+((3*m*(r*r))/20)}" ixy="0" ixz="0"
+              iyy="${((3*m*(h*h))/5)+((3*m*(r*r))/20)}" iyz="0"
               izz="${(3*m*(r*r))/10}"
      />
@@ -32,6 +32,6 @@
   <!-- TODO Solid cuboid of width w, height h, depth d, and mass m -->
   <xacro:macro name="solid_cuboid_inertia" params="m h d w">
-    <inertia  ixx="${(m*(h*h+d*d))/12}" ixy = "0" ixz = "0"
-              iyy="${(m*(w*w+d*d))/12}" iyz = "0"
+    <inertia  ixx="${(m*(h*h+d*d))/12}" ixy="0" ixz="0"
+              iyy="${(m*(w*w+d*d))/12}" iyz="0"
               izz="${(m*(w*w+h*h))/12}"
      />
@@ -39,6 +39,6 @@
   <!-- TODO Solid cylinder of radius r, height h and mass m -->
   <xacro:macro name="solid_cylinder_inertia" params="m r h">
-    <inertia  ixx="${m*(3*r*r+h*h)/12}" ixy = "0" ixz = "0"
-              iyy="${m*(3*r*r+h*h)/12}" iyz = "0"
+    <inertia  ixx="${m*(3*r*r+h*h)/12}" ixy="0" ixz="0"
+              iyy="${m*(3*r*r+h*h)/12}" iyz="0"
               izz="${m*r*r/2}"
      />
@@ -46,6 +46,6 @@
     <!-- TODO Thick-walled cylindrical tube with open ends, of inner radius r1, outer radius r2, length h and mass m -->
     <xacro:macro name="thick_walled_cylinder_inertia" params="m r1 r2 h">
-    <inertia  ixx="${m*((3*(r1*r1+r2*r2))+(h*h))/12}" ixy = "0" ixz = "0"
-              iyy="${m*((3*(r1*r1+r2*r2))+(h*h))/12}" iyz = "0"
+    <inertia  ixx="${m*((3*(r1*r1+r2*r2))+(h*h))/12}" ixy="0" ixz="0"
+              iyy="${m*((3*(r1*r1+r2*r2))+(h*h))/12}" iyz="0"
               izz="${m*(r1*r1+r2*r2)/2}"
      />

File: rb1_base_description/urdf/rb1_base.urdf.xacro (robot description, xacro)
@@ -70,27 +70,27 @@
 		<!-- SENSORS -->
 		<!-- LASER -->
-		<!-- xacro:sensor_hokuyo_utm30lx name="front_laser" parent="base_link">
+		<!-- xacro:sensor_hokuyo_utm30lx prefix="front_laser" parent="base_link">
 			<origin xyz="0.210 0.0 0.305" rpy="0 0 0"/>
 		</xacro:sensor_hokuyo_utm30lx -->
-		<!-- xacro:sensor_hokuyo_urg04lx name="front_laser" parent="base_link">
+		<!-- xacro:sensor_hokuyo_urg04lx prefix="front_laser" parent="base_link">
 			<origin xyz="0.220 0.0 0.170" rpy="0 3.1416 3.1416"/>
 		</xacro:sensor_hokuyo_urg04lx -->
-		<!-- xacro:sensor_hokuyo_ust10lx name="front_laser" parent="base_link">
+		<!-- xacro:sensor_hokuyo_ust10lx prefix="front_laser" parent="base_link">
 			<origin xyz="0.223 0.0 0.159" rpy="0 0 0"/>
 		</xacro:sensor_hokuyo_ust10lx -->
 		<!-- Name the components as base_front_laser or base_laser or front_laser or
 		a name which identify uniquely the component within the robot -->
-		<xacro:sensor_rplidar_a2 name="base_front_laser" parent="base_link">
+		<xacro:sensor_rplidar_a2 prefix="base_front_laser" parent="base_link">
 			<origin xyz="0.210 0.0 0.199" rpy="3.1415 0 0"/>
 		</xacro:sensor_rplidar_a2>
 		<!-- CAMERA -->
-		<!--xacro:sensor_orbbec_astra name="base_front_camera" parent="base_link">
+		<!--xacro:sensor_orbbec_astra prefix="base_front_camera" parent="base_link">
 			<origin xyz="0.234 0.0125 0.107" rpy="0 0 0"/>
 		</xacro:sensor_orbbec_astra-->
-		<!-- xacro:sensor_kinect name="front_camera" parent="base_link">
+		<!-- xacro:sensor_kinect prefix="front_camera" parent="base_link">
 			<origin xyz="0.6 0.0 0.102" rpy="0 0 0"/>
 		</xacro:sensor_kinect -->
 		<!-- IMU -->
-		<xacro:sensor_imu name="imu" parent="base_link">
+		<xacro:sensor_imu prefix="imu" parent="base_link">
 			<origin xyz="-0.18 0.0 0.170" rpy="0 0 0"/>
 		</xacro:sensor_imu>

File: rb1_base_description/urdf/wheels/omni_wheel.urdf.xacro (robot description, xacro)
@@ -7,6 +7,6 @@
   <xacro:property name="omni_wheel_mass" value="0.3" /> <!-- in kg-->
   <xacro:macro name="cylinder_inertia" params="m r h">
-    <inertia  ixx="${m*(3*r*r+h*h)/12}" ixy = "0" ixz = "0"
-              iyy="${m*(3*r*r+h*h)/12}" iyz = "0"
+    <inertia  ixx="${m*(3*r*r+h*h)/12}" ixy="0" ixz="0"
+              iyy="${m*(3*r*r+h*h)/12}" iyz="0"
               izz="${m*r*r/2}"
      />
