Commit message: rb1_base_description: fixing last push errors and eliminating anoying warnings

File: rb1_base_description/robots/rb1_base_platform_kinova.urdf.xacro (robot description, xacro)
@@ -6,7 +6,4 @@
 	<!-- First we import all posible elements defined in the urdf.xacro files. All these elements are defined as macro:xacros -->
 	<!-- Import RB1 base elements -->
-<<<<<<< HEAD:rb1_base_description/robots/rb1_base_platform_standalone.urdf.xacro
-    	<xacro:include filename="$(find rb1_base_description)/urdf/bases/rb1_base.urdf.xacro" />
-=======
     <xacro:include filename="$(find rb1_base_description)/urdf/bases/rb1_base.urdf.xacro" />
     <xacro:include filename="$(find rb1_base_description)/urdf/others/kinova_base.urdf.xacro" />
@@ -19,5 +16,4 @@
       </plugin>
     </gazebo>
->>>>>>> indigo-devel:rb1_base_description/robots/rb1_base_platform_kinova.urdf.xacro
 	<!-- Import RB1 wheels -->
 	<xacro:include filename="$(find rb1_base_description)/urdf/wheels/rubber_wheel.urdf.xacro" />
@@ -85,9 +81,4 @@
 		<origin xyz="-0.18 0.0 0.170" rpy="0 0 0"/>
 	</xacro:sensor_imu>
-<<<<<<< HEAD:rb1_base_description/robots/rb1_base_platform_standalone.urdf.xacro
-	<xacro:sensor_orbbec_astra name="orbbec_astra" parent="base_link">
-		<origin xyz="0.234 0.0125 0.107" rpy="0 0 0"/>
-	</xacro:sensor_orbbec_astra>
-=======
     <!-- xacro:sensor_orbbec_astra name="orbbec_astra" parent="base_link">
         <origin xyz="0.234 0.0125 0.107" rpy="0 0 0"/>
@@ -102,4 +93,3 @@
         <origin xyz="0.6 0.0 0.102" rpy="0 0 0"/>
     </xacro:sensor_kinect -->
->>>>>>> indigo-devel:rb1_base_description/robots/rb1_base_platform_kinova.urdf.xacro
 </robot>

File: rb1_base_description/robots/rb1_base_v2.urdf.xacro (robot description, xacro)
@@ -39,5 +39,5 @@
 	<!-- Here we create the robot elements using the xacro:macros imported at the beggining of this file -->
 	<!-- BASE -->
-	<xacro:rb1_base_v2 name="rb1_base" publish_bf="true" hq="${hq}" />
+	<xacro:rb1_base name="rb1_base" publish_bf="true" hq="${hq}" />
 	<!-- RUBBER WHEELS -->
 	<xacro:rubber_wheel name="right" parent="base_link" reflect="false" hq="${hq}">

File: rb1_base_description/robots/rb1_base_v2_elevator.urdf.xacro (robot description, xacro)
@@ -47,5 +47,5 @@
 	<!-- Here we create the robot elements using the xacro:macros imported at the beggining of this file -->
 	<!-- BASE -->
-	<xacro:rb1_base_v2 name="rb1_base" publish_bf="true" hq="${hq}" />
+	<xacro:rb1_base name="rb1_base" publish_bf="true" hq="${hq}" />
 	<!-- RUBBER WHEELS -->
 	<xacro:rubber_wheel name="right" parent="base_link" reflect="false" hq="${hq}">

File: rb1_base_description/urdf/bases/rb1_base.gazebo.xacro (robot description, xacro)
@@ -1,51 +1,4 @@
 <?xml version="1.0"?>
-<robot xmlns:xacro="http://ros.org/wiki/xacro">
-<<<<<<< HEAD
-  <!-- ros control plugin -->
-  <xacro:macro name="ros_control">
-    <gazebo>
-      <plugin name="ros_control" filename="libgazebo_ros_control.so">
-        <robotNamespace>/rb1</robotNamespace>
-        <robotParam>robot_description</robotParam>
-        <controlPeriod>0.001</controlPeriod>
-	    <robotSimType>gazebo_ros_control/DefaultRobotHWSim</robotSimType>
-      </plugin>
-    </gazebo>
-  </xacro:macro>
-	<!-- differential drive plugin -->
-	<xacro:macro name="diff_drive">
-    <gazebo>
-	<plugin name="differential_drive_controller" filename="libgazebo_ros_diff_drive.so">
-	    <alwaysOn>true</alwaysOn>
-        <updateRate>50.0</updateRate>
-        <!--leftJoint>joint_left_wheel</leftJoint>
-        <rightJoint>joint_right_wheel</rightJoint-->
-        <leftJoint>joint_right_wheel</leftJoint>
-        <rightJoint>joint_left_wheel</rightJoint>
-		<!-- For V0 0.365 -->
-        <!-- wheelSeparation>0.365</wheelSeparation -->
-        <wheelSeparation>0.433</wheelSeparation>
-        <wheelDiameter>0.1524</wheelDiameter>
-        <commandTopic>/rb1/cmd_vel</commandTopic>
-        <odometryTopic>odom</odometryTopic>
-        <odometryFrame>odom</odometryFrame>
-        <robotBaseFrame>base_footprint</robotBaseFrame>
-        <!-- robotNamespace></robotNamespace -->
-        <rosDebugLevel>na</rosDebugLevel>
-        <publishWheelTF>true</publishWheelTF>
-        <publishWheelJointState>false</publishWheelJointState>
-        <wheelAcceleration>0</wheelAcceleration>
-        <wheelTorque>5</wheelTorque>
-        <!-- odometrySource>encoder</odometrySource -->
-        <odometrySource>world</odometrySource>
-        <publishTf>1</publishTf>
-	<legacyMode>false</legacyMode>
-	</plugin>
-	</gazebo>
-    </xacro:macro>
-  <gazebo reference="base_footprint">
-    <material>Gazebo/Green</material>
-  </gazebo>
-=======
+<robot xmlns:xacro="http://www.ros.org/wiki/xacro">
 	<!-- DIFFERENCIAL DRIVE GAZEBO PLUGIN -->
 	<xacro:macro name="gazebo_differencial_drive">
@@ -88,4 +41,3 @@
 		<material>Gazebo/Black</material>
 	</gazebo>
->>>>>>> indigo-devel
 </robot>

File: rb1_base_description/urdf/bases/rb1_base.urdf.xacro (robot description, xacro)
@@ -1,8 +1,4 @@
 <?xml version="1.0"?>
 <robot name="rb1_base" xmlns:xacro="http://www.ros.org/wiki/xacro">
-<<<<<<< HEAD
-  <xacro:include filename="$(find rb1_base_description)/urdf/bases/rb1_base.gazebo.xacro" />
-=======
->>>>>>> indigo-devel
   <xacro:macro name="rb1_base" params="name publish_bf hq">
   <!-- Robot mechanical and motor parameters -->

File: rb1_base_description/urdf/wheels/rubber_wheel.transmission.xacro (robot description, xacro)
@@ -1,4 +1,4 @@
 <?xml version="1.0"?>
-<robot xmlns:xacro="http://ros.org/wiki/xacro">
+<robot xmlns:xacro="http://www.ros.org/wiki/xacro">
 	<!-- Rubber wheel transmission -->
 	<xacro:macro name="rubber_wheel_transmission" params="name">

File: rb1_base_description/urdf/wheels/rubber_wheel.urdf.xacro (robot description, xacro)
@@ -3,11 +3,4 @@
 	<xacro:include filename="$(find rb1_base_description)/urdf/wheels/rubber_wheel.transmission.xacro"/>
 	<xacro:include filename="$(find rb1_base_description)/urdf/wheels/rubber_wheel.gazebo.xacro"/>
-<<<<<<< HEAD
-  <xacro:property name="M_PI" value="3.1415926535897931" />
-  <!-- Wheels -->
-  <xacro:property name="wheel_radius" value="0.076" />
-  <xacro:property name="wheel_height" value="0.025" />
-  <xacro:property name="wheel_mass" value="1.0" /> <!-- in kg-->
-=======
 	<xacro:property name="M_PI" value="3.1415926535897931" />
 	<!-- Wheels -->
@@ -15,5 +8,4 @@
 	<xacro:property name="wheel_height" value="0.025" />
 	<xacro:property name="wheel_mass" value="1.0" /> <!-- in kg-->
->>>>>>> indigo-devel
 	<xacro:macro name="cylinder_inertia" params="m r h">
 		<inertia	ixx="${m*(3*r*r+h*h)/12}" ixy = "0" ixz = "0"
@@ -22,15 +14,4 @@
 	</xacro:macro>
 	<xacro:macro name="rubber_wheel" params="name parent *origin reflect hq">
-<<<<<<< HEAD
-  <!--WHEEL TIRE -->
-    <joint name="joint_${name}_wheel" type="continuous">
-      <parent link="${parent}"/>
-      <child link="${name}_wheel"/>
-      <xacro:insert_block name="origin" />
-      <axis xyz="0 1 0" rpy="0 0 0" />
-      <limit effort="100" velocity="100"/>
-      <joint_properties damping="0.0" friction="0.0"/>
-    </joint>
-=======
 	<!--WHEEL TIRE -->
 	<joint name="${name}_wheel_joint" type="continuous">
@@ -42,5 +23,4 @@
 		<joint_properties damping="0.0" friction="0.0"/>
 	</joint>
->>>>>>> indigo-devel
 	<link name="${name}_wheel_link">
 		<visual>

Commit message: Description: Fix urdf.xacro of kinova platform

File: rb1_base_description/robots/rb1_base_platform_kinova.urdf.xacro (robot description, xacro)
@@ -6,19 +6,13 @@
 	<!-- First we import all posible elements defined in the urdf.xacro files. All these elements are defined as macro:xacros -->
 	<!-- Import RB1 base elements -->
-    <xacro:include filename="$(find rb1_base_description)/urdf/bases/rb1_base.urdf.xacro" />
+    <xacro:include filename="$(find rb1_base_description)/urdf/bases/rb1_base_v3.urdf.xacro" />
     <xacro:include filename="$(find rb1_base_description)/urdf/others/kinova_base.urdf.xacro" />
-    <gazebo>
-      <plugin name="ros_control" filename="libgazebo_ros_control.so">
-        <robotNamespace>/rb1</robotNamespace>
-        <robotParam>robot_description</robotParam>
-        <controlPeriod>0.001</controlPeriod>
-	    <robotSimType>gazebo_ros_control/DefaultRobotHWSim</robotSimType>
-      </plugin>
-    </gazebo>
 	<!-- Import RB1 wheels -->
 	<xacro:include filename="$(find rb1_base_description)/urdf/wheels/rubber_wheel.urdf.xacro" />
 	<xacro:include filename="$(find rb1_base_description)/urdf/wheels/omni_wheel.urdf.xacro" />
 	<!-- Import all available sensors -->
-    	<xacro:include filename="$(find robotnik_sensors)/urdf/all_sensors.urdf.xacro"/>
+	<xacro:include filename="$(find robotnik_sensors)/urdf/all_sensors.urdf.xacro" />
+    <!-- Import Gazebo Stuff -->
+    <xacro:include filename="$(find rb1_base_description)/urdf/common.gazebo.xacro" />
 	<!-- ***************** -->
 	<!-- Global parameters -->
@@ -27,13 +21,13 @@
 	<!-- Wheel parameters -->
 	<xacro:property name="wheel_offset_x" value="0.0" />    <!-- x,y,z in translation from base_link to the center of the wheel -->
-	<xacro:property name="wheel_offset_y" value="0.217" />
-	<xacro:property name="wheel_offset_z" value="0.051" />
+	<xacro:property name="wheel_offset_y" value="0.218" />
+	<xacro:property name="wheel_offset_z" value="0.0512" />
 	<!-- Castor paramters -->
 	<xacro:property name="omni_back_x" value="0.195" />
 	<xacro:property name="omni_back_y" value="0.0" />
-	<xacro:property name="omni_back_z" value="0.0265" />
-	<xacro:property name="omni_front_x" value="0.133" />
-	<xacro:property name="omni_front_y" value="0.148" />
-	<xacro:property name="omni_front_z" value="0.0265" />
+	<xacro:property name="omni_back_z" value="0.0270" />
+	<xacro:property name="omni_front_x" value="0.132" />
+	<xacro:property name="omni_front_y" value="0.1535" />
+	<xacro:property name="omni_front_z" value="0.0270" />
 	<!-- Flag to select the high or low quality model -->
 	<xacro:property name="hq" value="true" />
@@ -43,53 +37,38 @@
 	<!-- Here we create the robot elements using the xacro:macros imported at the beggining of this file -->
 	<!-- RB-1 base -->
-	<xacro:rb1_base name="rb1_base" publish_bf="true" hq="${hq}" />
+	<xacro:rb1_base_v3 prefix="$(arg prefix)" publish_bf="true" hq="${hq}" />
+	<xacro:arg name="prefix" default="rb1_"/>
 	<!-- Gazebo ros control plugins -->
 	<xacro:ros_control/>
-	<!-- Gazebo skid steering plugins -->
-	<xacro:diff_drive/>
+	<xacro:gazebo_colors prefix="$(arg prefix)"/>
 	<!-- WHEELS -->
-	<xacro:rubber_wheel name="right" parent="base_link" reflect="false" hq="${hq}">
+	<xacro:rubber_wheel prefix="$(arg prefix)right" parent="$(arg prefix)base_link" reflect="false" hq="${hq}">
 		<origin xyz="${wheel_offset_x} -${wheel_offset_y} ${wheel_offset_z}" rpy="0 0 0"/>
 	</xacro:rubber_wheel>
-	<xacro:rubber_wheel name="left" parent="base_link" reflect="true" hq="${hq}">
+	<xacro:rubber_wheel prefix="$(arg prefix)left" parent="$(arg prefix)base_link" reflect="true" hq="${hq}">
 		<origin xyz="${wheel_offset_x} ${wheel_offset_y} ${wheel_offset_z}" rpy="0 0 0"/>
 	</xacro:rubber_wheel>
     <!-- OMNI DIRECTIONAL WHEELS -->
-	<xacro:omni_wheel name="omni_back" parent="base_link" hq="${hq}">
+	<xacro:omni_wheel prefix="$(arg prefix)omni_back" parent="$(arg prefix)base_link" hq="${hq}">
 		<origin xyz="-${omni_back_x} ${omni_back_y} ${omni_back_z}" rpy="0 0 0"/>
 	</xacro:omni_wheel>
-	<xacro:omni_wheel name="omni_front_left" parent="base_link" hq="${hq}">
+	<xacro:omni_wheel prefix="$(arg prefix)omni_front_left" parent="$(arg prefix)base_link" hq="${hq}">
 		<origin xyz="${omni_front_x} ${omni_front_y} ${omni_front_z}" rpy="0 0 0"/>
 	</xacro:omni_wheel>
-	<xacro:omni_wheel name="omni_front_right" parent="base_link" hq="${hq}">
+	<xacro:omni_wheel prefix="$(arg prefix)omni_front_right" parent="$(arg prefix)base_link" hq="${hq}">
 		<origin xyz="${omni_front_x} -${omni_front_y} ${omni_front_z}" rpy="0 0 0"/>
 	</xacro:omni_wheel>
 	<!-- SENSORS -->
-	<!-- xacro:sensor_hokuyo_utm30lx name="hokuyo" parent="base_link">
-		<origin xyz="0.210 0.0 0.305" rpy="0 0 0"/>
-	</xacro:sensor_hokuyo_utm30lx -->
-	<!-- xacro:sensor_hokuyo_urg04lx name="hokuyo1" parent="base_link">
-		<origin xyz="0.220 0.0 0.170" rpy="0 3.1416 3.1416"/>
-	</xacro:sensor_hokuyo_urg04lx -->
-	<!-- xacro:sensor_hokuyo_ust10lx name="hokuyo" parent="base_link">
-		<origin xyz="0.223 0.0 0.159" rpy="0 0 0"/>
-	</xacro:sensor_hokuyo_ust10lx -->
-	<xacro:sensor_hokuyo_ust10lx name="hokuyo" parent="base_link">
-		<origin xyz="0.223 0.0 0.159" rpy="0 3.1416 3.1416"/>
+	<xacro:sensor_hokuyo_ust10lx prefix="$(arg prefix)front_laser" parent="$(arg prefix)base_link" prefix_topic="front_laser">
+		<origin xyz="0.210 0.0 0.159" rpy="0 3.1416 3.1416"/>
 	</xacro:sensor_hokuyo_ust10lx>
-	<xacro:sensor_imu name="imu" parent="base_link">
-		<origin xyz="-0.18 0.0 0.170" rpy="0 0 0"/>
-	</xacro:sensor_imu>
-    <!-- xacro:sensor_orbbec_astra name="orbbec_astra" parent="base_link">
-        <origin xyz="0.234 0.0125 0.107" rpy="0 0 0"/>
-    </xacro:sensor_orbbec_astra -->
-    <xacro:sensor_orbbec_astra name="orbbec_astra" parent="base_link">
+	<xacro:sensor_imu_hector prefix="$(arg prefix)imu" parent="$(arg prefix)base_link">
+		<origin xyz="0.002 0.053 0.1485" rpy="0 0 0"/>
+	</xacro:sensor_imu_hector>
+    <xacro:sensor_orbbec_astra prefix="$(arg prefix)front_rgbd_camera" parent="$(arg prefix)base_link" prefix_topic="front_rgbd_camera">
         <origin xyz="0.234 0.0125 0.107" rpy="0 0 0"/>
     </xacro:sensor_orbbec_astra>
-    <xacro:kinova_base parent="base_link" prefix="">
+    <xacro:kinova_base parent="$(arg prefix)base_link" prefix="">
         <origin xyz="0.0 0.0 0.213" rpy="0 0 0"/>
     </xacro:kinova_base>
-    <!-- xacro:sensor_kinect name="kinect" parent="base_link">
-        <origin xyz="0.6 0.0 0.102" rpy="0 0 0"/>
-    </xacro:sensor_kinect -->
 </robot>

File: rb1_base_description/robots/rb1_base_std.urdf.xacro (robot description, xacro)
@@ -40,5 +40,5 @@
 	<xacro:rb1_base_v3 prefix="$(arg prefix)" publish_bf="true" hq="${hq}" />
 	<xacro:arg name="prefix" default="rb1_"/>
-	<!-- Gazebo ros control pluggins -->
+	<!-- Gazebo ros control plugins -->
 	<xacro:ros_control/>
 	<xacro:gazebo_colors prefix="$(arg prefix)"/>
