Commit message: Add rb1_dual_ur3 MoveIt package

File: rb1_base_description/robots/rb1_dual_ur3.urdf.xacro (robot description, xacro)
@@ -85,5 +85,6 @@
 	<xacro:ur3_robot prefix="$(arg prefix)right_arm_" joint_limited="true"
 		shoulder_pan_lower_limit="${-pi}" shoulder_pan_upper_limit="${pi}"
-		wrist_3_lower_limit="${-pi}" wrist_3_upper_limit="${pi}">
+		wrist_3_lower_limit="${-pi}" wrist_3_upper_limit="${pi}"
+		kinematics_file="${load_yaml('$(find rb1_base_control)/config/ur3_calibration.yaml')}">
 	</xacro:ur3_robot>
 	<joint name="$(arg prefix)right_arm_base_joint" type="fixed">
@@ -94,5 +95,6 @@
 	<xacro:ur3_robot prefix="$(arg prefix)left_arm_" joint_limited="true"
 		shoulder_pan_lower_limit="${-pi}" shoulder_pan_upper_limit="${pi}"
-		wrist_3_lower_limit="${-pi}" wrist_3_upper_limit="${pi}">
+		wrist_3_lower_limit="${-pi}" wrist_3_upper_limit="${pi}"
+		kinematics_file="${load_yaml('$(find rb1_base_control)/config/ur3_calibration.yaml')}">
 	</xacro:ur3_robot>
 	<joint name="$(arg prefix)left_arm_base_joint" type="fixed">

File: rb1_base_description/urdf/others/torso_ur3.urdf.xacro (robot description, xacro)
@@ -33,5 +33,5 @@
       <parent link="${prefix}torso_link"/>
       <child link="${prefix}torso_ur3_right_link"/>
-      <origin xyz="0.170 -0.12625 0.95775" rpy="${pi/4} 0 0"/>
+      <origin xyz="0.170 -0.12625 0.95775" rpy="${-pi/4} 0 ${pi}"/>
     </joint>
     <link name="${prefix}torso_ur3_right_link">
