Commit message: description: setting omni wheels height (z) for rb1 with elevator at the same one than rb1 without elevator

File: rb1_base_description/robots/rb1_base_std_elevator.urdf.xacro (robot description, xacro)
@@ -27,8 +27,8 @@
 	<xacro:property name="omni_back_x" value="0.195" />
 	<xacro:property name="omni_back_y" value="0.0" />
-	<xacro:property name="omni_back_z" value="0.0258" />
+	<xacro:property name="omni_back_z" value="0.027" />
 	<xacro:property name="omni_front_x" value="0.132" />
 	<xacro:property name="omni_front_y" value="0.1535" />
-	<xacro:property name="omni_front_z" value="0.0258" />
+	<xacro:property name="omni_front_z" value="0.027" />
 	<!-- Flag to select the high or low quality model -->
 	<xacro:property name="hq" value="true" />

File: rb1_base_description/urdf/elevator/elevator.urdf.xacro (robot description, xacro)
@@ -7,4 +7,10 @@
 	<!-- name : name of the link: -->
 	<!-- hq: selects model in high quality (.dae) -->
+    <xacro:macro name="solid_cuboid_inertia" params="m h d w">
+		<inertia  ixx="${(m*(h*h+d*d))/12}" ixy = "0" ixz = "0"
+              iyy="${(m*(w*w+d*d))/12}" iyz = "0"
+              izz="${(m*(w*w+h*h))/12}"
+     />
+    </xacro:macro>
 	<!-- ELEVATOR_BASE_LINK -->
 	<joint name="${prefix}_base_joint" type="fixed">
@@ -14,10 +20,15 @@
 	</joint>
 	<link name="${prefix}_base_link">
-		<inertial>
-			<mass value="25.0" />
+		<!--inertial>
+			<mass value="0.1" />
 			<origin xyz="0 0 0" />
 			<inertia	ixx="0.007" ixy="0.0"  ixz="0.0"
 						iyy="0.007"  iyz="0.0"
 						izz="0.78125"/>
+		</inertial-->
+		<inertial>
+			<mass value="0.005" />
+			<origin xyz="0 0 -0.27" />
+			<solid_cuboid_inertia m="0.005" h="0.05" d="0.05" w="0.05"/>
 		</inertial>
 		<visual>
@@ -53,8 +64,13 @@
 	</joint>
 	<link name="${prefix}_platform_link">
-		<inertial>
+		<!--inertial>
 			<mass value="0.05" />
 			<origin xyz="0 0 0" />
 			<inertia  ixx="0.00007" ixy="0.0"  ixz="0.0"  iyy="0.00007"  iyz="0.0"  izz="0.0078" />
+		</inertial-->
+		<inertial>
+			<mass value="0.005" />
+			<origin xyz="0 0 -0.27" />
+			<solid_cuboid_inertia m="0.005" h="0.05" d="0.05" w="0.05"/>
 		</inertial>
 		<visual>

Commit message: added flash light OFF to robot model

File: rb1_base_description/robots/rb1_base_std_elevator.urdf.xacro (robot description, xacro)
@@ -16,4 +16,6 @@
     <!-- Import Elevator -->
 	<xacro:include filename="$(find rb1_base_description)/urdf/elevator/elevator.urdf.xacro"/>
+	<!-- Import Led -->
+	<xacro:include filename="$(find rb1_base_description)/urdf/others/led.urdf.xacro"/>
 	<!-- ***************** -->
 	<!-- Global parameters -->
@@ -80,3 +82,7 @@
         <origin xyz="0.234 0.0125 0.107" rpy="0 0 0"/>
     </xacro:sensor_orbbec_astra>
+    <!-- LED -->
+    <xacro:led prefix="$(arg prefix)led" parent="$(arg prefix)base_link">
+    	<origin xyz="0.0 0.0 1.4" rpy="3.14 0 0"/>
+    </xacro:led>
 </robot>

File: rb1_base_description/urdf/others/led.urdf.xacro (robot description, xacro)
@@ -1,18 +1,14 @@
 <?xml version="1.0"?>
 <robot xmlns:xacro="http://wiki.ros.org/xacro">
-  <xacro:macro name="led" params="prefix">
-  <gazebo>
-    <joint name="${prefix}led_joint" type="fixed">
-      <parent>${prefix}front_case_link</parent>
-      <child>light_model::${prefix}light_link</child>
-    </joint>
-    <model name="light_model">
-      <pose>1.5207 0 0.68 0 0 0</pose>
-      <link name="${prefix}light_link">
+<xacro:macro name="led" params="prefix parent *origin">
+<gazebo>
+   <model name='light_model'>
+      <static>1</static>
+      <link name="light_box">
         <visual name="${prefix}led_light">
-          <pose>0 0 0 0 0 0</pose>
+          <pose>0.25 0 0 0 0 0</pose>
           <geometry>
             <box>
-              <size>0.35 0.568 0.01</size>
+              <size>0.01 0.01 0.01</size>
             </box>
           </geometry>
@@ -24,17 +20,18 @@
           </material>
         </visual>
-        <light name="${prefix}led_light" type="point">
-          <pose>0 0 0 0 0 0</pose>
+        <light name='light_source' type='spot'>
+          <pose frame='${prefix}_base_link'>0.25 0 0.25 0 -1.57 0</pose>
           <attenuation>
-            <range>20</range>
-            <!--linear>0.10</linear-->
+            <range>10</range>
+            <linear>0.25</linear>
           </attenuation>
           <diffuse>0 0 0 1</diffuse>
           <specular>0 0 0 1</specular>
           <spot>
-            <inner_angle>0.1</inner_angle>
-            <outer_angle>0.15</outer_angle>
-            <falloff>1</falloff>
+            <inner_angle>2.3</inner_angle>
+            <outer_angle>2.35</outer_angle>
+            <falloff>15</falloff>
           </spot>
+          <direction>0 0 -1</direction>
         </light>
         <inertial>
@@ -49,22 +46,16 @@
             <izz>0.0001</izz>
           </inertia>
-  </inertial>
+        </inertial>
       </link>
-      <!--plugin name='light_control' filename='libLedPlugin.so'>
-       <enable>true</enable>
+      <plugin name='light_control' filename='libFlashLightPlugin.so'>
+        <enable>true</enable>
         <light>
-          <id>light_link/light_source</id>
-            <enable>true</enable>
-            <duration>1</duration>
-            <interval>0.5</interval>
-            <color>1 0 0</color>
-            <attenuation>
-               <range>20</range>
-               <linear>0.10</linear>
-            </attenuation>
+          <id>light_box/light_source</id>
+          <duration>0.75</duration>
+          <interval>0.5</interval>
         </light>
-      </plugin-->
-    </model>
-  </gazebo>
-  </xacro:macro>
+      </plugin>
+   </model>
+</gazebo>
+</xacro:macro>
 </robot>
