Commit message: description: model v3 modification in default laser, topic names

File: rb1_base_description/robots/rb1_base_std.urdf.xacro (robot description, xacro)
@@ -27,8 +27,8 @@
 	<xacro:property name="omni_back_x" value="0.195" />
 	<xacro:property name="omni_back_y" value="0.0" />
-	<xacro:property name="omni_back_z" value="0.0258" />
+	<xacro:property name="omni_back_z" value="0.0270" />
 	<xacro:property name="omni_front_x" value="0.132" />
 	<xacro:property name="omni_front_y" value="0.1535" />
-	<xacro:property name="omni_front_z" value="0.0258" />
+	<xacro:property name="omni_front_z" value="0.0270" />
 	<!-- Flag to select the high or low quality model -->
 	<xacro:property name="hq" value="true" />
@@ -61,11 +61,11 @@
 	</xacro:omni_wheel>
 	<!-- SENSORS -->
-	<xacro:sensor_hokuyo_ust20lx prefix="$(arg prefix)front_laser" parent="$(arg prefix)base_link">
+	<xacro:sensor_hokuyo_ust10lx prefix="$(arg prefix)front_laser" parent="$(arg prefix)base_link" prefix_topic="front_laser">
 		<origin xyz="0.223 0.0 0.159" rpy="0 3.1416 3.1416"/>
-	</xacro:sensor_hokuyo_ust20lx>
-	<xacro:sensor_imu prefix="$(arg prefix)imu" parent="$(arg prefix)base_link">
+	</xacro:sensor_hokuyo_ust10lx>
+	<xacro:sensor_imu_hector prefix="$(arg prefix)imu" parent="$(arg prefix)base_link">
 		<origin xyz="0.002 0.053 0.1485" rpy="0 0 0"/>
-	</xacro:sensor_imu>
-    <xacro:sensor_orbbec_astra prefix="$(arg prefix)front_rgbd_camera" parent="$(arg prefix)base_link">
+	</xacro:sensor_imu_hector>
+    <xacro:sensor_orbbec_astra prefix="$(arg prefix)front_rgbd_camera" parent="$(arg prefix)base_link" prefix_topic="front_rgbd_camera">
         <origin xyz="0.234 0.0125 0.107" rpy="0 0 0"/>
     </xacro:sensor_orbbec_astra>

File: rb1_base_description/urdf/bases/rb1_base_v3.urdf.xacro (robot description, xacro)
@@ -47,5 +47,5 @@
        <origin xyz="0 0 0" rpy="0 0 0 " />
        <geometry>
-         <mesh filename="package://rb1_base_description/meshes/bases/rb1_base_v3.stl"/>
+         <mesh filename="package://rb1_base_description/meshes/bases/rb1_base_v3.dae"/>
        </geometry>
     </collision>
@@ -82,5 +82,5 @@
        <origin xyz="0 0 0" rpy="0 0 0 " />
        <geometry>
-         <mesh filename="package://rb1_base_description/meshes/bases/rb1_front_cover_v3.stl"/>
+         <mesh filename="package://rb1_base_description/meshes/bases/rb1_front_cover_v3.dae"/>
        </geometry>
     </collision>
@@ -101,12 +101,12 @@
        <origin xyz="0 0 0" rpy="0 0 0" />
        <xacro:if value="${hq}">
-       <geometry>
-	     <mesh filename="package://rb1_base_description/meshes/bases/rb1_top_cover_v3.stl"/>
-       </geometry>
+		   <geometry>
+			 <mesh filename="package://rb1_base_description/meshes/bases/rb1_top_cover_v3.stl"/>
+		   </geometry>
        </xacro:if>
        <xacro:unless value="${hq}">
-       <geometry>
-       <mesh filename="package://rb1_base_description/meshes/bases/rb1_top_cover_v3.stl"/>
-       </geometry>
+		   <geometry>
+		   <mesh filename="package://rb1_base_description/meshes/bases/rb1_top_cover_v3.stl"/>
+		   </geometry>
        </xacro:unless>
        <material name="black">
@@ -117,5 +117,5 @@
        <origin xyz="0 0 0" rpy="0 0 0 " />
        <geometry>
-         <mesh filename="package://rb1_base_description/meshes/bases/rb1_top_cover_v3.stl"/>
+         <mesh filename="package://rb1_base_description/meshes/bases/rb1_top_cover_v3.dae"/>
        </geometry>
     </collision>

Commit message: description: changing laser 2d pose (210 mm from the base_footprint

File: rb1_base_description/robots/rb1_base_std.urdf.xacro (robot description, xacro)
@@ -62,5 +62,5 @@
 	<!-- SENSORS -->
 	<xacro:sensor_hokuyo_ust10lx prefix="$(arg prefix)front_laser" parent="$(arg prefix)base_link" prefix_topic="front_laser">
-		<origin xyz="0.223 0.0 0.159" rpy="0 3.1416 3.1416"/>
+		<origin xyz="0.210 0.0 0.159" rpy="0 3.1416 3.1416"/>
 	</xacro:sensor_hokuyo_ust10lx>
 	<xacro:sensor_imu_hector prefix="$(arg prefix)imu" parent="$(arg prefix)base_link">

File: rb1_base_description/robots/rb1_base_std_elevator.urdf.xacro (robot description, xacro)
@@ -72,5 +72,5 @@
 	<!-- SENSORS -->
 	<xacro:sensor_hokuyo_ust20lx prefix="$(arg prefix)front_laser" parent="$(arg prefix)base_link">
-		<origin xyz="0.223 0.0 0.159" rpy="0 3.1416 3.1416"/>
+		<origin xyz="0.210 0.0 0.159" rpy="0 3.1416 3.1416"/>
 	</xacro:sensor_hokuyo_ust20lx>
 	<xacro:sensor_imu prefix="$(arg prefix)imu" parent="$(arg prefix)base_link">

Commit message: description:Change omni wheels configuration
For visualization and simulation purposes
Reduction of omniwheel diameter
Change the 3 omniwheels config by just two wheels

File: rb1_base_description/robots/rb1_base_std.urdf.xacro (robot description, xacro)
@@ -54,10 +54,13 @@
 		<origin xyz="-${omni_back_x} ${omni_back_y} ${omni_back_z}" rpy="0 0 0"/>
 	</xacro:omni_wheel>
-	<xacro:omni_wheel prefix="$(arg prefix)omni_front_left" parent="$(arg prefix)base_link" hq="${hq}">
+	<xacro:omni_wheel prefix="$(arg prefix)omni_front" parent="$(arg prefix)base_link" hq="${hq}">
+		<origin xyz="${omni_back_x} ${omni_back_y} ${omni_back_z}" rpy="0 0 0"/>
+	</xacro:omni_wheel>
+	<!--xacro:omni_wheel prefix="$(arg prefix)omni_front_left" parent="$(arg prefix)base_link" hq="${hq}">
 		<origin xyz="${omni_front_x} ${omni_front_y} ${omni_front_z}" rpy="0 0 0"/>
 	</xacro:omni_wheel>
 	<xacro:omni_wheel prefix="$(arg prefix)omni_front_right" parent="$(arg prefix)base_link" hq="${hq}">
 		<origin xyz="${omni_front_x} -${omni_front_y} ${omni_front_z}" rpy="0 0 0"/>
-	</xacro:omni_wheel>
+	</xacro:omni_wheel-->
 	<!-- SENSORS -->
 	<xacro:sensor_hokuyo_ust10lx prefix="$(arg prefix)front_laser" parent="$(arg prefix)base_link" prefix_topic="front_laser">

File: rb1_base_description/robots/rb1_base_std_elevator.urdf.xacro (robot description, xacro)
@@ -60,10 +60,13 @@
 		<origin xyz="-${omni_back_x} ${omni_back_y} ${omni_back_z}" rpy="0 0 0"/>
 	</xacro:omni_wheel>
-	<xacro:omni_wheel prefix="$(arg prefix)omni_front_left" parent="$(arg prefix)base_link" hq="${hq}">
+	<xacro:omni_wheel prefix="$(arg prefix)omni_front" parent="$(arg prefix)base_link" hq="${hq}">
+		<origin xyz="${omni_back_x} ${omni_back_y} ${omni_back_z}" rpy="0 0 0"/>
+	</xacro:omni_wheel>
+	<!--xacro:omni_wheel prefix="$(arg prefix)omni_front_left" parent="$(arg prefix)base_link" hq="${hq}">
 		<origin xyz="${omni_front_x} ${omni_front_y} ${omni_front_z}" rpy="0 0 0"/>
 	</xacro:omni_wheel>
 	<xacro:omni_wheel prefix="$(arg prefix)omni_front_right" parent="$(arg prefix)base_link" hq="${hq}">
 		<origin xyz="${omni_front_x} -${omni_front_y} ${omni_front_z}" rpy="0 0 0"/>
-	</xacro:omni_wheel>
+	</xacro:omni_wheel-->
 	<!-- ELEVATOR_PLATFORM -->
 	<xacro:elevator_platform prefix="$(arg prefix)elevator" parent="$(arg prefix)base_link" hq="${hq}">

File: rb1_base_description/urdf/wheels/omni_wheel.urdf.xacro (robot description, xacro)
@@ -3,5 +3,5 @@
   <xacro:property name="M_PI" value="3.1415926535897931" />
   <!-- Wheels -->
-  <xacro:property name="omni_wheel_radius" value="0.051" />
+  <xacro:property name="omni_wheel_radius" value="0.050" />
   <xacro:property name="omni_wheel_height" value="0.040" />
   <xacro:property name="omni_wheel_mass" value="0.3" /> <!-- in kg-->

Commit message: Added option to use ros_planar_plugin

File: rb1_base_description/robots/rb1_base_std.urdf.xacro (robot description, xacro)
@@ -1,4 +1,5 @@
 <?xml version="1.0"?>
-<robot name="rb1_base" xmlns:xacro="http://www.ros.org/wiki/xacro">
+<robot name="rb1_base"
+	xmlns:xacro="http://www.ros.org/wiki/xacro">
 	<!-- ***************** -->
 	<!-- Imported elements -->
@@ -6,5 +7,6 @@
 	<!-- First we import all posible elements defined in the urdf.xacro files. All these elements are defined as macro:xacros -->
 	<!-- Import RB1 base elements -->
-    <xacro:include filename="$(find rb1_base_description)/urdf/bases/rb1_base_v3.urdf.xacro" /> <!-- v3 name from engineering department -->
+	<xacro:include filename="$(find rb1_base_description)/urdf/bases/rb1_base_v3.urdf.xacro" />
+	<!-- v3 name from engineering department -->
 	<!-- Import RB1 wheels -->
 	<xacro:include filename="$(find rb1_base_description)/urdf/wheels/rubber_wheel.urdf.xacro" />
@@ -12,7 +14,7 @@
 	<!-- Import all available sensors -->
 	<xacro:include filename="$(find robotnik_sensors)/urdf/all_sensors.urdf.xacro" />
-    <!-- Import Gazebo Stuff -->
-    <xacro:include filename="$(find rb1_base_description)/urdf/common.gazebo.xacro" />
-    <!-- Import Elevator -->
+	<!-- Import Gazebo Stuff -->
+	<xacro:include filename="$(find rb1_base_description)/urdf/common.gazebo.xacro" />
+	<!-- Import Elevator -->
 	<xacro:include filename="$(find rb1_base_description)/urdf/elevator/elevator.urdf.xacro"/>
 	<!-- ***************** -->
@@ -21,5 +23,6 @@
 	<xacro:property name="PI" value="3.1415926535897931"/>
 	<!-- Wheel parameters -->
-	<xacro:property name="wheel_offset_x" value="0.0" />    <!-- x,y,z in translation from base_link to the center of the wheel -->
+	<xacro:property name="wheel_offset_x" value="0.0" />
+	<!-- x,y,z in translation from base_link to the center of the wheel -->
 	<xacro:property name="wheel_offset_y" value="0.218" />
 	<xacro:property name="wheel_offset_z" value="0.0512" />
@@ -40,6 +43,10 @@
 	<xacro:rb1_base_v3 prefix="$(arg prefix)" publish_bf="true" hq="${hq}" />
 	<xacro:arg name="prefix" default="rb1_"/>
+	<xacro:arg name="ros_planar_move_plugin" default="false"/>
 	<!-- Gazebo ros control plugins -->
 	<xacro:ros_control/>
+	<xacro:if value="$(arg ros_planar_move_plugin)">
+		<xacro:skid_steering prefix="$(arg prefix)" publish_tf="true"/>
+	</xacro:if>
 	<xacro:gazebo_colors prefix="$(arg prefix)"/>
 	<!-- WHEELS -->
@@ -50,5 +57,5 @@
 		<origin xyz="${wheel_offset_x} ${wheel_offset_y} ${wheel_offset_z}" rpy="0 0 0"/>
 	</xacro:rubber_wheel>
-    <!-- OMNI DIRECTIONAL WHEELS -->
+	<!-- OMNI DIRECTIONAL WHEELS -->
 	<xacro:omni_wheel prefix="$(arg prefix)omni_back" parent="$(arg prefix)base_link" hq="${hq}">
 		<origin xyz="-${omni_back_x} ${omni_back_y} ${omni_back_z}" rpy="0 0 0"/>
@@ -67,6 +74,6 @@
 		<origin xyz="0.002 0.053 0.1485" rpy="0 0 0"/>
 	</xacro:sensor_imu_hector>
-    <xacro:sensor_orbbec_astra prefix="$(arg prefix)front_rgbd_camera" parent="$(arg prefix)base_link" prefix_topic="front_rgbd_camera">
-        <origin xyz="0.234 0.0125 0.107" rpy="0 0 0"/>
-    </xacro:sensor_orbbec_astra>
+	<xacro:sensor_orbbec_astra prefix="$(arg prefix)front_rgbd_camera" parent="$(arg prefix)base_link" prefix_topic="front_rgbd_camera">
+		<origin xyz="0.234 0.0125 0.107" rpy="0 0 0"/>
+	</xacro:sensor_orbbec_astra>
 </robot>

File: rb1_base_description/robots/rb1_base_std_elevator.urdf.xacro (robot description, xacro)
@@ -1,4 +1,5 @@
 <?xml version="1.0"?>
-<robot name="rb1_base" xmlns:xacro="http://www.ros.org/wiki/xacro">
+<robot name="rb1_base"
+	xmlns:xacro="http://www.ros.org/wiki/xacro">
 	<!-- ***************** -->
 	<!-- Imported elements -->
@@ -6,5 +7,6 @@
 	<!-- First we import all posible elements defined in the urdf.xacro files. All these elements are defined as macro:xacros -->
 	<!-- Import RB1 base elements -->
-    <xacro:include filename="$(find rb1_base_description)/urdf/bases/rb1_base_v3.urdf.xacro" /> <!-- v3 name from engineering department -->
+	<xacro:include filename="$(find rb1_base_description)/urdf/bases/rb1_base_v3.urdf.xacro" />
+	<!-- v3 name from engineering department -->
 	<!-- Import RB1 wheels -->
 	<xacro:include filename="$(find rb1_base_description)/urdf/wheels/rubber_wheel.urdf.xacro" />
@@ -12,7 +14,7 @@
 	<!-- Import all available sensors -->
 	<xacro:include filename="$(find robotnik_sensors)/urdf/all_sensors.urdf.xacro" />
-    <!-- Import Gazebo Stuff -->
-    <xacro:include filename="$(find rb1_base_description)/urdf/common.gazebo.xacro" />
-    <!-- Import Elevator -->
+	<!-- Import Gazebo Stuff -->
+	<xacro:include filename="$(find rb1_base_description)/urdf/common.gazebo.xacro" />
+	<!-- Import Elevator -->
 	<xacro:include filename="$(find rb1_base_description)/urdf/elevator/elevator.urdf.xacro"/>
 	<!-- ***************** -->
@@ -21,5 +23,6 @@
 	<xacro:property name="PI" value="3.1415926535897931"/>
 	<!-- Wheel parameters -->
-	<xacro:property name="wheel_offset_x" value="0.0" />    <!-- x,y,z in translation from base_link to the center of the wheel -->
+	<xacro:property name="wheel_offset_x" value="0.0" />
+	<!-- x,y,z in translation from base_link to the center of the wheel -->
 	<xacro:property name="wheel_offset_y" value="0.218" />
 	<xacro:property name="wheel_offset_z" value="0.0512" />
@@ -46,6 +49,10 @@
 	<xacro:rb1_base_v3 prefix="$(arg prefix)" publish_bf="true" hq="${hq}" />
 	<xacro:arg name="prefix" default="rb1_"/>
+	<xacro:arg name="ros_planar_move_plugin" default="false"/>
 	<!-- Gazebo ros control pluggins -->
 	<xacro:ros_control/>
+	<xacro:if value="$(arg ros_planar_move_plugin)">
+		<xacro:skid_steering prefix="$(arg prefix)" publish_tf="true"/>
+	</xacro:if>
 	<xacro:gazebo_colors prefix="$(arg prefix)"/>
 	<!-- WHEELS -->
@@ -56,5 +63,5 @@
 		<origin xyz="${wheel_offset_x} ${wheel_offset_y} ${wheel_offset_z}" rpy="0 0 0"/>
 	</xacro:rubber_wheel>
-    <!-- OMNI DIRECTIONAL WHEELS -->
+	<!-- OMNI DIRECTIONAL WHEELS -->
 	<xacro:omni_wheel prefix="$(arg prefix)omni_back" parent="$(arg prefix)base_link" hq="${hq}">
 		<origin xyz="-${omni_back_x} ${omni_back_y} ${omni_back_z}" rpy="0 0 0"/>
@@ -77,6 +84,6 @@
 		<origin xyz="0.002 0.053 0.1485" rpy="0 0 0"/>
 	</xacro:sensor_imu>
-    <xacro:sensor_orbbec_astra prefix="$(arg prefix)front_rgbd_camera" parent="$(arg prefix)base_link">
-        <origin xyz="0.234 0.0125 0.107" rpy="0 0 0"/>
-    </xacro:sensor_orbbec_astra>
+	<xacro:sensor_orbbec_astra prefix="$(arg prefix)front_rgbd_camera" parent="$(arg prefix)base_link">
+		<origin xyz="0.234 0.0125 0.107" rpy="0 0 0"/>
+	</xacro:sensor_orbbec_astra>
 </robot>

File: rb1_base_description/urdf/common.gazebo.xacro (robot description, xacro)
@@ -1,22 +1,35 @@
 <?xml version="1.0"?>
 <robot xmlns:xacro="http://www.ros.org/wiki/xacro">
-<!-- ROS CONTROL GAZEBO PLUGIN -->
+	<!-- ROS CONTROL GAZEBO PLUGIN -->
 	<xacro:macro name="ros_control">
-	   <gazebo>
-      <plugin name="ros_control" filename="libgazebo_ros_control.so">
-        <!--robotNamespace>/rb1</robotNamespace-->
-        <robotParam>robot_description</robotParam>
-        <controlPeriod>0.001</controlPeriod>
-	      <robotSimType>gazebo_ros_control/DefaultRobotHWSim</robotSimType>
+		<gazebo>
+			<plugin name="ros_control" filename="libgazebo_ros_control.so">
+				<!--robotNamespace>/rb1</robotNamespace-->
+				<robotParam>robot_description</robotParam>
+				<controlPeriod>0.001</controlPeriod>
+				<robotSimType>gazebo_ros_control/DefaultRobotHWSim</robotSimType>
 				<legacyModeNS>true</legacyModeNS>
-      </plugin>
-   </gazebo>
-   </xacro:macro>
-   <xacro:macro name="gazebo_colors" params="prefix">
+			</plugin>
+		</gazebo>
+	</xacro:macro>
+	<xacro:macro name="skid_steering" params="prefix publish_tf">
+		<gazebo>
+			<plugin name="skid_steering" filename="libgazebo_ros_planar_move.so">
+				<commandTopic>robotnik_base_control/cmd_vel</commandTopic>
+				<odometryTopic>robotnik_base_control/odom</odometryTopic>
+				<odometryFrame>${prefix}odom</odometryFrame>
+				<odometryRate>50.0</odometryRate>
+				<robotBaseFrame>${prefix}base_footprint</robotBaseFrame>
+				<publishTF>${publish_tf}</publishTF>
+				<enableYAxis>false</enableYAxis>
+			</plugin>
+		</gazebo>
+	</xacro:macro>
+	<xacro:macro name="gazebo_colors" params="prefix">
 		<gazebo reference="$(arg prefix)base_footprint">
 			<material>Gazebo/Green</material>
 		</gazebo>
 		<gazebo reference="$(arg prefix)base_link">
-			<material>Gazebo/Grey</material>
+			<material>Gazebo/Black</material>
 		</gazebo>
 		<gazebo reference="$(arg prefix)front_cover_link">

Commit message: added gpu usage value on simulation default false

File: rb1_base_description/robots/rb1_base_std.urdf.xacro (robot description, xacro)
@@ -40,4 +40,6 @@
 	<xacro:rb1_base_v3 prefix="$(arg prefix)" publish_bf="true" hq="${hq}" />
 	<xacro:arg name="prefix" default="rb1_"/>
+	<xacro:arg name="use_gpu_for_simulation" default="false" />
+	<xacro:property name="gpu" value="$(arg use_gpu_for_simulation)" />
 	<!-- Gazebo ros control plugins -->
 	<xacro:ros_control/>

Commit message: Added flag for selecting hq on urdf

File: rb1_base_description/robots/rb1_base_std.urdf.xacro (robot description, xacro)
@@ -32,5 +32,6 @@
 	<xacro:property name="omni_front_z" value="0.0270" />
 	<!-- Flag to select the high or low quality model -->
-	<xacro:property name="hq" value="true" />
+	<xacro:arg name="hq_models" default="true" />
+	<xacro:property name="hq" value="$(arg hq_models)" />
 	<!-- *************** -->
 	<!-- Robots Elements -->

Commit message: Added to base

File: rb1_base_description/robots/rb1_base_std.urdf.xacro (robot description, xacro)
@@ -16,4 +16,6 @@
     <!-- Import Elevator -->
 	<xacro:include filename="$(find rb1_base_description)/urdf/elevator/elevator.urdf.xacro"/>
+	<!-- Import Led -->
+	<xacro:include filename="$(find rb1_base_description)/urdf/others/led.urdf.xacro"/>
 	<!-- ***************** -->
 	<!-- Global parameters -->
@@ -73,3 +75,7 @@
         <origin xyz="0.234 0.0125 0.107" rpy="0 0 0"/>
     </xacro:sensor_orbbec_astra>
+    <!-- LED -->
+    <xacro:led prefix="$(arg prefix)led" parent="$(arg prefix)base_link">
+    	<origin xyz="0.0 0.0 1.4" rpy="3.14 0 0"/>
+    </xacro:led>
 </robot>
