Commit message: description: Fix hokuyo position on default robot models

File: rb1_base_description/robots/rb1_base.urdf.xacro (robot description, xacro)
@@ -68,5 +68,5 @@
 	<!-- SENSORS -->
 	<xacro:sensor_hokuyo_ust20lx prefix="$(arg prefix)front_laser" parent="$(arg prefix)base_link" prefix_topic="front_laser" gpu="$(arg gpu)">
-		<origin xyz="0.210 0.0 0.159" rpy="0 3.1416 3.1416"/>
+		<origin xyz="0.210 0.0 0.21" rpy="0 3.1416 3.1416"/>
 	</xacro:sensor_hokuyo_ust20lx>
 	<xacro:sensor_imu_hector prefix="$(arg prefix)imu" parent="$(arg prefix)base_link">

File: rb1_base_description/robots/rb1_base_elevator.urdf.xacro (robot description, xacro)
@@ -78,5 +78,5 @@
 	<!-- SENSORS -->
 	<xacro:sensor_hokuyo_ust20lx prefix="$(arg prefix)front_laser" parent="$(arg prefix)base_link" prefix_topic="front_laser" gpu="$(arg gpu)">
-		<origin xyz="0.210 0.0 0.159" rpy="0 3.1416 3.1416"/>
+		<origin xyz="0.210 0.0 0.21" rpy="0 3.1416 3.1416"/>
 	</xacro:sensor_hokuyo_ust20lx>
 	<xacro:sensor_imu prefix="$(arg prefix)imu" parent="$(arg prefix)base_link">

Commit message: description: update rgbd camera default position

File: rb1_base_description/robots/rb1_base.urdf.xacro (robot description, xacro)
@@ -74,5 +74,5 @@
 	</xacro:sensor_imu_hector>
 	<xacro:sensor_orbbec_astra prefix="$(arg prefix)front_rgbd_camera" parent="$(arg prefix)base_link" prefix_topic="front_rgbd_camera">
-		<origin xyz="0.234 0.0125 0.107" rpy="0 0 0"/>
+		<origin xyz="0.234 0.0 0.092" rpy="0 0 0"/>
 	</xacro:sensor_orbbec_astra>
 	<!-- Gazebo ros control plugins -->

File: rb1_base_description/robots/rb1_base_elevator.urdf.xacro (robot description, xacro)
@@ -84,5 +84,5 @@
 	</xacro:sensor_imu>
 	<xacro:sensor_orbbec_astra prefix="$(arg prefix)front_rgbd_camera" parent="$(arg prefix)base_link">
-		<origin xyz="0.234 0.0125 0.107" rpy="0 0 0"/>
+		<origin xyz="0.234 0.0 0.092" rpy="0 0 0"/>
 	</xacro:sensor_orbbec_astra>
 	<!-- Gazebo ros control pluggins -->

Commit message: Removed prefix arg and clean rb1_base_v3

File: rb1_base_description/robots/rb1_base.urdf.xacro (robot description, xacro)
@@ -1,83 +1,73 @@
 <?xml version="1.0"?>
-<robot name="rb1_base"
-	xmlns:xacro="http://www.ros.org/wiki/xacro">
-	<!-- ***************** -->
-	<!-- Imported elements -->
-	<!-- ***************** -->
-	<!-- First we import all posible elements defined in the urdf.xacro files. All these elements are defined as macro:xacros -->
-	<!-- Import RB1 base elements -->
-	<xacro:include filename="$(find rb1_base_description)/urdf/bases/rb1_base_v3.urdf.xacro" />
-	<!-- v3 name from engineering department -->
-	<!-- Import RB1 wheels -->
-	<xacro:include filename="$(find rb1_base_description)/urdf/wheels/rubber_wheel.urdf.xacro" />
-	<xacro:include filename="$(find rb1_base_description)/urdf/wheels/omni_wheel.urdf.xacro" />
-	<!-- Import all available sensors -->
-	<xacro:include filename="$(find robotnik_sensors)/urdf/all_sensors.urdf.xacro" />
-	<!-- Import Gazebo Stuff -->
-	<xacro:include filename="$(find rb1_base_description)/urdf/common.gazebo.xacro" />
-	<!-- Import Elevator -->
-	<xacro:include filename="$(find rb1_base_description)/urdf/elevator/elevator.urdf.xacro"/>
-	<!-- ***************** -->
-	<!-- Global parameters -->
-	<!-- ***************** -->
-	<xacro:property name="PI" value="3.1415926535897931"/>
-	<!-- Wheel parameters -->
-	<xacro:property name="wheel_offset_x" value="0.0" />
-	<!-- x,y,z in translation from base_link to the center of the wheel -->
-	<xacro:property name="wheel_offset_y" value="0.218" />
-	<xacro:property name="wheel_offset_z" value="0.0512" />
-	<!-- Castor paramters -->
-	<xacro:property name="omni_back_x" value="0.195" />
-	<xacro:property name="omni_back_y" value="0.0" />
-	<xacro:property name="omni_back_z" value="0.0270" />
-	<xacro:property name="omni_front_x" value="0.132" />
-	<xacro:property name="omni_front_y" value="0.1535" />
-	<xacro:property name="omni_front_z" value="0.0270" />
-	<!-- Flag to select the high or low quality model -->
-	<xacro:property name="hq" value="true" />
-	<xacro:arg name="robot_id" default="robot"/>
-	<xacro:arg name="prefix" default=""/>
-	<xacro:arg name="config_controllers" default=""/>
-	<xacro:arg name="ros_planar_move_plugin" default="false"/>
-	<xacro:arg name="gpu" default="false"/>
-	<!-- *************** -->
-	<!-- Robots Elements -->
-	<!-- *************** -->
-	<!-- Here we create the robot elements using the xacro:macros imported at the beggining of this file -->
-	<!-- RB-1 base -->
-	<xacro:rb1_base_v3 prefix="$(arg prefix)" publish_bf="true" hq="${hq}" />
-	<xacro:if value="$(arg ros_planar_move_plugin)">
-		<xacro:skid_steering prefix="$(arg prefix)" publish_tf="true"/>
-	</xacro:if>
-	<xacro:gazebo_colors prefix="$(arg prefix)"/>
-	<!-- WHEELS -->
-	<xacro:rubber_wheel prefix="$(arg prefix)right" parent="$(arg prefix)base_link" reflect="false" hq="${hq}">
-		<origin xyz="${wheel_offset_x} -${wheel_offset_y} ${wheel_offset_z}" rpy="0 0 0"/>
-	</xacro:rubber_wheel>
-	<xacro:rubber_wheel prefix="$(arg prefix)left" parent="$(arg prefix)base_link" reflect="true" hq="${hq}">
-		<origin xyz="${wheel_offset_x} ${wheel_offset_y} ${wheel_offset_z}" rpy="0 0 0"/>
-	</xacro:rubber_wheel>
-	<!-- OMNI DIRECTIONAL WHEELS -->
-	<xacro:omni_wheel prefix="$(arg prefix)omni_back" parent="$(arg prefix)base_link" hq="${hq}">
-		<origin xyz="-${omni_back_x} ${omni_back_y} ${omni_back_z}" rpy="0 0 0"/>
-	</xacro:omni_wheel>
-	<xacro:omni_wheel prefix="$(arg prefix)omni_front_left" parent="$(arg prefix)base_link" hq="${hq}">
-		<origin xyz="${omni_front_x} ${omni_front_y} ${omni_front_z}" rpy="0 0 0"/>
-	</xacro:omni_wheel>
-	<xacro:omni_wheel prefix="$(arg prefix)omni_front_right" parent="$(arg prefix)base_link" hq="${hq}">
-		<origin xyz="${omni_front_x} -${omni_front_y} ${omni_front_z}" rpy="0 0 0"/>
-	</xacro:omni_wheel>
-	<!-- SENSORS -->
-	<xacro:sensor_hokuyo_ust20lx prefix="$(arg prefix)front_laser" parent="$(arg prefix)base_link" prefix_topic="front_laser" gpu="$(arg gpu)">
-		<origin xyz="0.210 0.0 0.21" rpy="0 3.1416 3.1416"/>
-	</xacro:sensor_hokuyo_ust20lx>
-	<xacro:sensor_imu_hector prefix="$(arg prefix)imu" parent="$(arg prefix)base_link">
-		<origin xyz="0.002 0.053 0.1485" rpy="0 0 0"/>
-	</xacro:sensor_imu_hector>
-	<xacro:sensor_orbbec_astra prefix="$(arg prefix)front_rgbd_camera" parent="$(arg prefix)base_link" prefix_topic="front_rgbd_camera">
-		<origin xyz="0.234 0.0 0.092" rpy="0 0 0"/>
-	</xacro:sensor_orbbec_astra>
-	<!-- Gazebo ros control plugins -->
-    <xacro:include filename="$(find rb1_base_description)/urdf/ros2_control.urdf.xacro"/>
-    <xacro:ros2_control prefix="$(arg prefix)"/>
+<robot name="rb1_base" xmlns:xacro="http://www.ros.org/wiki/xacro">
+  <!-- ***************** -->
+  <!-- Imported elements -->
+  <!-- ***************** -->
+  <!-- Import RB1 base elements (base + wheels) -->
+  <xacro:include filename="$(find rb1_base_description)/urdf/bases/rb1_base_v3.urdf.xacro"/>
+  <xacro:include filename="$(find rb1_base_description)/urdf/wheels/rubber_wheel.urdf.xacro"/>
+  <xacro:include filename="$(find rb1_base_description)/urdf/wheels/omni_wheel.urdf.xacro"/>
+  <!-- Import all available sensors -->
+  <xacro:include filename="$(find robotnik_sensors)/urdf/all_sensors.urdf.xacro"/>
+  <!-- Import Gazebo Stuff -->
+  <xacro:include filename="$(find rb1_base_description)/urdf/common.gazebo.xacro"/>
+  <!-- Import Elevator -->
+  <xacro:include filename="$(find rb1_base_description)/urdf/elevator/elevator.urdf.xacro"/>
+  <!-- ***************** -->
+  <!-- Global parameters -->
+  <!-- ***************** -->
+  <xacro:property name="PI" value="3.1415926535897931"/>
+  <!-- Wheel parameters -->
+  <!-- x,y,z in translation from base_link to the center of the wheel -->
+  <xacro:property name="wheel_offset_x" value="0.0"/>
+  <xacro:property name="wheel_offset_y" value="0.218"/>
+  <xacro:property name="wheel_offset_z" value="0.0512"/>
+  <!-- Castor paramters -->
+  <xacro:property name="omni_back_x" value="0.195" />
+  <xacro:property name="omni_back_y" value="0.0"/>
+  <xacro:property name="omni_back_z" value="0.0270"/>
+  <xacro:property name="omni_front_x" value="0.132"/>
+  <xacro:property name="omni_front_y" value="0.1535"/>
+  <xacro:property name="omni_front_z" value="0.0270"/>
+  <!-- Flag to select the high or low quality model -->
+  <xacro:property name="hq" value="true"/>
+  <xacro:arg name="robot_id" default="robot"/>
+  <xacro:arg name="robot_ns" default="$(arg robot_id)"/>
+  <!-- *************** -->
+  <!-- Robots Elements -->
+  <!-- *************** -->
+  <!-- RB-1 base -->
+  <xacro:rb1_base_v3 publish_bf="true" hq="${hq}"/>
+  <xacro:gazebo_colors />
+  <!-- WHEELS -->
+  <xacro:rubber_wheel prefix="right" parent="base_link" reflect="false" hq="${hq}">
+    <origin xyz="${wheel_offset_x} -${wheel_offset_y} ${wheel_offset_z}" rpy="0 0 0"/>
+  </xacro:rubber_wheel>
+  <xacro:rubber_wheel prefix="left" parent="base_link" reflect="true" hq="${hq}">
+    <origin xyz="${wheel_offset_x} ${wheel_offset_y} ${wheel_offset_z}" rpy="0 0 0"/>
+  </xacro:rubber_wheel>
+  <!-- OMNI DIRECTIONAL WHEELS -->
+  <xacro:omni_wheel prefix="omni_back" parent="base_link" hq="${hq}">
+    <origin xyz="-${omni_back_x} ${omni_back_y} ${omni_back_z}" rpy="0 0 0"/>
+  </xacro:omni_wheel>
+  <xacro:omni_wheel prefix="omni_front_left" parent="base_link" hq="${hq}">
+    <origin xyz="${omni_front_x} ${omni_front_y} ${omni_front_z}" rpy="0 0 0"/>
+  </xacro:omni_wheel>
+  <xacro:omni_wheel prefix="omni_front_right" parent="base_link" hq="${hq}">
+    <origin xyz="${omni_front_x} -${omni_front_y} ${omni_front_z}" rpy="0 0 0"/>
+  </xacro:omni_wheel>
+  <!-- SENSORS -->
+  <xacro:sensor_hokuyo_ust20lx ns="$(arg robot_ns)" prefix="front_laser" parent="base_link">
+    <origin xyz="0.210 0.0 0.21" rpy="0 3.1416 3.1416"/>
+  </xacro:sensor_hokuyo_ust20lx>
+  <xacro:sensor_imu_hector ns="$(arg robot_ns)" prefix="imu" parent="base_link">
+    <origin xyz="0.002 0.053 0.1485" rpy="0 0 0"/>
+  </xacro:sensor_imu_hector>
+  <xacro:sensor_orbbec_astra ns="$(arg robot_ns)" prefix="front_rgbd_camera" parent="base_link">
+    <origin xyz="0.234 0.0 0.092" rpy="0 0 0"/>
+  </xacro:sensor_orbbec_astra>
+  <!-- Gazebo ros control plugins -->
+  <xacro:arg name="config_controllers" default=""/>
+  <xacro:include filename="$(find rb1_base_description)/urdf/ros2_control.urdf.xacro"/>
+  <xacro:ros2_control/>
 </robot>

File: rb1_base_description/urdf/bases/rb1_base_v3.urdf.xacro (robot description, xacro)
@@ -1,5 +1,5 @@
 <?xml version="1.0"?>
 <robot name="rb1_base" xmlns:xacro="http://www.ros.org/wiki/xacro">
-  <xacro:macro name="rb1_base_v3" params="prefix publish_bf hq">
+  <xacro:macro name="rb1_base_v3" params="publish_bf hq">
   <!-- Robot mechanical and motor parameters -->
   <xacro:property name="PI" value="3.1415926535897931"/>
@@ -7,5 +7,5 @@
   <!-- BASE FOOTPRINT -->
   <xacro:if value="${publish_bf}">
-    <link name="${prefix}base_footprint">
+    <link name="base_footprint">
       <!--visual>
           <origin xyz="0 0 0" rpy="0 0 0" />
@@ -15,15 +15,15 @@
       </visual-->
     </link>
-    <joint name="${prefix}base_footprint_joint" type="fixed">
+    <joint name="base_footprint_joint" type="fixed">
        <origin xyz="0 0 ${wheel_radius - wheel_offset_z}" rpy="0 0 0" />
-      <parent link="${prefix}base_footprint"/>
-      <child link="${prefix}base_link" />
+      <parent link="base_footprint"/>
+      <child link="base_link" />
     </joint>
   </xacro:if>
   <!-- BASE_LINK -->
-  <link name="${prefix}base_link">
+  <link name="base_link">
     <inertial>
       <mass value="25.0" />
-      <origin xyz="0 0 0" />
+      <origin xyz="0 0 0.07" />
       <inertia  ixx="0.605" ixy="0.0"  ixz="0.0"  iyy="0.5435"  iyz="0.0"  izz="0.981" />
     </inertial>
@@ -51,15 +51,15 @@
     </collision-->
   </link>
-  <joint name="${prefix}front_cover_joint" type="fixed">
+  <joint name="front_cover_joint" type="fixed">
      <origin xyz="0.220 0.0 0.004" rpy="0 0 0 " />
-     <parent link="${prefix}base_link"/>
-     <child link="${prefix}front_cover_link" />
+     <parent link="base_link"/>
+     <child link="front_cover_link" />
   </joint>
   <!-- FRONT COVER -->
-  <link name="${prefix}front_cover_link">
+  <link name="front_cover_link">
     <inertial>
       <mass value="0.25" />
-      <origin xyz="0 0 0" />
-      <inertia  ixx="0.00007" ixy="0.0"  ixz="0.0"  iyy="0.00007"  iyz="0.0"  izz="0.0078" />
+      <origin xyz="0 0 0.05" />
+      <inertia  ixx="0.001" ixy="0.0"  ixz="0.0"  iyy="0.001"  iyz="0.0"  izz="0.001" />
     </inertial>
     <visual>
@@ -86,15 +86,15 @@
     </collision>
   </link>
-  <joint name="${prefix}top_covert_joint" type="fixed">
+  <joint name="top_covert_joint" type="fixed">
      <origin xyz="0.0 0.0 0.243" rpy="0 0 0 " />
-     <parent link="${prefix}base_footprint"/>
-     <child link="${prefix}top_cover_link" />
+     <parent link="base_footprint"/>
+     <child link="top_cover_link" />
   </joint>
   <!-- FRONT COVER -->
-  <link name="${prefix}top_cover_link">
+  <link name="top_cover_link">
     <inertial>
       <mass value="0.25" />
       <origin xyz="0 0 0" />
-      <inertia  ixx="0.00007" ixy="0.0"  ixz="0.0"  iyy="0.00007"  iyz="0.0"  izz="0.0078" />
+      <inertia  ixx="0.0007" ixy="0.0"  ixz="0.0"  iyy="0.0007"  iyz="0.0"  izz="0.001" />
     </inertial>
     <visual>
@@ -122,11 +122,11 @@
   </link>
   <!-- DOCKING CONTACTS -->
-  <joint name="${prefix}base_docking_joint" type="fixed">
+  <joint name="base_docking_joint" type="fixed">
      <origin xyz="0.030 0.000 0.068" rpy="0 0 0 " />
-     <parent link="${prefix}front_cover_link"/>
-     <child link="${prefix}base_docking_contact_link" />
+     <parent link="front_cover_link"/>
+     <child link="base_docking_contact_link" />
   </joint>
   <!-- DOCKING LINK -->
-  <link name="${prefix}base_docking_contact_link" />
+  <link name="base_docking_contact_link" />
   </xacro:macro>
 </robot>

File: rb1_base_description/urdf/common.gazebo.xacro (robot description, xacro)
@@ -18,7 +18,7 @@
 				<commandTopic>robotnik_base_control/cmd_vel</commandTopic>
 				<odometryTopic>robotnik_base_control/odom</odometryTopic>
-				<odometryFrame>${prefix}odom</odometryFrame>
+				<odometryFrame>odom</odometryFrame>
 				<odometryRate>50.0</odometryRate>
-				<robotBaseFrame>${prefix}base_footprint</robotBaseFrame>
+				<robotBaseFrame>base_footprint</robotBaseFrame>
 				<publishTF>${publish_tf}</publishTF>
 				<enableYAxis>false</enableYAxis>
@@ -27,13 +27,13 @@
 		</gazebo>
 	</xacro:macro>
-	<xacro:macro name="gazebo_colors" params="prefix">
-		<gazebo reference="$(arg prefix)base_footprint">
+	<xacro:macro name="gazebo_colors">
+		<gazebo reference="base_footprint">
 			<material>Gazebo/Green</material>
 		</gazebo>
-		<gazebo reference="$(arg prefix)base_link">
-			<material>Gazebo/Black</material>
+		<gazebo reference="base_link">
+			<material>Gazebo/DarkGrey</material>
 		</gazebo>
-		<gazebo reference="$(arg prefix)front_cover_link">
-			<material>Gazebo/Black</material>
+		<gazebo reference="front_cover_link">
+			<material>Gazebo/DarkGrey</material>
 		</gazebo>
 	</xacro:macro>

File: rb1_base_description/urdf/ros2_control.urdf.xacro (robot description, xacro)
@@ -1,5 +1,5 @@
 <?xml version="1.0"?>
 <robot xmlns:xacro="http://wiki.ros.org/xacro">
-  <xacro:macro name="ros2_control" params="prefix">
+  <xacro:macro name="ros2_control">
       <gazebo>
         <plugin name="ros_control" filename="libgazebo_ros2_control.so">
@@ -12,5 +12,5 @@
           <plugin>gazebo_ros2_control/GazeboSystem</plugin>
         </hardware>
-        <joint name="${prefix}left_wheel_joint">
+        <joint name="left_wheel_joint">
           <command_interface name="velocity">
             <param name="min">-10</param>
@@ -21,5 +21,5 @@
           <state_interface name="effort"/>
         </joint>
-        <joint name="${prefix}right_wheel_joint">
+        <joint name="right_wheel_joint">
           <command_interface name="velocity">
             <param name="min">-10</param>

Commit message: Added base texture

File: rb1_base_description/robots/rb1_base.urdf.xacro (robot description, xacro)
@@ -39,5 +39,5 @@
   <!-- RB-1 base -->
   <xacro:rb1_base_v3 publish_bf="true" hq="${hq}"/>
-  <xacro:gazebo_colors />
+  <!--xacro:gazebo_colors /-->
   <!-- WHEELS -->
   <xacro:rubber_wheel prefix="right" parent="base_link" reflect="false" hq="${hq}">

File: rb1_base_description/urdf/bases/rb1_base_v3.urdf.xacro (robot description, xacro)
@@ -7,12 +7,5 @@
   <!-- BASE FOOTPRINT -->
   <xacro:if value="${publish_bf}">
-    <link name="base_footprint">
-      <!--visual>
-          <origin xyz="0 0 0" rpy="0 0 0" />
-          <geometry>
-             <box size="0.001 0.001 0.001" />
-          </geometry>
-      </visual-->
-    </link>
+    <link name="base_footprint"/>
     <joint name="base_footprint_joint" type="fixed">
        <origin xyz="0 0 ${wheel_radius - wheel_offset_z}" rpy="0 0 0" />
@@ -29,25 +22,9 @@
     </inertial>
     <visual>
-       <origin xyz="0 0 0" rpy="0 0 0" />
-       <xacro:if value="${hq}">
-       <geometry>
-	     <mesh filename="package://rb1_base_description/meshes/bases/rb1_base_v3.stl"/>
-       </geometry>
-       </xacro:if>
-       <xacro:unless value="${hq}">
-       <geometry>
-       <mesh filename="package://rb1_base_description/meshes/bases/rb1_base_v3.stl"/>
-       </geometry>
-       </xacro:unless>
-       <material name="darkgrey">
-         <color rgba="0.1 0.1 0.1 1"/>
-       </material>
+      <origin xyz="0 0 0" rpy="0 0 0" />
+      <geometry>
+        <mesh filename="package://rb1_base_description/meshes/bases/rb1_base_v3_color.dae"/>
+      </geometry>
     </visual>
-    <!--collision>
-       <origin xyz="0 0 0" rpy="0 0 0 " />
-       <geometry>
-         <mesh filename="package://rb1_base_description/meshes/bases/rb1_base_v3.dae"/>
-       </geometry>
-    </collision-->
   </link>
   <joint name="front_cover_joint" type="fixed">
