Commit message: Update physics, and formated

File: rb1_base_description/robots/rb1_base.urdf.xacro (robot description, xacro)
@@ -10,6 +10,4 @@
   <!-- Import all available sensors -->
   <xacro:include filename="$(find robotnik_sensors)/urdf/all_sensors.urdf.xacro"/>
-  <!-- Import Gazebo Stuff -->
-  <xacro:include filename="$(find rb1_base_description)/urdf/common.gazebo.xacro"/>
   <!-- Import Elevator -->
   <xacro:include filename="$(find rb1_base_description)/urdf/elevator/elevator.urdf.xacro"/>
@@ -41,18 +39,18 @@
   <!--xacro:gazebo_colors /-->
   <!-- WHEELS -->
-  <xacro:rubber_wheel prefix="right" parent="base_link" reflect="false" hq="${hq}">
+  <xacro:rubber_wheel prefix="right_" parent="base_link" reflect="false" hq="${hq}">
     <origin xyz="${wheel_offset_x} -${wheel_offset_y} ${wheel_offset_z}" rpy="0 0 0"/>
   </xacro:rubber_wheel>
-  <xacro:rubber_wheel prefix="left" parent="base_link" reflect="true" hq="${hq}">
+  <xacro:rubber_wheel prefix="left_" parent="base_link" reflect="true" hq="${hq}">
     <origin xyz="${wheel_offset_x} ${wheel_offset_y} ${wheel_offset_z}" rpy="0 0 0"/>
   </xacro:rubber_wheel>
   <!-- OMNI DIRECTIONAL WHEELS -->
-  <xacro:omni_wheel prefix="omni_back" parent="base_link" hq="${hq}">
+  <xacro:omni_wheel prefix="omni_back_" parent="base_link" hq="${hq}">
     <origin xyz="-${omni_back_x} ${omni_back_y} ${omni_back_z}" rpy="0 0 0"/>
   </xacro:omni_wheel>
-  <xacro:omni_wheel prefix="omni_front_left" parent="base_link" hq="${hq}">
+  <xacro:omni_wheel prefix="omni_front_left_" parent="base_link" hq="${hq}">
     <origin xyz="${omni_front_x} ${omni_front_y} ${omni_front_z}" rpy="0 0 0"/>
   </xacro:omni_wheel>
-  <xacro:omni_wheel prefix="omni_front_right" parent="base_link" hq="${hq}">
+  <xacro:omni_wheel prefix="omni_front_right_" parent="base_link" hq="${hq}">
     <origin xyz="${omni_front_x} -${omni_front_y} ${omni_front_z}" rpy="0 0 0"/>
   </xacro:omni_wheel>

File: rb1_base_description/urdf/bases/rb1_base_v3.urdf.xacro (robot description, xacro)
@@ -2,108 +2,93 @@
 <robot name="rb1_base" xmlns:xacro="http://www.ros.org/wiki/xacro">
   <xacro:macro name="rb1_base_v3" params="publish_bf hq">
-  <!-- Robot mechanical and motor parameters -->
-  <xacro:property name="PI" value="3.1415926535897931"/>
-  <xacro:property name="wheel_width" value="0.175" />
-  <!-- BASE FOOTPRINT -->
-  <xacro:if value="${publish_bf}">
-    <link name="base_footprint"/>
-    <joint name="base_footprint_joint" type="fixed">
-       <origin xyz="0 0 ${wheel_radius - wheel_offset_z}" rpy="0 0 0" />
+    <!-- Robot mechanical and motor parameters -->
+    <xacro:property name="PI" value="3.1415926535897931"/>
+    <xacro:property name="wheel_width" value="0.175" />
+    <!-- BASE FOOTPRINT -->
+    <xacro:if value="${publish_bf}">
+      <link name="base_footprint"/>
+      <joint name="base_footprint_joint" type="fixed">
+        <origin xyz="0 0 ${wheel_radius - wheel_offset_z}" rpy="0 0 0"/>
+        <parent link="base_footprint"/>
+        <child link="base_link"/>
+      </joint>
+    </xacro:if>
+    <!-- BASE_LINK -->
+    <link name="base_link">
+      <inertial>
+        <mass value="25.0" />
+        <origin xyz="0 0 0.07" />
+        <inertia  ixx="0.605" ixy="0.0"  ixz="0.0"  iyy="0.5435"  iyz="0.0"  izz="0.981" />
+      </inertial>
+      <visual>
+        <origin xyz="0 0 0" rpy="0 0 0" />
+        <geometry>
+          <mesh filename="file://$(find rb1_base_description)/meshes/bases/rb1_base_v3_color.dae"/>
+        </geometry>
+      </visual>
+      <collision>
+        <origin xyz="0 0 0" rpy="0 0 0" />
+        <geometry>
+          <mesh filename="file://$(find rb1_base_description)/meshes/bases/rb1_base_v3_color.dae"/>
+        </geometry>
+      </collision>
+    </link>
+    <joint name="front_cover_joint" type="fixed">
+      <origin xyz="0.220 0.0 0.004" rpy="0 0 0 " />
+      <parent link="base_link"/>
+      <child link="front_cover_link" />
+    </joint>
+    <!-- FRONT COVER -->
+    <link name="front_cover_link">
+      <inertial>
+        <mass value="0.25"/>
+        <origin xyz="0 0 0.05"/>
+        <inertia  ixx="0.001" ixy="0.0"  ixz="0.0"  iyy="0.001"  iyz="0.0"  izz="0.001"/>
+      </inertial>
+      <visual>
+        <origin xyz="0 0 0" rpy="0 0 0"/>
+        <geometry>
+          <mesh filename="file://$(find rb1_base_description)/meshes/bases/rb1_front_cover_v3.stl"/>
+        </geometry>
+      </visual>
+      <collision>
+        <origin xyz="0 0 0" rpy="0 0 0"/>
+        <geometry>
+          <mesh filename="file://$(find rb1_base_description)/meshes/bases/rb1_front_cover_v3.dae"/>
+        </geometry>
+      </collision>
+    </link>
+    <joint name="top_covert_joint" type="fixed">
+      <origin xyz="0.0 0.0 0.243" rpy="0 0 0"/>
       <parent link="base_footprint"/>
-      <child link="base_link" />
+      <child link="top_cover_link" />
     </joint>
-  </xacro:if>
-  <!-- BASE_LINK -->
-  <link name="base_link">
-    <inertial>
-      <mass value="25.0" />
-      <origin xyz="0 0 0.07" />
-      <inertia  ixx="0.605" ixy="0.0"  ixz="0.0"  iyy="0.5435"  iyz="0.0"  izz="0.981" />
-    </inertial>
-    <visual>
-      <origin xyz="0 0 0" rpy="0 0 0" />
-      <geometry>
-        <mesh filename="file://$(find rb1_base_description)/meshes/bases/rb1_base_v3_color.dae"/>
-      </geometry>
-    </visual>
-  </link>
-  <joint name="front_cover_joint" type="fixed">
-     <origin xyz="0.220 0.0 0.004" rpy="0 0 0 " />
-     <parent link="base_link"/>
-     <child link="front_cover_link" />
-  </joint>
-  <!-- FRONT COVER -->
-  <link name="front_cover_link">
-    <inertial>
-      <mass value="0.25" />
-      <origin xyz="0 0 0.05" />
-      <inertia  ixx="0.001" ixy="0.0"  ixz="0.0"  iyy="0.001"  iyz="0.0"  izz="0.001" />
-    </inertial>
-    <visual>
-       <origin xyz="0 0 0" rpy="0 0 0" />
-       <xacro:if value="${hq}">
-       <geometry>
-	     <mesh filename="file://$(find rb1_base_description)/meshes/bases/rb1_front_cover_v3.stl"/>
-       </geometry>
-       </xacro:if>
-       <xacro:unless value="${hq}">
-       <geometry>
-       <mesh filename="file://$(find rb1_base_description)/meshes/bases/rb1_front_cover_v3.stl"/>
-       </geometry>
-       </xacro:unless>
-       <material name="black">
-         <color rgba="0.0 0.0 0.0 1"/>
-       </material>
-    </visual>
-    <collision>
-       <origin xyz="0 0 0" rpy="0 0 0 " />
-       <geometry>
-         <mesh filename="file://$(find rb1_base_description)/meshes/bases/rb1_front_cover_v3.dae"/>
-       </geometry>
-    </collision>
-  </link>
-  <joint name="top_covert_joint" type="fixed">
-     <origin xyz="0.0 0.0 0.243" rpy="0 0 0 " />
-     <parent link="base_footprint"/>
-     <child link="top_cover_link" />
-  </joint>
-  <!-- FRONT COVER -->
-  <link name="top_cover_link">
-    <inertial>
-      <mass value="0.25" />
-      <origin xyz="0 0 0" />
-      <inertia  ixx="0.0007" ixy="0.0"  ixz="0.0"  iyy="0.0007"  iyz="0.0"  izz="0.001" />
-    </inertial>
-    <visual>
-       <origin xyz="0 0 0" rpy="0 0 0" />
-       <xacro:if value="${hq}">
-		   <geometry>
-			 <mesh filename="file://$(find rb1_base_description)/meshes/bases/rb1_top_cover_v3.stl"/>
-		   </geometry>
-       </xacro:if>
-       <xacro:unless value="${hq}">
-		   <geometry>
-		   <mesh filename="file://$(find rb1_base_description)/meshes/bases/rb1_top_cover_v3.stl"/>
-		   </geometry>
-       </xacro:unless>
-       <material name="black">
-         <color rgba="0.0 0.0 0.0 1"/>
-       </material>
-    </visual>
-    <collision>
-       <origin xyz="0 0 0" rpy="0 0 0 " />
-       <geometry>
-         <mesh filename="file://$(find rb1_base_description)/meshes/bases/rb1_top_cover_v3.dae"/>
-       </geometry>
-    </collision>
-  </link>
-  <!-- DOCKING CONTACTS -->
-  <joint name="base_docking_joint" type="fixed">
-     <origin xyz="0.030 0.000 0.068" rpy="0 0 0 " />
-     <parent link="front_cover_link"/>
-     <child link="base_docking_contact_link" />
-  </joint>
-  <!-- DOCKING LINK -->
-  <link name="base_docking_contact_link" />
+    <!-- TOP COVER -->
+    <link name="top_cover_link">
+      <inertial>
+        <mass value="0.25" />
+        <origin xyz="0 0 0" />
+        <inertia  ixx="0.0007" ixy="0.0"  ixz="0.0"  iyy="0.0007"  iyz="0.0"  izz="0.001"/>
+      </inertial>
+      <visual>
+        <origin xyz="0 0 0" rpy="0 0 0"/>
+        <geometry>
+          <mesh filename="file://$(find rb1_base_description)/meshes/bases/rb1_top_cover_v3.stl"/>
+        </geometry>
+      </visual>
+      <collision>
+        <origin xyz="0 0 0" rpy="0 0 0"/>
+        <geometry>
+          <mesh filename="file://$(find rb1_base_description)/meshes/bases/rb1_top_cover_v3.dae"/>
+        </geometry>
+      </collision>
+    </link>
+    <!-- DOCKING -->
+    <joint name="base_docking_joint" type="fixed">
+      <origin xyz="0.030 0.000 0.068" rpy="0 0 0 "/>
+      <parent link="front_cover_link"/>
+      <child link="base_docking_contact_link"/>
+    </joint>
+    <link name="base_docking_contact_link"/>
   </xacro:macro>
 </robot>

File: rb1_base_description/urdf/wheels/omni_wheel.urdf.xacro (robot description, xacro)
@@ -1,25 +1,16 @@
 <?xml version="1.0"?>
-<robot name="omnidirectional_wheel" xmlns:xacro="http://www.ros.org/wiki/xacro">
+<robot name="omni_wheel" xmlns:xacro="http://www.ros.org/wiki/xacro">
+  <xacro:include filename="$(find rb1_base_description)/urdf/inertia.urdf.xacro"/>
+  <!-- CONSTANTS -->
   <xacro:property name="M_PI" value="3.1415926535897931" />
-  <!-- Wheels -->
   <xacro:property name="omni_wheel_radius" value="0.051" />
   <xacro:property name="omni_wheel_height" value="0.040" />
-  <xacro:property name="omni_wheel_mass" value="0.3" /> <!-- in kg-->
-  <xacro:macro name="cylinder_inertia" params="m r h">
-    <inertia  ixx="${m*(3*r*r+h*h)/12}" ixy = "0" ixz = "0"
-              iyy="${m*(3*r*r+h*h)/12}" iyz = "0"
-              izz="${m*r*r/2}"
-     />
-  </xacro:macro>
+  <xacro:property name="omni_wheel_mass" value="0.3" />
   <xacro:macro name="omni_wheel" params="prefix parent *origin hq">
-<!--WHEEL TIRE -->
-    <!-- joint name="joint_${name}_wheel" type="continuous" -->
+    <!--WHEEL TIRE -->
     <joint name="${prefix}wheel_joint" type="fixed">
+      <xacro:insert_block name="origin" />
       <parent link="${parent}"/>
       <child link="${prefix}wheel_link"/>
-      <xacro:insert_block name="origin" />
-      <axis xyz="0 1 0" rpy="0 0 0" />
-      <limit effort="100" velocity="100"/>
-      <joint_properties damping="0.0" friction="0.0"/>
     </joint>
     <link name="${prefix}wheel_link">
@@ -29,5 +20,5 @@
           <origin xyz="0 0 0" rpy="0 0 0" />
           <geometry>
-				<mesh filename="file://$(find rb1_base_description)/meshes/wheels/rb1v2_omniwheel.dae" />
+            <mesh filename="file://$(find rb1_base_description)/meshes/wheels/rb1v2_omniwheel.dae" />
           </geometry>
         </xacro:if>
@@ -41,51 +32,23 @@
       </visual>
       <collision>
-      <origin xyz="0 0 0" rpy="${M_PI/2} 0 0" />
+        <origin xyz="0 0 0" rpy="${M_PI/2} 0 0" />
         <geometry>
           <cylinder length="0.03" radius="${omni_wheel_radius}" />
         </geometry>
       </collision>
-      <!--collision>
-      <origin xyz="0 0 0" rpy="${M_PI/2} 0 0" />
-       <geometry>
-         <sphere radius="${omni_wheel_radius}"/>
-       </geometry>
-     </collision-->
       <inertial>
         <mass value="${wheel_mass}" />
         <origin xyz="0 0 0" />
-        <xacro:cylinder_inertia  m="${omni_wheel_mass}" r="${omni_wheel_radius}" h="${omni_wheel_height}" />
-        <!-- inertia  ixx="0.001" ixy="0.0"  ixz="0.0"  iyy="0.001"  iyz="0.0"  izz="0.001" / -->
+        <xacro:solid_cylinder_inertia  m="${omni_wheel_mass}" r="${omni_wheel_radius}" h="${omni_wheel_height}" />
       </inertial>
     </link>
-    <!-- transmission name="${name}_wheel_joint_trans">
-      <type>transmission_interface/SimpleTransmission</type>
-      <joint name="joint_${name}_wheel" />
-      <actuator name="${name}_wheel_joint_motor">
-        <hardwareInterface>EffortJointInterface</hardwareInterface>
-        <mechanicalReduction>1</mechanicalReduction>
-      </actuator>
-    </transmission -->
-    <gazebo reference="${prefix}wheel">
-		<mu1 value="0"/>
-		<mu2 value="0"/>
-		<kp value="10000000.0" />
-		<kd value="1.0" />
-		<fdir1 value="1 0 0"/>
-		<material>Gazebo/Black</material>
-		<turnGravityOff>false</turnGravityOff>
+    <gazebo reference="${prefix}wheel_link">
+      <mu1>0.001</mu1>
+      <mu2>0.001</mu2>
+      <kp>2.75e7</kp>
+      <kd>8.25e1</kd>
+      <fdir1>0 0 0</fdir1>
+      <maxContacts>4</maxContacts>
     </gazebo>
-    <!--gazebo reference="${name}_wheel">
-		<kp>500000.0</kp>
-		<kd>10.0</kd>
-		<mu1>10</mu1>
-		<mu2>10</mu2>
-		<fdir1>1 0 0</fdir1>
-		<maxVel>1.0</maxVel>
-		<minDepth>0.003</minDepth>
-		<material>Gazebo/Black</material>
-		<turnGravityOff>false</turnGravityOff>
-		<implicitSpringDamper>1</implicitSpringDamper>
-    </gazebo-->
   </xacro:macro>
 </robot>

File: rb1_base_description/urdf/wheels/rubber_wheel.urdf.xacro (robot description, xacro)
@@ -1,62 +1,58 @@
 <?xml version="1.0"?>
 <robot name="wheel" xmlns:xacro="http://www.ros.org/wiki/xacro">
-	<xacro:include filename="$(find rb1_base_description)/urdf/wheels/rubber_wheel.transmission.xacro"/>
-	<xacro:include filename="$(find rb1_base_description)/urdf/wheels/rubber_wheel.gazebo.xacro"/>
-	<xacro:property name="M_PI" value="3.1415926535897931" />
-	<!-- Wheels -->
-	<xacro:property name="wheel_radius" value="0.076" />
-	<xacro:property name="wheel_height" value="0.025" />
-	<xacro:property name="wheel_mass" value="1.0" /> <!-- in kg-->
-	<xacro:macro name="cylinder_inertia" params="m r h">
-		<inertia	ixx="${m*(3*r*r+h*h)/12}" ixy = "0" ixz = "0"
-					iyy="${m*(3*r*r+h*h)/12}" iyz = "0"
-					izz="${m*r*r/2}" />
-	</xacro:macro>
-	<xacro:macro name="rubber_wheel" params="prefix parent *origin reflect hq">
-	<!--WHEEL TIRE -->
-	<joint name="${prefix}_wheel_joint" type="continuous">
-		<parent link="${parent}"/>
-		<child link="${prefix}_wheel_link"/>
-		<xacro:insert_block name="origin" />
-		<axis xyz="0 1 0" rpy="0 0 0" />
-		<limit effort="100" velocity="100"/>
-		<joint_properties damping="0.0" friction="0.0"/>
-	</joint>
-	<link name="${prefix}_wheel_link">
-		<visual>
-		<!-- HIGH RESOLUTION WHEELS -->
-		<xacro:if value="${hq}">
-			<origin xyz="0 0 0" rpy="0 0 0" />
-			<geometry>
-				<xacro:if value="${reflect}">
-					<mesh filename="file://$(find rb1_base_description)/meshes/wheels/wheel_rubber_6inch.dae" />
-				</xacro:if>
-				<xacro:unless value="${reflect}">
-					<mesh filename="file://$(find rb1_base_description)/meshes/wheels/wheel_rubber_6inch.dae" />
-				</xacro:unless>
-			</geometry>
-		</xacro:if>
-		<!-- LOW RESOLUTION WHEELS -->
-		<xacro:unless value="${hq}">
-			<origin xyz="0 0 0" rpy="${M_PI/2} 0 0" />
-			<geometry>
-				<cylinder length="${wheel_height}" radius="${wheel_radius}" />
-			</geometry>
-		</xacro:unless>
-		</visual>
+  <xacro:include filename="$(find rb1_base_description)/urdf/inertia.urdf.xacro"/>
+  <!-- CONSTANTS -->
+  <xacro:property name="M_PI" value="3.1415926535897931"/>
+  <xacro:property name="wheel_radius" value="0.076"/>
+  <xacro:property name="wheel_height" value="0.025"/>
+  <xacro:property name="wheel_mass" value="1.0"/>
+  <!-- WHEEL XACRO -->
+  <xacro:macro name="rubber_wheel" params="prefix parent *origin reflect hq">
+    <!--TIRE -->
+    <joint name="${prefix}wheel_joint" type="continuous">
+      <xacro:insert_block name="origin"/>
+      <parent link="${parent}"/>
+      <child link="${prefix}wheel_link"/>
+      <axis xyz="0 1 0" rpy="0 0 0" />
+      <limit effort="100" velocity="100"/>
+      <dynamics damping="0.05" friction="0.1"/>
+    </joint>
+    <link name="${prefix}wheel_link">
+      <visual>
+        <!-- HIGH RESOLUTION WHEELS -->
+        <xacro:if value="${hq}">
+          <origin xyz="0 0 0" rpy="0 0 0"/>
+          <geometry>
+            <mesh filename="file://$(find rb1_base_description)/meshes/wheels/wheel_rubber_6inch.dae"/>
+          </geometry>
+        </xacro:if>
+        <!-- LOW RESOLUTION WHEELS -->
+        <xacro:unless value="${hq}">
+          <origin xyz="0 0 0" rpy="${M_PI/2} 0 0"/>
+          <geometry>
+            <cylinder length="${wheel_height}" radius="${wheel_radius}"/>
+          </geometry>
+        </xacro:unless>
+      </visual>
       <collision>
-		<origin xyz="0 0 0" rpy="${M_PI/2} 0 0" />
-        <geometry>
-          <cylinder length="${wheel_height}" radius="${wheel_radius}" />
-        </geometry>
-      </collision>
-      <inertial>
-        <mass value="${wheel_mass}" />
         <origin xyz="0 0 0" rpy="${M_PI/2} 0 0"/>
-        <xacro:cylinder_inertia   m="${wheel_mass}" r="${wheel_radius}" h="${wheel_height}" />
-      </inertial>
-    </link>
-	<xacro:rubber_wheel_transmission prefix="${prefix}" />
-	<xacro:rubber_wheel_gazebo prefix="${prefix}" />
+          <geometry>
+            <cylinder length="${wheel_height}" radius="${wheel_radius}"/>
+          </geometry>
+        </collision>
+        <inertial>
+          <mass value="${wheel_mass}"/>
+          <origin xyz="0 0 0" rpy="${M_PI/2} 0 0"/>
+          <xacro:solid_cylinder_inertia m="${wheel_mass}" r="${wheel_radius}" h="${wheel_height}"/>
+        </inertial>
+      </link>
+    <gazebo reference="${prefix}wheel_link">
+      <mu1>0.95</mu1>
+      <mu2>0.90</mu2>
+      <kp>2.75e6</kp>
+      <kd>8.25e1</kd>
+      <fdir1>0 0 0</fdir1>
+      <maxContacts>4</maxContacts>
+    </gazebo>
   </xacro:macro>
 </robot>
