Commit message: Added elevator description

File: rb1_base_description/urdf/rb1_base.urdf.xacro (robot description, xacro)
@@ -13,4 +13,6 @@
 	<!-- IMPORT SENSORS -->
 	<xacro:include filename="$(find robotnik_sensors)/urdf/all_sensors.urdf.xacro"/>
+	<!-- IMPORT ELEVATOR -->
+	<xacro:include filename="$(find rb1_base_description)/urdf/elevator/elevator.urdf.xacro"/>
 	<!-- ***************** -->
 	<!-- GLOBAL PARAMETERS -->
@@ -31,4 +33,7 @@
 	<xacro:property name="omni_front_y" value="0.1535" />
 	<xacro:property name="omni_front_z" value="0.0258" />
+	<xacro:property name="elevator_x" value="0.0" />
+	<xacro:property name="elevator_y" value="0.0" />
+	<xacro:property name="elevator_z" value="0.0213" />
 	<!-- *************** -->
 	<!-- ROBOT COMPONENTS -->
@@ -56,4 +61,8 @@
 			<origin xyz="${omni_front_x} -${omni_front_y} ${omni_front_z}" rpy="0 0 0"/>
 		</xacro:omni_wheel>
+		<!-- ELEVATOR_PLATFORM -->
+		<xacro:elevator_platform parent="base_link" hq="${hq}">
+			<origin xyz="${omni_front_x} -${omni_front_y} ${omni_front_z}" rpy="0 0 0"/>
+		</xacro:elevator_platform>
 		<!-- SENSORS -->
 		<!-- LASER -->
