Commit message: Last changes

File: rb1_base_description/urdf/bases/base.urdf.xacro (robot description, xacro)
@@ -39,10 +39,10 @@
 			<xacro:if value="${hq}">
 				<geometry>
-					<mesh filename="package://rb1_base_description/meshes/bases/rb1v2_base.dae"/>
+					<mesh filename="package://rb1_base_description/meshes/bases/rb1v3_base.dae"/>
 				</geometry>
 			</xacro:if>
 			<xacro:unless value="${hq}">
 				<geometry>
-					<mesh filename="package://rb1_base_description/meshes/bases/rb1v2_base.stl"/>
+					<mesh filename="package://rb1_base_description/meshes/bases/rb1v3_base.stl"/>
 				</geometry>
 			</xacro:unless>
@@ -54,5 +54,5 @@
 			<origin xyz="0 0 0" rpy="0 0 0 " />
 			<geometry>
-				<mesh filename="package://rb1_base_description/meshes/bases/rb1v2_base.dae"/>
+				<mesh filename="package://rb1_base_description/meshes/bases/rb1v3_base.dae"/>
 			</geometry>
 		</collision>

File: rb1_base_description/urdf/rb1_base.urdf.xacro (robot description, xacro)
@@ -22,13 +22,13 @@
 	<!-- FOR RUBBER WHEEL -->
 	<xacro:property name="wheel_offset_x" value="0.0" />    <!-- x,y,z in translation from base_link to the center of the wheel -->
-	<xacro:property name="wheel_offset_y" value="0.217" />
-	<xacro:property name="wheel_offset_z" value="0.051" />
+	<xacro:property name="wheel_offset_y" value="0.218" />
+	<xacro:property name="wheel_offset_z" value="0.0512" />
 	<!-- FOR OMNI WHEEL -->
 	<xacro:property name="omni_back_x" value="0.195" />
 	<xacro:property name="omni_back_y" value="0.0" />
-	<xacro:property name="omni_back_z" value="0.0265" />
-	<xacro:property name="omni_front_x" value="0.133" />
-	<xacro:property name="omni_front_y" value="0.148" />
-	<xacro:property name="omni_front_z" value="0.0265" />
+	<xacro:property name="omni_back_z" value="0.0258" />
+	<xacro:property name="omni_front_x" value="0.132" />
+	<xacro:property name="omni_front_y" value="0.1535" />
+	<xacro:property name="omni_front_z" value="0.0258" />
 	<!-- *************** -->
 	<!-- ROBOT COMPONENTS -->
@@ -69,11 +69,11 @@
 		<!-- Name the components as base_front_laser or base_laser or front_laser or
 		a name which identify uniquely the component within the robot -->
-		<xacro:sensor_hokuyo_ust10lx name="base_front_laser" parent="base_link">
-			<origin xyz="0.223 0.0 0.159" rpy="0 3.1416 3.1416"/>
-		</xacro:sensor_hokuyo_ust10lx>
+		<xacro:sensor_rplidar_a2 name="base_front_laser" parent="base_link">
+			<origin xyz="0.210 0.0 0.199" rpy="3.1415 0 0"/>
+		</xacro:sensor_rplidar_a2>
 		<!-- CAMERA -->
-		<xacro:sensor_orbbec_astra name="base_front_camera" parent="base_link">
+		<!--xacro:sensor_orbbec_astra name="base_front_camera" parent="base_link">
 			<origin xyz="0.234 0.0125 0.107" rpy="0 0 0"/>
-		</xacro:sensor_orbbec_astra>
+		</xacro:sensor_orbbec_astra-->
 		<!-- xacro:sensor_kinect name="front_camera" parent="base_link">
 			<origin xyz="0.6 0.0 0.102" rpy="0 0 0"/>

File: rb1_base_description/urdf/wheels/omni_wheel.urdf.xacro (robot description, xacro)
@@ -29,5 +29,5 @@
           <origin xyz="0 0 0" rpy="0 0 0" />
           <geometry>
-				<mesh filename="package://rb1_base_description/meshes/wheels/rb1v2_omniwheel.dae" />
+				<mesh filename="package://rb1_base_description/meshes/wheels/rb1v3_omniwheel.dae" />
           </geometry>
         </xacro:if>

File: rb1_base_description/urdf/wheels/rubber_wheel.urdf.xacro (robot description, xacro)
@@ -30,8 +30,8 @@
 			<geometry>
 				<xacro:if value="${reflect}">
-					<mesh filename="package://rb1_base_description/meshes/wheels/wheel_rubber_6inch.dae" />
+					<mesh filename="package://rb1_base_description/meshes/wheels/rb1v3_rubberwheel_6inch.dae" />
 				</xacro:if>
 				<xacro:unless value="${reflect}">
-					<mesh filename="package://rb1_base_description/meshes/wheels/wheel_rubber_6inch.dae" />
+					<mesh filename="package://rb1_base_description/meshes/wheels/rb1v3_rubberwheel_6inch.dae" />
 				</xacro:unless>
 			</geometry>

Commit message: Fixed distances of rb1 model

File: rb1_base_description/urdf/bases/base.urdf.xacro (robot description, xacro)
@@ -39,10 +39,10 @@
 			<xacro:if value="${hq}">
 				<geometry>
-					<mesh filename="package://rb1_base_description/meshes/bases/rb1v3_base.dae"/>
+					<mesh filename="package://rb1_base_description/meshes/bases/rb1v2_base.dae"/>
 				</geometry>
 			</xacro:if>
 			<xacro:unless value="${hq}">
 				<geometry>
-					<mesh filename="package://rb1_base_description/meshes/bases/rb1v3_base.stl"/>
+					<mesh filename="package://rb1_base_description/meshes/bases/rb1v2_base.stl"/>
 				</geometry>
 			</xacro:unless>
@@ -54,5 +54,5 @@
 			<origin xyz="0 0 0" rpy="0 0 0 " />
 			<geometry>
-				<mesh filename="package://rb1_base_description/meshes/bases/rb1v3_base.dae"/>
+				<mesh filename="package://rb1_base_description/meshes/bases/rb1v2_base.dae"/>
 			</geometry>
 		</collision>

File: rb1_base_description/urdf/elevator/elevator.urdf.xacro (robot description, xacro)
@@ -2,5 +2,5 @@
 <robot xmlns:xacro="http://www.ros.org/wiki/xacro">
 	<!--xacro:include filename="$(find rb1_base_description)/urdf/bases/rb1_elevator.gazebo.xacro" /-->
-	<xacro:macro name="elevator_platform" params="parent hq origin">
+	<xacro:macro name="elevator_platform" params="parent hq *origin">
 	<!-- PARAMS: -->
 	<!-- name : name of the link: -->
@@ -23,5 +23,5 @@
 			<origin xyz="0 0 0" rpy="0 0 0" />
 			<xacro:if value="${hq}">
-				<geomet
+				<geometry>
 					<mesh filename="package://rb1_base_description/meshes/elevator/rb1_elevator_base.dae"/>
 				</geometry>
@@ -45,9 +45,9 @@
 	<!-- ELEVATOR PLATFORM -->
 	<joint name="elevator_platform_joint" type="prismatic">
-			<origin xyz="0.0 0.0 0.0041" rpy="0 0 0 " />
+			<origin xyz="0.0 0.0 0.041" rpy="0 0 0 " />
 			<parent link="elevator_base_link"/>
 			<child link="elevator_platform_link" />
 			<axis xyz="0 0 1"/>
-			<limit lower="0.0" upper="0.0034" velocity="0.5"/>
+			<limit effort="1.0" lower="0.0" upper="0.034" velocity="0.5"/>
 	</joint>
 	<link name="elevator_platform_link">

File: rb1_base_description/urdf/rb1_base.urdf.xacro (robot description, xacro)
@@ -24,5 +24,5 @@
 	<!-- FOR RUBBER WHEEL -->
 	<xacro:property name="wheel_offset_x" value="0.0" />    <!-- x,y,z in translation from base_link to the center of the wheel -->
-	<xacro:property name="wheel_offset_y" value="0.218" />
+	<xacro:property name="wheel_offset_y" value="0.2165" />
 	<xacro:property name="wheel_offset_z" value="0.0512" />
 	<!-- FOR OMNI WHEEL -->
@@ -30,10 +30,13 @@
 	<xacro:property name="omni_back_y" value="0.0" />
 	<xacro:property name="omni_back_z" value="0.0258" />
-	<xacro:property name="omni_front_x" value="0.132" />
-	<xacro:property name="omni_front_y" value="0.1535" />
+	<xacro:property name="omni_front_x" value="0.133" />
+	<xacro:property name="omni_front_y" value="0.148" />
 	<xacro:property name="omni_front_z" value="0.0258" />
+	<!-- ******************* -->
+	<!-- ELEVATOR PARAMETERS -->
+	<!-- ******************* -->
 	<xacro:property name="elevator_x" value="0.0" />
 	<xacro:property name="elevator_y" value="0.0" />
-	<xacro:property name="elevator_z" value="0.0213" />
+	<xacro:property name="elevator_z" value="0.213" />
 	<!-- *************** -->
 	<!-- ROBOT COMPONENTS -->
@@ -63,5 +66,5 @@
 		<!-- ELEVATOR_PLATFORM -->
 		<xacro:elevator_platform parent="base_link" hq="${hq}">
-			<origin xyz="${omni_front_x} -${omni_front_y} ${omni_front_z}" rpy="0 0 0"/>
+			<origin xyz="${elevator_x} -${elevator_y} ${elevator_z}" rpy="0 0 0"/>
 		</xacro:elevator_platform>
 		<!-- SENSORS -->
