Commit message: Now all the models can be selected via environment variable RB1_BASE_VERSION

File: rb1_base_description/urdf/bases/rb1_base_v2.urdf.xacro (robot description, xacro)
@@ -1,5 +1,5 @@
 <?xml version="1.0"?>
 <robot name="rb1_base" xmlns:xacro="http://www.ros.org/wiki/xacro">
-  <xacro:macro name="rb1_base" params="name publish_bf hq">
+  <xacro:macro name="rb1_base_v2" params="name publish_bf hq">
   <!-- Robot mechanical and motor parameters -->
   <xacro:property name="PI" value="3.1415926535897931"/>
@@ -92,5 +92,5 @@
      <child link="base_docking_contact" />
   </joint>
-  <!-- FRONT COVER -->
+  <!-- DOCKING LINK -->
   <link name="base_docking_contact" />
   </xacro:macro>
