Commit message: URDF Kinova platform: Update to kinetic

File: rb1_base_description/urdf/bases/rb1_base_v3.urdf.xacro (robot description, xacro)
@@ -24,5 +24,5 @@
   <link name="${prefix}base_link">
     <inertial>
-      <mass value="25.0" />
+      <mass value="26.0" />
       <origin xyz="0 0 0" />
       <inertia  ixx="0.007" ixy="0.0"  ixz="0.0"  iyy="0.007"  iyz="0.0"  izz="0.78" />

Commit message: Changed base_link and rubber_wheel inertias

File: rb1_base_description/urdf/bases/rb1_base_v3.urdf.xacro (robot description, xacro)
@@ -8,10 +8,10 @@
   <xacro:if value="${publish_bf}">
     <link name="${prefix}base_footprint">
-      <visual>
+      <!--visual>
           <origin xyz="0 0 0" rpy="0 0 0" />
           <geometry>
              <box size="0.001 0.001 0.001" />
           </geometry>
-      </visual>
+      </visual-->
     </link>
     <joint name="${prefix}base_footprint_joint" type="fixed">
@@ -24,7 +24,7 @@
   <link name="${prefix}base_link">
     <inertial>
-      <mass value="26.0" />
+      <mass value="25.0" />
       <origin xyz="0 0 0" />
-      <inertia  ixx="0.007" ixy="0.0"  ixz="0.0"  iyy="0.007"  iyz="0.0"  izz="0.78" />
+      <inertia  ixx="0.605" ixy="0.0"  ixz="0.0"  iyy="0.5435"  iyz="0.0"  izz="0.981" />
     </inertial>
     <visual>

File: rb1_base_description/urdf/wheels/rubber_wheel.urdf.xacro (robot description, xacro)
@@ -53,5 +53,5 @@
       <inertial>
         <mass value="${wheel_mass}" />
-        <origin xyz="0 0 0" />
+        <origin xyz="0 0 0" rpy="${M_PI/2} 0 0"/>
         <cylinder_inertia  m="${wheel_mass}" r="${wheel_radius}" h="${wheel_height}" />
       </inertial>

Commit message: Changed omni-wheel collision sphere -> cylinder

File: rb1_base_description/urdf/bases/rb1_base_v3.urdf.xacro (robot description, xacro)
@@ -44,10 +44,10 @@
        </material>
     </visual>
-    <collision>
+    <!--collision>
        <origin xyz="0 0 0" rpy="0 0 0 " />
        <geometry>
          <mesh filename="package://rb1_base_description/meshes/bases/rb1_base_v3.dae"/>
        </geometry>
-    </collision>
+    </collision-->
   </link>
   <joint name="${prefix}front_cover_joint" type="fixed">

File: rb1_base_description/urdf/wheels/omni_wheel.urdf.xacro (robot description, xacro)
@@ -40,16 +40,16 @@
         </xacro:unless>
       </visual>
-      <!-- collision>
+      <collision>
       <origin xyz="0 0 0" rpy="${M_PI/2} 0 0" />
         <geometry>
-          <cylinder length="${omni_wheel_height}" radius="${omni_wheel_radius}" />
+          <cylinder length="0.03" radius="${omni_wheel_radius}" />
         </geometry>
-      </collision -->
-      <collision>
+      </collision>
+      <!--collision>
       <origin xyz="0 0 0" rpy="${M_PI/2} 0 0" />
        <geometry>
          <sphere radius="${omni_wheel_radius}"/>
        </geometry>
-      </collision>
+     </collision-->
       <inertial>
         <mass value="${wheel_mass}" />

Commit message: Changed color base from dark grey to black

File: rb1_base_description/urdf/bases/rb1_base_v3.urdf.xacro (robot description, xacro)
@@ -40,6 +40,6 @@
        </geometry>
        </xacro:unless>
-       <material name="darkgrey">
-         <color rgba="0.1 0.1 0.1 1"/>
+       <material name="black">
+         <color rgba="0.0 0.0 0.0 1"/>
        </material>
     </visual>

Commit message: add collision to rb1

File: rb1_base_description/urdf/bases/rb1_base_v3.urdf.xacro (robot description, xacro)
@@ -44,10 +44,10 @@
        </material>
     </visual>
-    <!--collision>
+    <collision>
        <origin xyz="0 0 0" rpy="0 0 0 " />
        <geometry>
          <mesh filename="package://rb1_base_description/meshes/bases/rb1_base_v3.dae"/>
        </geometry>
-    </collision-->
+    </collision>
   </link>
   <joint name="${prefix}front_cover_joint" type="fixed">
