Commit message: removed gazebo plugin (in effort) and changed wheel controller to velocity

File: rb1_base_description/urdf/bases/rb1_base.urdf.xacro (robot description, xacro)
@@ -1,5 +1,5 @@
 <?xml version="1.0"?>
 <robot name="rb1_base" xmlns:xacro="http://www.ros.org/wiki/xacro">
-  <xacro:include filename="$(find rb1_base_description)/urdf/bases/rb1_base.gazebo.xacro" />
+  <!-- xacro:include filename="$(find rb1_base_description)/urdf/bases/rb1_base.gazebo.xacro" / -->
   <xacro:macro name="rb1_base" params="name publish_bf hq">
   <!-- Robot mechanical and motor parameters -->

File: rb1_base_description/urdf/wheels/rubber_wheel.urdf.xacro (robot description, xacro)
@@ -12,5 +12,5 @@
   </xacro:macro>
   <xacro:macro name="rubber_wheel" params="name parent *origin reflect hq">
-<!--WHEEL TIRE -->
+  <!--WHEEL TIRE -->
     <joint name="joint_${name}_wheel" type="continuous">
       <parent link="${parent}"/>
@@ -27,10 +27,10 @@
           <origin xyz="0 0 0" rpy="0 0 0" />
           <geometry>
-						<xacro:if value="${reflect}">
-							<mesh filename="package://rb1_base_description/meshes/wheels/wheel_rubber_6inch.dae" />
-						</xacro:if>
-						<xacro:unless value="${reflect}">
-							<mesh filename="package://rb1_base_description/meshes/wheels/wheel_rubber_6inch.dae" />
-						</xacro:unless>
+			<xacro:if value="${reflect}">
+				<mesh filename="package://rb1_base_description/meshes/wheels/wheel_rubber_6inch.dae" />
+			</xacro:if>
+			<xacro:unless value="${reflect}">
+				<mesh filename="package://rb1_base_description/meshes/wheels/wheel_rubber_6inch.dae" />
+			</xacro:unless>
           </geometry>
         </xacro:if>
@@ -59,10 +59,12 @@
       <type>transmission_interface/SimpleTransmission</type>
       <joint name="joint_${name}_wheel">
-          <hardwareInterface>EffortJointInterface</hardwareInterface>
+          <!-- for the gazebo plugin -->
+          <!-- hardwareInterface>EffortJointInterface</hardwareInterface -->
+          <!-- for ros control controller -->
+          <hardwareInterface>VelocityJointInterface</hardwareInterface>
       </joint>
       <actuator name="${name}_wheel_joint_motor">
-        <!-- hardwareInterface>EffortJointInterface</hardwareInterface -->
         <mechanicalReduction>1</mechanicalReduction>
-        <motorTorqueConstant>10</motorTorqueConstant>
+        <motorTorqueConstant>20</motorTorqueConstant>
       </actuator>
     </transmission>

Commit message: rb1_base_description: added contact link

File: rb1_base_description/urdf/bases/rb1_base.urdf.xacro (robot description, xacro)
@@ -87,4 +87,12 @@
     </collision>
   </link>
+  <!-- DOCKING CONTACTS -->
+  <joint name="base_docking_joint" type="fixed">
+     <origin xyz="0.030 0.000 0.068" rpy="0 0 0 " />
+     <parent link="front_cover_link"/>
+     <child link="base_docking_contact" />
+  </joint>
+  <!-- FRONT COVER -->
+  <link name="base_docking_contact" />
   </xacro:macro>
 </robot>

Commit message: Changed inertia of base_link in each base version

File: rb1_base_description/urdf/bases/rb1_base.urdf.xacro (robot description, xacro)
@@ -26,5 +26,5 @@
       <mass value="25.0" />
       <origin xyz="0 0 0" />
-      <inertia  ixx="0.007" ixy="0.0"  ixz="0.0"  iyy="0.007"  iyz="0.0"  izz="0.78" />
+      <inertia  ixx="0.605" ixy="0.0"  ixz="0.0"  iyy="0.5435"  iyz="0.0"  izz="0.981" />
     </inertial>
     <visual>

File: rb1_base_description/urdf/bases/rb1_base_v0.urdf.xacro (robot description, xacro)
@@ -26,5 +26,5 @@
       <mass value="25.0" />
       <origin xyz="0 0 0" />
-      <inertia  ixx="1.0" ixy="0.0"  ixz="0.0"  iyy="1.0"  iyz="0.0"  izz="1.0" />
+      <inertia  ixx="0.605" ixy="0.0"  ixz="0.0"  iyy="0.5435"  iyz="0.0"  izz="0.981" />
     </inertial>
     <visual>

File: rb1_base_description/urdf/bases/rb1_base_v1.urdf.xacro (robot description, xacro)
@@ -26,5 +26,5 @@
       <mass value="25.0" />
       <origin xyz="0 0 0" />
-      <inertia  ixx="0.007" ixy="0.0"  ixz="0.0"  iyy="0.007"  iyz="0.0"  izz="0.78" />
+      <inertia  ixx="0.605" ixy="0.0"  ixz="0.0"  iyy="0.5435"  iyz="0.0"  izz="0.981" />
     </inertial>
     <visual>

File: rb1_base_description/urdf/bases/rb1_base_v2.urdf.xacro (robot description, xacro)
@@ -26,5 +26,5 @@
       <mass value="25.0" />
       <origin xyz="0 0 0" />
-      <inertia  ixx="0.007" ixy="0.0"  ixz="0.0"  iyy="0.007"  iyz="0.0"  izz="0.78" />
+      <inertia  ixx="0.605" ixy="0.0"  ixz="0.0"  iyy="0.5435"  iyz="0.0"  izz="0.981" />
     </inertial>
     <visual>

Commit message: Changed package to find for each xacro

File: rb1_base_description/urdf/bases/rb1_base.urdf.xacro (robot description, xacro)
@@ -32,10 +32,10 @@
        <xacro:if value="${hq}">
        <geometry>
-         <mesh filename="package://rb1_base_description/meshes/bases/rb1v2_base.dae"/>
+         <mesh filename="file://$(find rb1_base_description)/meshes/bases/rb1v2_base.dae"/>
        </geometry>
        </xacro:if>
        <xacro:unless value="${hq}">
        <geometry>
-       <mesh filename="package://rb1_base_description/meshes/bases/rb1v2_base.stl"/>
+       <mesh filename="file://$(find rb1_base_description)/meshes/bases/rb1v2_base.stl"/>
        </geometry>
        </xacro:unless>
@@ -47,5 +47,5 @@
        <origin xyz="0 0 0" rpy="0 0 0 " />
        <geometry>
-         <mesh filename="package://rb1_base_description/meshes/bases/rb1v2_base.dae"/>
+         <mesh filename="file://$(find rb1_base_description)/meshes/bases/rb1v2_base.dae"/>
        </geometry>
     </collision>
@@ -67,10 +67,10 @@
        <xacro:if value="${hq}">
        <geometry>
-	     <mesh filename="package://rb1_base_description/meshes/bases/rb1v2_front_cover.dae"/>
+	     <mesh filename="file://$(find rb1_base_description)/meshes/bases/rb1v2_front_cover.dae"/>
        </geometry>
        </xacro:if>
        <xacro:unless value="${hq}">
        <geometry>
-       <mesh filename="package://rb1_base_description/meshes/bases/rb1v2_front_cover.stl"/>
+       <mesh filename="file://$(find rb1_base_description)/meshes/bases/rb1v2_front_cover.stl"/>
        </geometry>
        </xacro:unless>
@@ -82,5 +82,5 @@
        <origin xyz="0 0 0" rpy="0 0 0 " />
        <geometry>
-         <mesh filename="package://rb1_base_description/meshes/bases/rb1v2_front_cover.dae"/>
+         <mesh filename="file://$(find rb1_base_description)/meshes/bases/rb1v2_front_cover.dae"/>
        </geometry>
     </collision>

File: rb1_base_description/urdf/bases/rb1_base_v0.urdf.xacro (robot description, xacro)
@@ -32,10 +32,10 @@
        <xacro:if value="${hq}">
        <geometry>
-         <mesh filename="package://rb1_base_description/meshes/bases/rb1v0_base.dae"/>
+         <mesh filename="file://$(find rb1_base_description)/meshes/bases/rb1v0_base.dae"/>
        </geometry>
        </xacro:if>
        <xacro:unless value="${hq}">
        <geometry>
-       <mesh filename="package://rb1_base_description/meshes/bases/rb1v0_base.stl"/>
+       <mesh filename="file://$(find rb1_base_description)/meshes/bases/rb1v0_base.stl"/>
        </geometry>
        </xacro:unless>
@@ -47,5 +47,5 @@
        <origin xyz="0 0 0" rpy="0 0 0 " />
        <geometry>
-         <mesh filename="package://rb1_base_description/meshes/bases/rb1v0_base.dae"/>
+         <mesh filename="file://$(find rb1_base_description)/meshes/bases/rb1v0_base.dae"/>
        </geometry>
     </collision>

File: rb1_base_description/urdf/bases/rb1_base_v1.urdf.xacro (robot description, xacro)
@@ -32,10 +32,10 @@
        <xacro:if value="${hq}">
        <geometry>
-	     <mesh filename="package://rb1_base_description/meshes/bases/rb1v1_base.dae"/>
+	     <mesh filename="file://$(find rb1_base_description)/meshes/bases/rb1v1_base.dae"/>
        </geometry>
        </xacro:if>
        <xacro:unless value="${hq}">
        <geometry>
-       <mesh filename="package://rb1_base_description/meshes/bases/rb1v1_base.stl"/>
+       <mesh filename="file://$(find rb1_base_description)/meshes/bases/rb1v1_base.stl"/>
        </geometry>
        </xacro:unless>
@@ -47,5 +47,5 @@
        <origin xyz="0 0 0" rpy="0 0 0 " />
        <geometry>
-         <mesh filename="package://rb1_base_description/meshes/bases/rb1v1_base.dae"/>
+         <mesh filename="file://$(find rb1_base_description)/meshes/bases/rb1v1_base.dae"/>
        </geometry>
     </collision>

File: rb1_base_description/urdf/bases/rb1_base_v2.urdf.xacro (robot description, xacro)
@@ -32,10 +32,10 @@
        <xacro:if value="${hq}">
        <geometry>
-	     <mesh filename="package://rb1_base_description/meshes/bases/rb1v2_base.dae"/>
+	     <mesh filename="file://$(find rb1_base_description)/meshes/bases/rb1v2_base.dae"/>
        </geometry>
        </xacro:if>
        <xacro:unless value="${hq}">
        <geometry>
-       <mesh filename="package://rb1_base_description/meshes/bases/rb1v2_base.stl"/>
+       <mesh filename="file://$(find rb1_base_description)/meshes/bases/rb1v2_base.stl"/>
        </geometry>
        </xacro:unless>
@@ -47,5 +47,5 @@
        <origin xyz="0 0 0" rpy="0 0 0 " />
        <geometry>
-         <mesh filename="package://rb1_base_description/meshes/bases/rb1v2_base.dae"/>
+         <mesh filename="file://$(find rb1_base_description)/meshes/bases/rb1v2_base.dae"/>
        </geometry>
     </collision>
@@ -67,10 +67,10 @@
        <xacro:if value="${hq}">
        <geometry>
-	     <mesh filename="package://rb1_base_description/meshes/bases/rb1v2_front_cover.dae"/>
+	     <mesh filename="file://$(find rb1_base_description)/meshes/bases/rb1v2_front_cover.dae"/>
        </geometry>
        </xacro:if>
        <xacro:unless value="${hq}">
        <geometry>
-       <mesh filename="package://rb1_base_description/meshes/bases/rb1v2_front_cover.stl"/>
+       <mesh filename="file://$(find rb1_base_description)/meshes/bases/rb1v2_front_cover.stl"/>
        </geometry>
        </xacro:unless>
@@ -82,5 +82,5 @@
        <origin xyz="0 0 0" rpy="0 0 0 " />
        <geometry>
-         <mesh filename="package://rb1_base_description/meshes/bases/rb1v2_front_cover.dae"/>
+         <mesh filename="file://$(find rb1_base_description)/meshes/bases/rb1v2_front_cover.dae"/>
        </geometry>
     </collision>

File: rb1_base_description/urdf/bases/rb1_base_v3.urdf.xacro (robot description, xacro)
@@ -24,5 +24,5 @@
       <origin xyz="0 0 0" rpy="0 0 0" />
       <geometry>
-        <mesh filename="package://rb1_base_description/meshes/bases/rb1_base_v3_color.dae"/>
+        <mesh filename="file://$(find rb1_base_description)/meshes/bases/rb1_base_v3_color.dae"/>
       </geometry>
     </visual>
@@ -44,10 +44,10 @@
        <xacro:if value="${hq}">
        <geometry>
-	     <mesh filename="package://rb1_base_description/meshes/bases/rb1_front_cover_v3.stl"/>
+	     <mesh filename="file://$(find rb1_base_description)/meshes/bases/rb1_front_cover_v3.stl"/>
        </geometry>
        </xacro:if>
        <xacro:unless value="${hq}">
        <geometry>
-       <mesh filename="package://rb1_base_description/meshes/bases/rb1_front_cover_v3.stl"/>
+       <mesh filename="file://$(find rb1_base_description)/meshes/bases/rb1_front_cover_v3.stl"/>
        </geometry>
        </xacro:unless>
@@ -59,5 +59,5 @@
        <origin xyz="0 0 0" rpy="0 0 0 " />
        <geometry>
-         <mesh filename="package://rb1_base_description/meshes/bases/rb1_front_cover_v3.dae"/>
+         <mesh filename="file://$(find rb1_base_description)/meshes/bases/rb1_front_cover_v3.dae"/>
        </geometry>
     </collision>
@@ -79,10 +79,10 @@
        <xacro:if value="${hq}">
 		   <geometry>
-			 <mesh filename="package://rb1_base_description/meshes/bases/rb1_top_cover_v3.stl"/>
+			 <mesh filename="file://$(find rb1_base_description)/meshes/bases/rb1_top_cover_v3.stl"/>
 		   </geometry>
        </xacro:if>
        <xacro:unless value="${hq}">
 		   <geometry>
-		   <mesh filename="package://rb1_base_description/meshes/bases/rb1_top_cover_v3.stl"/>
+		   <mesh filename="file://$(find rb1_base_description)/meshes/bases/rb1_top_cover_v3.stl"/>
 		   </geometry>
        </xacro:unless>
@@ -94,5 +94,5 @@
        <origin xyz="0 0 0" rpy="0 0 0 " />
        <geometry>
-         <mesh filename="package://rb1_base_description/meshes/bases/rb1_top_cover_v3.dae"/>
+         <mesh filename="file://$(find rb1_base_description)/meshes/bases/rb1_top_cover_v3.dae"/>
        </geometry>
     </collision>

File: rb1_base_description/urdf/elevator/elevator.urdf.xacro (robot description, xacro)
@@ -36,10 +36,10 @@
 			<xacro:if value="${hq}">
 				<geometry>
-					<mesh filename="package://rb1_base_description/meshes/elevator/rb1_elevator_base.dae"/>
+					<mesh filename="file://$(find rb1_base_description)/meshes/elevator/rb1_elevator_base.dae"/>
 				</geometry>
 			</xacro:if>
 			<xacro:unless value="${hq}">
 				<geometry>
-					<mesh filename="package://rb1_base_description/meshes/elevator/rb1_elevator_base.stl"/>
+					<mesh filename="file://$(find rb1_base_description)/meshes/elevator/rb1_elevator_base.stl"/>
 				</geometry>
 			</xacro:unless>
@@ -51,5 +51,5 @@
 			<origin xyz="0 0 0" rpy="0 0 0 " />
 			<geometry>
-				<mesh filename="package://rb1_base_description/meshes/elevator/rb1_elevator_base.dae"/>
+				<mesh filename="file://$(find rb1_base_description)/meshes/elevator/rb1_elevator_base.dae"/>
 			</geometry>
 		</collision>
@@ -78,10 +78,10 @@
 			<xacro:if value="${hq}">
 				<geometry>
-					<mesh filename="package://rb1_base_description/meshes/elevator/rb1_elevator_platform.dae"/>
+					<mesh filename="file://$(find rb1_base_description)/meshes/elevator/rb1_elevator_platform.dae"/>
 				</geometry>
 			</xacro:if>
 			<xacro:unless value="${hq}">
 				<geometry>
-					<mesh filename="package://rb1_base_description/meshes/elevator/rb1_elevator_platform.stl"/>
+					<mesh filename="file://$(find rb1_base_description)/meshes/elevator/rb1_elevator_platform.stl"/>
 				</geometry>
 			</xacro:unless>
@@ -93,5 +93,5 @@
 			<origin xyz="0 0 0" rpy="0 0 0 " />
 			<geometry>
-				<mesh filename="package://rb1_base_description/meshes/elevator/rb1_elevator_platform.dae"/>
+				<mesh filename="file://$(find rb1_base_description)/meshes/elevator/rb1_elevator_platform.dae"/>
 			</geometry>
 		</collision>

File: rb1_base_description/urdf/others/kinova_base.urdf.xacro (robot description, xacro)
@@ -15,5 +15,5 @@
        	  <origin xyz="0 0 0" rpy="0 0 0" />
 		  <geometry>
-			<mesh filename="package://rb1_base_description/meshes/others/rb1_kinova_base-v1.dae" />
+			<mesh filename="file://$(find rb1_base_description)/meshes/others/rb1_kinova_base-v1.dae" />
 		  </geometry>
       </visual>
@@ -21,5 +21,5 @@
 		<origin xyz="0 0 0" rpy="${M_PI/2} 0 0" />
         <geometry>
-          <mesh filename="package://rb1_base_description/meshes/others/rb1_kinova_base-v1.dae" />
+          <mesh filename="file://$(find rb1_base_description)/meshes/others/rb1_kinova_base-v1.dae" />
         </geometry>
       </collision>

File: rb1_base_description/urdf/others/tayg_box_6415.urdf.xacro (robot description, xacro)
@@ -13,5 +13,5 @@
        	  <origin xyz="0 0 0" rpy="0 0 0" />
 		  <geometry>
-			<mesh filename="package://rb1_base_description/meshes/others/tayg_box_6415.stl" />
+			<mesh filename="file://$(find rb1_base_description)/meshes/others/tayg_box_6415.stl" />
 		  </geometry>
 		<material name="blue">
@@ -22,5 +22,5 @@
 		<origin xyz="0 0 0" rpy="0 0 0" />
         <geometry>
-          <mesh filename="package://rb1_base_description/meshes/others/tayg_box_6415.stl" />
+          <mesh filename="file://$(find rb1_base_description)/meshes/others/tayg_box_6415.stl" />
         </geometry>
       </collision>

File: rb1_base_description/urdf/others/torso_ur3.urdf.xacro (robot description, xacro)
@@ -15,5 +15,5 @@
        	<origin xyz="0 0 0" rpy="0 0 0" />
         <geometry>
-          <mesh filename="package://rb1_base_description/meshes/others/rb1_torso_ur3.dae" />
+          <mesh filename="file://$(find rb1_base_description)/meshes/others/rb1_torso_ur3.dae" />
         </geometry>
       </visual>
@@ -21,5 +21,5 @@
 		    <origin xyz="0 0 0" rpy="${M_PI/2} 0 0" />
         <geometry>
-          <mesh filename="package://rb1_base_description/meshes/others/rb1_torso_ur3.dae" />
+          <mesh filename="file://$(find rb1_base_description)/meshes/others/rb1_torso_ur3.dae" />
         </geometry>
       </collision>

File: rb1_base_description/urdf/wheels/omni_wheel.urdf.xacro (robot description, xacro)
@@ -29,5 +29,5 @@
           <origin xyz="0 0 0" rpy="0 0 0" />
           <geometry>
-				<mesh filename="package://rb1_base_description/meshes/wheels/rb1v2_omniwheel.dae" />
+				<mesh filename="file://$(find rb1_base_description)/meshes/wheels/rb1v2_omniwheel.dae" />
           </geometry>
         </xacro:if>

File: rb1_base_description/urdf/wheels/omni_wheel_v1.urdf.xacro (robot description, xacro)
@@ -28,5 +28,5 @@
           <origin xyz="0 0 0" rpy="0 0 0" />
           <geometry>
-				<mesh filename="package://rb1_base_description/meshes/wheels/wheel_omni_4inch.dae" />
+				<mesh filename="file://$(find rb1_base_description)/meshes/wheels/wheel_omni_4inch.dae" />
           </geometry>
         </xacro:if>

File: rb1_base_description/urdf/wheels/rubber_wheel.urdf.xacro (robot description, xacro)
@@ -30,8 +30,8 @@
 			<geometry>
 				<xacro:if value="${reflect}">
-					<mesh filename="package://rb1_base_description/meshes/wheels/wheel_rubber_6inch.dae" />
+					<mesh filename="file://$(find rb1_base_description)/meshes/wheels/wheel_rubber_6inch.dae" />
 				</xacro:if>
 				<xacro:unless value="${reflect}">
-					<mesh filename="package://rb1_base_description/meshes/wheels/wheel_rubber_6inch.dae" />
+					<mesh filename="file://$(find rb1_base_description)/meshes/wheels/wheel_rubber_6inch.dae" />
 				</xacro:unless>
 			</geometry>
