Commit message: rb1_base_description: updated stl to remove warning

File: rb1_base_description/urdf/others/tayg_box_6415.urdf.xacro (robot description, xacro)
@@ -15,4 +15,7 @@
 			<mesh filename="package://rb1_base_description/meshes/others/tayg_box_6415.stl" />
 		  </geometry>
+		<material name="blue">
+		<color rgba="0 0 1 1"/>
+      </material>
       </visual>
       <collision>
