Commit message: Changed light to led

File: rb1_base_description/urdf/others/led.urdf.xacro (robot description, xacro)
@@ -3,7 +3,7 @@
 <xacro:macro name="led" params="prefix parent *origin">
 <gazebo>
-   <model name='light_model'>
+   <model name='led_model'>
       <static>1</static>
-      <link name="light_box">
+      <link name="led_box">
         <visual name="${prefix}led_light">
           <pose>0.25 0 0 0 0 0</pose>
@@ -20,5 +20,5 @@
           </material>
         </visual>
-        <light name='light_source' type='spot'>
+        <light name='led_source' type='spot'>
           <pose frame='${prefix}_base_link'>0.25 0 0.25 0 -1.57 0</pose>
           <attenuation>
@@ -48,8 +48,8 @@
         </inertial>
       </link>
-      <plugin name='light_control' filename='libFlashLightPlugin.so'>
+      <plugin name='led_control' filename='libFlashLightPlugin.so'>
         <enable>true</enable>
         <light>
-          <id>light_box/light_source</id>
+          <id>led_box/led_source</id>
           <duration>0.75</duration>
           <interval>0.5</interval>
