Commit message: description: Fix urdf dual ur3 collision issue

File: rb1_base_description/urdf/others/torso_ur3.urdf.xacro (robot description, xacro)
@@ -19,5 +19,5 @@
       </visual>
       <collision>
-		    <origin xyz="0 0 0" rpy="${M_PI/2} 0 0" />
+		    <origin xyz="0 0 0" rpy="0 0 0" />
         <geometry>
           <mesh filename="package://rb1_base_description/meshes/others/rb1_torso_ur3.dae" />
