Commit message: [rb1_base_description]:gazebo elevator with prefix

File: rb1_base_description/urdf/elevator/elevator.gazebo.xacro (robot description, xacro)
@@ -1,43 +1,40 @@
 <?xml version="1.0"?>
-<robot xmlns:xacro="http://ros.org/wiki/xacro">
-	<!-- DIFFERENCIAL DRIVE GAZEBO PLUGIN -->
-	<xacro:macro name="gazebo_differencial_drive">
-		<gazebo>
-			<plugin name="differential_drive_controller" filename="libgazebo_ros_diff_drive.so">
-				<!--alwaysOn>true</alwaysOn-->
-				<updateRate>50.0</updateRate>
-				<leftJoint>left_wheel_joint</leftJoint>
-				<rightJoint>right_wheel_joint</rightJoint>
-				<!--leftJoint>joint_right_wheel</leftJoint>
-				<rightJoint>joint_left_wheel</rightJoint-->
-				<!-- For V0 0.365 -->
-				<!-- wheelSeparation>0.365</wheelSeparation -->
-				<wheelSeparation>0.433</wheelSeparation>
-				<wheelDiameter>0.1524</wheelDiameter>
-				<commandTopic>rb1/cmd_vel</commandTopic>
-				<odometryTopic>odom</odometryTopic>
-				<odometryFrame>odom</odometryFrame>
-				<robotBaseFrame>base_link</robotBaseFrame>
-				<!-- robotNamespace></robotNamespace -->
-				<rosDebugLevel>na</rosDebugLevel>
-				<publishWheelTF>false</publishWheelTF>
-				<publishWheelJointState>true</publishWheelJointState>
-				<wheelAcceleration>0</wheelAcceleration>
-				<wheelTorque>5</wheelTorque>
-				<!-- odometrySource>encoder</odometrySource -->
-				<odometrySource>encoder</odometrySource>
-				<legacyMode>false</legacyMode>
-				<publishTf>1</publishTf>
-			</plugin>
+<robot xmlns:xacro="http://www.ros.org/wiki/xacro">
+	<xacro:macro name="elevator_gazebo" params="prefix">
+		<gazebo reference="${prefix}_platform_link">
+			<mu1 value="5.0"/>
+			<mu2 value="0.5"/>
+			<kp value="10000000.0" />
+			<kd value="1.0" />
+			<fdir1 value="1 0 0"/>
+			<material>Gazebo/Yellow</material>
+			<turnGravityOff>false</turnGravityOff>
+			<!--kp>500000.0</kp>
+			<kd>10.0</kd>
+			<mu1>10</mu1>
+			<mu2>10</mu2>
+			<fdir1>1 0 0</fdir1-->
+			<!--minDepth>0.001</minDepth-->
+			<!--material>Gazebo/Black</material-->
+			<!--mu1 value="10"/>
+			<mu2 value="5"/>
+			<kp value="500000.0" />
+			<kd value="10.0" />
+			<fdir1 value="1 0 0"/>
+			<material>Gazebo/Yellow</material>
+			<turnGravityOff>false</turnGravityOff-->
 		</gazebo>
+		<!--gazebo reference="${name}_wheel_link">
+			<kp>500000.0</kp>
+			<kd>10.0</kd>
+			<mu1>10</mu1>
+			<mu2>10</mu2>
+			<fdir1>1 0 0</fdir1>
+			<maxVel>1.0</maxVel>
+			<minDepth>0.003</minDepth>
+			<material>Gazebo/Yellow</material>
+			<turnGravityOff>false</turnGravityOff>
+			<implicitSpringDamper>1</implicitSpringDamper>
+		</gazebo-->
 	</xacro:macro>
-	<gazebo reference="base_footprint">
-		<material>Gazebo/Green</material>
-	</gazebo>
-	<gazebo reference="base_link">
-		<material>Gazebo/Grey</material>
-	</gazebo>
-	<gazebo reference="front_cover_link">
-		<material>Gazebo/Black</material>
-	</gazebo>
 </robot>
