Commit message: enabling Gazebo fake elevator and fixing elevator urdf model(transmission & gazebo were commented)

File: rb1_base_description/urdf/elevator/elevator.transmission.xacro (robot description, xacro)
@@ -10,9 +10,9 @@
 				<!--hardwareInterface>EffortJointInterface</hardwareInterface-->
 				<!-- for ros control controller -->
-				<hardwareInterface>hardware_interface/PositionJointInterface</hardwareInterface>
+				<hardwareInterface>hardware_interface/EffortJointInterface</hardwareInterface>
 			</joint>
 			<actuator name="${prefix}_platform_joint_motor">
+				<hardwareInterface>EffortJointInterface</hardwareInterface>
 				<mechanicalReduction>1</mechanicalReduction>
-				<motorTorqueConstant>20</motorTorqueConstant>
 			</actuator>
 		</transmission>

File: rb1_base_description/urdf/elevator/elevator.urdf.xacro (robot description, xacro)
@@ -14,5 +14,5 @@
 	</joint>
 	<link name="${prefix}_base_link">
-		<!--inertial>
+		<inertial>
 			<mass value="25.0" />
 			<origin xyz="0 0 0" />
@@ -20,5 +20,5 @@
 						iyy="0.007"  iyz="0.0"
 						izz="0.78125"/>
-		</inertial-->
+		</inertial>
 		<visual>
 			<origin xyz="0 0 0" rpy="0 0 0" />
@@ -50,12 +50,12 @@
 			<child link="${prefix}_platform_link" />
 			<axis xyz="0 0 1"/>
-			<limit effort="1.0" lower="0.0" upper="0.034" velocity="0.5"/>
+			<limit effort="10.0" lower="0.0" upper="0.034" velocity="0.5"/>
 	</joint>
 	<link name="${prefix}_platform_link">
-		<!--inertial>
-			<mass value="0.25" />
+		<inertial>
+			<mass value="0.05" />
 			<origin xyz="0 0 0" />
 			<inertia  ixx="0.00007" ixy="0.0"  ixz="0.0"  iyy="0.00007"  iyz="0.0"  izz="0.0078" />
-		</inertial-->
+		</inertial>
 		<visual>
 			<origin xyz="0 0 0" rpy="0 0 0" />
@@ -81,6 +81,6 @@
 		</collision>
 	</link>
-	<!--xacro:elevator_transmission prefix="${prefix}" />
-	<xacro:elevator_gazebo prefix="${prefix}" /-->
+	<xacro:elevator_transmission prefix="${prefix}" />
+	<xacro:elevator_gazebo prefix="${prefix}" />
 	</xacro:macro>
 </robot>
