Commit message: rb1_base_description: added elevator platform in the model

File: rb1_base_description/robots/versions/rb1_base_171019A.urdf.xacro (robot description, xacro)
@@ -33,4 +33,10 @@
 	<!-- Flag to select the high or low quality model -->
 	<xacro:property name="hq" value="true" />
+	<!-- ******************* -->
+	<!-- ELEVATOR PARAMETERS -->
+	<!-- ******************* -->
+	<xacro:property name="elevator_x" value="0.0" />
+	<xacro:property name="elevator_y" value="0.0" />
+	<xacro:property name="elevator_z" value="0.213" />
 	<!-- *************** -->
 	<!-- Robots Elements -->
@@ -60,4 +66,8 @@
 		<origin xyz="${omni_front_x} -${omni_front_y} ${omni_front_z}" rpy="0 0 0"/>
 	</xacro:omni_wheel>
+	<!-- ELEVATOR_PLATFORM -->
+	<xacro:elevator_platform prefix="$(arg prefix)elevator" parent="$(arg prefix)base_link" hq="${hq}">
+		<origin xyz="${elevator_x} -${elevator_y} ${elevator_z}" rpy="0 0 0"/>
+	</xacro:elevator_platform>
 	<!-- SENSORS -->
 	<xacro:sensor_sick_tim571 prefix="$(arg prefix)front_laser" parent="$(arg prefix)base_link" prefix_topic="front_laser">
